Commit message: pi value

File: reachy_description/urdf/orbita2dof.urdf.xacro (robot description, xacro)
@@ -32,5 +32,5 @@
       <xacro:joint2axis joint="${joint1}"/>
       <limit lower="${joint1_min_angle}" upper="${joint1_max_angle}" effort="1000.0" velocity="100.0"/>
-      <safety_controller k_velocity="500" k_position="500" soft_lower_limit="-3.1415" soft_upper_limit="3.1415.0" />
+      <safety_controller k_velocity="500" k_position="500" soft_lower_limit="-3.1415" soft_upper_limit="3.1415" />
       <dynamics damping="${damping}" friction="${friction}"/>
     </joint>

File: reachy_description/urdf/reachy.urdf.xacro (robot description, xacro)
@@ -35,5 +35,5 @@
   <!-- MODEL PARAMETERS -->
   <xacro:property name="base_collision" value="false"/>
-  <xacro:property name="base_visual" value="false"/>
+  <xacro:property name="base_visual" value="true"/>
   <xacro:property name="damping" value="0.1"/>
   <xacro:property name="friction" value="0.1"/>
@@ -59,8 +59,12 @@
     <xacro:if value="${base_visual}">
       <visual>
-        <origin xyz="0 0 -0.5" rpy="0 0 0"/>
+        <origin xyz="0 0 -0.1" rpy="0 0.0 0"/>
         <geometry>
-          <cylinder length="1" radius="0.03"/>
+          <box size="0.11 0.2 0.32"/>
         </geometry>
+        <!-- <origin xyz="0 0 -0.5" rpy="0 0 0"/> -->
+        <!-- <geometry> -->
+        <!--   <cylinder length="1" radius="0.03"/> -->
+        <!-- </geometry> -->
         <material name="black"/>
       </visual>
