Commit message: fix gazebo

File: reachy_description/urdf/reachy.urdf.xacro (robot description, xacro)
@@ -6,4 +6,5 @@
   <xacro:include filename="$(find reachy_description)/urdf/head.urdf.xacro"/>
   <xacro:include filename="$(find pollen_generic_description)/urdf/inertial_primitives.urdf.xacro"/>
+  <xacro:include filename="$(find pollen_generic_description)/urdf/materials.urdf.xacro"/>
   <!-- config  -->
   <xacro:arg name="neck_config" default="$(find orbita3d_controller)/config/fake.yaml"/>
@@ -26,7 +27,7 @@
   <xacro:property name="forearm_length" value="0.28"/>
   <!-- MODEL PARAMETERS -->
-    <material name="torsoblack">
-        <color rgba="0.5 0.5 0.5 1.0"/>
-    </material>
+    <!-- <material name="torsoblack"> -->
+    <!--     <color rgba="0.5 0.5 0.5 1.0"/> -->
+    <!-- </material> -->
   <link name="world"/>
   <joint name="world_joint" type="fixed">
@@ -55,5 +56,6 @@
         <!--   <cylinder length="1" radius="0.03"/> -->
         <!-- </geometry> -->
-        <material name="torsoblack"/>
+        <!-- <material name="torsoblack"/> -->
+	<xacro:torsoblack/>
       </visual>
     </xacro:if>
@@ -105,3 +107,12 @@
     <!-- gripper_id="${left_gripper_id}" -->
     <!-- /> -->
+    <xacro:if value="$(arg use_gazebo)">
+        <gazebo>
+            <plugin name="gazebo_ros2_control" filename="libgazebo_ros2_control.so">
+                <!-- <parameters>$(find reachy_bringup)/config/reachy_${robot_config}_controllers.yaml</parameters> -->
+                <parameters>$(find reachy_bringup)/config/reachy_full_kit_controllers.yaml</parameters>
+                <robotNamespace>/reachy</robotNamespace>
+            </plugin>
+        </gazebo>
+    </xacro:if>
 </robot>

Commit message: change everything to reachy_v2_wip

File: reachy_description/urdf/reachy.urdf.xacro (robot description, xacro)
@@ -1,4 +1,4 @@
 <?xml version="1.0" ?>
-<robot xmlns:xacro="http://www.ros.org/wiki/xacro" name="generic_arm">
+<robot xmlns:xacro="http://www.ros.org/wiki/xacro" name="reachy_v2">
   <xacro:arg name="use_fake_hardware" default="false"/>
   <xacro:arg name="use_gazebo" default="false"/>
@@ -8,8 +8,8 @@
   <xacro:include filename="$(find pollen_generic_description)/urdf/materials.urdf.xacro"/>
   <!-- config  -->
-  <xacro:arg name="neck_config" default="$(find orbita3d_controller)/config/fake.yaml"/>
-  <xacro:arg name="r_shoulder_config" default="$(find orbita2d_controller)/config/fake.yaml"/>
-  <xacro:arg name="r_elbow_config" default="$(find orbita2d_controller)/config/fake.yaml"/>
-  <xacro:arg name="r_wrist_config" default="$(find orbita3d_controller)/config/fake.yaml"/>
+  <xacro:arg name="neck_config" default="$(find orbita3d_description)/config/fake.yaml"/>
+  <xacro:arg name="r_shoulder_config" default="$(find orbita2d_description)/config/fake.yaml"/>
+  <xacro:arg name="r_elbow_config" default="$(find orbita2d_description)/config/fake.yaml"/>
+  <xacro:arg name="r_wrist_config" default="$(find orbita3d_description)/config/fake.yaml"/>
   <xacro:property name="right_gripper_id" value="11"/>
   <xacro:property name="right_gripper_port" value="/dev/right_gripper"/>

File: reachy_moveit_config/config/reachy_v2_wip.ros2_control.xacro (robot description, xacro)
@@ -1,5 +1,5 @@
 <?xml version="1.0"?>
 <robot xmlns:xacro="http://www.ros.org/wiki/xacro">
-    <xacro:macro name="reachy_2023_ros2_control" params="name initial_positions_file">
+    <xacro:macro name="reachy_v2_ros2_control" params="name initial_positions_file">
         <xacro:property name="initial_positions" value="${load_yaml(initial_positions_file)['initial_positions']}"/>
         <ros2_control name="${name}" type="system">

File: reachy_moveit_config/config/reachy_v2_wip.urdf.xacro (robot description, xacro)
@@ -2,5 +2,5 @@
 <robot xmlns:xacro="http://www.ros.org/wiki/xacro" name="reachy_v2_wip">
     <xacro:arg name="initial_positions_file" default="initial_positions.yaml" />
-    <!-- Import reachy_2023 urdf file -->
+    <!-- Import reachy_v2 urdf file -->
     <xacro:arg name="use_fake_hardware" default="true" />
     <xacro:arg name="use_gazebo" default="true" />
@@ -10,5 +10,5 @@
     <!-- No need as we use the reachy_description -->
     <!-- Import control_xacro -->
-    <!-- <xacro:include filename="reachy_2023.ros2_control.xacro" /> -->
-    <!-- <xacro:reachy_2023_ros2_control name="FakeSystem" initial_positions_file="$(arg initial_positions_file)"/> -->
+    <!-- <xacro:include filename="reachy_v2_wip.ros2_control.xacro" /> -->
+    <!-- <xacro:reachy_v2_wip_ros2_control name="FakeSystem" initial_positions_file="$(arg initial_positions_file)"/> -->
 </robot>

Commit message: it seems to work in fake

File: reachy_description/urdf/reachy.urdf.xacro (robot description, xacro)
@@ -14,9 +14,10 @@
   <xacro:property name="right_gripper_id" value="11"/>
   <xacro:property name="right_gripper_port" value="/dev/right_gripper"/>
+  <xacro:arg name="l_shoulder_config" default="$(find orbita2d_description)/config/fake.yaml"/>
+  <xacro:arg name="l_elbow_config" default="$(find orbita2d_description)/config/fake.yaml"/>
+  <xacro:arg name="l_wrist_config" default="$(find orbita3d_description)/config/fake.yaml"/>
+  <xacro:property name="left_gripper_id" value="12"/>
+  <xacro:property name="left_gripper_port" value="/dev/left_gripper"/>
   <!-- config  -->
-  <!-- HWI IDs -->
-    <!-- <xacro:property name="left_gripper_id" value="12"/> -->
-    <!-- <xacro:property name="left_gripper_port" value="/dev/left_gripper"/> -->
-  <!-- HWI IDs -->
   <!-- MODEL PARAMETERS -->
   <xacro:property name="base_collision" value="false"/>
@@ -83,4 +84,14 @@
     gripper_port="${right_gripper_port}"
     />
+  <!-- LEFT ARM -->
+  <xacro:arm
+    prefix="l" parent="torso" side="left"
+    damping="${damping}" friction="${friction}"
+    orbita2d_shoulder_config="$(arg l_shoulder_config)"
+    orbita2d_elbow_config="$(arg l_elbow_config)"
+    orbita3d_wrist_config="$(arg l_wrist_config)"
+    gripper_id="${left_gripper_id}"
+    gripper_port="${left_gripper_port}"
+    />
   <!-- <link name="r_wrist_cam_frame"/> -->
   <!-- <joint name="r_wrist_cam_frame_joint" type="fixed"> -->
@@ -95,16 +106,4 @@
   <!--   <child link="r_wrist_camera"/> -->
   <!-- </joint> -->
-  <!-- LEFT ARM -->
-    <!-- <xacro:arm -->
-    <!-- prefix="l" parent="torso" side="left" -->
-    <!-- damping="${damping}" friction="${friction}" -->
-    <!-- shoulder_port_a="${left_shoulder_port_a}" shoulder_port_b="${left_shoulder_port_b}" -->
-    <!-- elbow_port_a="${left_elbow_port_a}" elbow_port_b="${left_elbow_port_b}" -->
-    <!-- wrist_port="${left_wrist_port}" -->
-    <!-- shoulder_id_a="${left_shoulder_id_a}" shoulder_id_b="${left_shoulder_id_b}" -->
-    <!-- elbow_id_a="${left_elbow_id_a}" elbow_id_b="${left_elbow_id_b}" -->
-    <!-- wrist_id="${left_wrist_id}" -->
-    <!-- gripper_id="${left_gripper_id}" -->
-    <!-- /> -->
     <xacro:if value="$(arg use_gazebo)">
         <gazebo>

File: reachy_description/urdf/smartgripper.urdf.xacro (robot description, xacro)
@@ -3,4 +3,5 @@
 <xacro:macro name="smartgripper" params="prefix parent side damping friction gripper_port gripper_id">
   <xacro:include filename="$(find reachy_description)/ros2_control/smartgripper.ros2_control.xacro"/>
+  <xacro:include filename="$(find pollen_generic_description)/urdf/materials.urdf.xacro"/>
   <xacro:property name="gripper_length" value="0.12"/>
   <xacro:property name="gripper_radius" value="0.03"/>
@@ -16,10 +17,10 @@
     <xacro:property name="max_grasping_finger" value="2.094"/>
   </xacro:if>
-    <material name="gripperblack">
-        <color rgba="0.4 0.4 0.4 1"/>
-    </material>
-    <material name="gripperwhite">
-        <color rgba="0.9 0.9 0.9 1"/>
-    </material>
+    <!-- <material name="gripperblack"> -->
+    <!--     <color rgba="0.4 0.4 0.4 1"/> -->
+    <!-- </material> -->
+    <!-- <material name="gripperwhite"> -->
+    <!--     <color rgba="0.9 0.9 0.9 1"/> -->
+    <!-- </material> -->
   <xacro:property name="p" value="${prefix}_gripper"/>
   <link name="${p}_palm_link">
@@ -35,5 +36,6 @@
         <box size="${gripper_radius} ${gripper_radius*2} ${gripper_length/2}"/>
       </geometry>
-      <material name="gripperblack"/>
+      <!-- <material name="gripperblack"/> -->
+      <xacro:gripperblack/>
     </visual>
     <xacro:inertial_cuboid mass="${gripper_mass*0.85}" xyz="0 0 ${gripper_length/4}"  rpy="0 0 0" x_length="${gripper_radius}" y_length="${gripper_radius*2}" z_length="${gripper_length/2}"/>
@@ -56,5 +58,6 @@
         <box size="${gripper_radius} 0.01 ${gripper_length/2}"/>
       </geometry>
-      <material name="gripperwhite"/>
+      <!-- <material name="gripperwhite"/> -->
+      <xacro:gripperwhite/>
     </visual>
     <xacro:inertial_cuboid mass="${gripper_mass*0.1}" xyz="0 ${gripper_radius} ${gripper_length/4}"  rpy="0 0 0" x_length="${gripper_radius}" y_length="0.01" z_length="${gripper_length/2}"/>
@@ -72,5 +75,6 @@
         <box size="${gripper_radius} 0.01 ${gripper_length/2}"/>
       </geometry>
-      <material name="gripperwhite"/>
+      <!-- <material name="gripperwhite"/> -->
+      <xacro:gripperwhite/>
     </visual>
     <xacro:inertial_cuboid mass="${gripper_mass*0.1}" xyz="0 ${gripper_radius} ${gripper_length/4}"  rpy="0 0 0" x_length="${gripper_radius}" y_length="0.01" z_length="${gripper_length/2}"/>

Commit message: octomap ok

File: reachy_description/urdf/reachy.urdf.xacro (robot description, xacro)
@@ -22,5 +22,5 @@
   <!-- config  -->
   <!-- MODEL PARAMETERS -->
-  <xacro:property name="base_collision" value="false"/>
+  <xacro:property name="base_collision" value="true"/>
   <xacro:property name="base_visual" value="true"/>
   <xacro:property name="damping" value="0.1"/>
@@ -42,5 +42,15 @@
     <xacro:if value="${base_collision}">
       <collision>
-        <origin xyz="0 0 -0.5" rpy="0 0 0"/>
+        <origin xyz="-0.05 0 -0.05" rpy="0 0.0 0"/>
+        <geometry>
+          <box size="0.1 0.2 0.22"/>
+        </geometry>
+        <!-- <origin xyz="0 0 -0.5" rpy="0 0 0"/> -->
+        <!-- <geometry> -->
+        <!--   <cylinder length="1" radius="0.03"/> -->
+        <!-- </geometry> -->
+      </collision>
+      <collision>
+        <origin xyz="-0.15 0 -0.5" rpy="0 0 0"/>
         <geometry>
           <cylinder length="1" radius="0.03"/>
@@ -54,9 +64,12 @@
           <box size="0.1 0.2 0.22"/>
         </geometry>
-        <!-- <origin xyz="0 0 -0.5" rpy="0 0 0"/> -->
-        <!-- <geometry> -->
-        <!--   <cylinder length="1" radius="0.03"/> -->
-        <!-- </geometry> -->
         <!-- <material name="torsoblack"/> -->
+	<xacro:torsoblack/>
+      </visual>
+      <visual>
+        <origin xyz="-0.15 0 -0.5" rpy="0 0 0"/>
+        <geometry>
+          <cylinder length="1" radius="0.03"/>
+        </geometry>
 	<xacro:torsoblack/>
       </visual>

Commit message: every controller is loaded, only moveit seems to be working though, no sdk

File: reachy_description/urdf/reachy.urdf.xacro (robot description, xacro)
@@ -29,7 +29,7 @@
   <xacro:property name="forearm_length" value="0.28"/>
   <!-- MODEL PARAMETERS -->
-    <!-- <material name="torsoblack"> -->
-    <!--     <color rgba="0.5 0.5 0.5 1.0"/> -->
-    <!-- </material> -->
+  <!-- <material name="torsoblack"> -->
+  <!--     <color rgba="0.5 0.5 0.5 1.0"/> -->
+  <!-- </material> -->
   <link name="world"/>
   <joint name="world_joint" type="fixed">
@@ -65,5 +65,5 @@
         </geometry>
         <!-- <material name="torsoblack"/> -->
-	<xacro:torsoblack/>
+        <xacro:torsoblack/>
       </visual>
       <visual>
@@ -72,5 +72,5 @@
           <cylinder length="1" radius="0.03"/>
         </geometry>
-	<xacro:torsoblack/>
+        <xacro:torsoblack/>
       </visual>
     </xacro:if>
@@ -83,29 +83,29 @@
   <!-- TORSO -->
   <xacro:head
-    parent="torso"
-    damping="${damping}" friction="${friction}"
-    neck_config="$(arg neck_config)"
+          parent="torso"
+          damping="${damping}" friction="${friction}"
+          neck_config="$(arg neck_config)"
   />
-<!-- <xacro:macro name="arm" params="prefix parent side damping friction orbita2d_shoulder_config orbita2d_elbow_config orbita3d_wrist_config gripper_port gripper_id"> -->
+  <!-- <xacro:macro name="arm" params="prefix parent side damping friction orbita2d_shoulder_config orbita2d_elbow_config orbita3d_wrist_config gripper_port gripper_id"> -->
   <!-- RIGHT ARM -->
   <xacro:arm
-    prefix="r" parent="torso" side="right"
-    damping="${damping}" friction="${friction}"
-    orbita2d_shoulder_config="$(arg r_shoulder_config)"
-    orbita2d_elbow_config="$(arg r_elbow_config)"
-    orbita3d_wrist_config="$(arg r_wrist_config)"
-    gripper_id="${right_gripper_id}"
-    gripper_port="${right_gripper_port}"
-    />
+          prefix="r" parent="torso" side="right"
+          damping="${damping}" friction="${friction}"
+          orbita2d_shoulder_config="$(arg r_shoulder_config)"
+          orbita2d_elbow_config="$(arg r_elbow_config)"
+          orbita3d_wrist_config="$(arg r_wrist_config)"
+          gripper_id="${right_gripper_id}"
+          gripper_port="${right_gripper_port}"
+  />
   <!-- LEFT ARM -->
   <xacro:arm
-    prefix="l" parent="torso" side="left"
-    damping="${damping}" friction="${friction}"
-    orbita2d_shoulder_config="$(arg l_shoulder_config)"
-    orbita2d_elbow_config="$(arg l_elbow_config)"
-    orbita3d_wrist_config="$(arg l_wrist_config)"
-    gripper_id="${left_gripper_id}"
-    gripper_port="${left_gripper_port}"
-    />
+          prefix="l" parent="torso" side="left"
+          damping="${damping}" friction="${friction}"
+          orbita2d_shoulder_config="$(arg l_shoulder_config)"
+          orbita2d_elbow_config="$(arg l_elbow_config)"
+          orbita3d_wrist_config="$(arg l_wrist_config)"
+          gripper_id="${left_gripper_id}"
+          gripper_port="${left_gripper_port}"
+  />
   <!-- <link name="r_wrist_cam_frame"/> -->
   <!-- <joint name="r_wrist_cam_frame_joint" type="fixed"> -->
@@ -120,22 +120,13 @@
   <!--   <child link="r_wrist_camera"/> -->
   <!-- </joint> -->
-    <xacro:if value="$(arg use_gazebo)">
-      <xacro:unless value="$(arg use_moveit_gazebo)">
-        <gazebo>
-            <plugin name="gazebo_ros2_control" filename="libgazebo_ros2_control.so">
-                <!-- <parameters>$(find reachy_bringup)/config/reachy_${robot_config}_controllers.yaml</parameters> -->
-                <parameters>$(find reachy_bringup)/config/reachy_full_kit_controllers.yaml</parameters>
-                <robotNamespace>/reachy</robotNamespace>
-            </plugin>
-        </gazebo>
-        </xacro:unless>
-	<xacro:if value="$(arg use_moveit_gazebo)">
-      <gazebo>
-	<plugin name="gazebo_ros2_control" filename="libgazebo_ros2_control.so">
-	  <parameters>$(find reachy_moveit_config)/config/ros2_controllers.yaml</parameters>
-	  <robotNamespace>/reachy</robotNamespace>
-	</plugin>
-      </gazebo>
-    </xacro:if>
-   </xacro:if>
+  <xacro:if value="$(arg use_gazebo)">
+    <gazebo>
+      <plugin name="gazebo_ros2_control" filename="libgazebo_ros2_control.so">
+        <!-- <parameters>$(find reachy_bringup)/config/reachy_${robot_config}_controllers.yaml</parameters> -->
+        <!--          <parameters>$(find reachy_bringup)/config/reachy_full_kit_controllers.yaml</parameters>-->
+        <parameters>$(find reachy_bringup)/config/ros2_controllers_ultimate_combo_top_moumoute.yaml</parameters>
+        <robotNamespace>/reachy</robotNamespace>
+      </plugin>
+    </gazebo>
+  </xacro:if>
 </robot>
