Commit message: conf rework wip

File: reachy_description/urdf/reachy.urdf.xacro (robot description, xacro)
@@ -1,47 +1,33 @@
-<?xml version="1.0" ?>
+<?xml version="1.0"?>
 <robot xmlns:xacro="http://www.ros.org/wiki/xacro" name="reachy2">
-  <xacro:arg name="use_fake_hardware" default="false"/>
-  <xacro:arg name="use_gazebo" default="false"/>
-  <xacro:arg name="use_moveit_gazebo" default="false"/>
-  <xacro:include filename="$(find reachy_description)/urdf/arm.urdf.xacro"/>
-  <xacro:include filename="$(find reachy_description)/urdf/head.urdf.xacro"/>
-  <xacro:include filename="$(find pollen_generic_description)/urdf/inertial_primitives.urdf.xacro"/>
-  <xacro:include filename="$(find pollen_generic_description)/urdf/materials.urdf.xacro"/>
+  <xacro:arg name="use_fake_hardware" default="false" />
+  <xacro:arg name="use_gazebo" default="false" />
+  <xacro:arg name="use_moveit_gazebo" default="false" />
+  <xacro:include filename="$(find reachy_description)/urdf/head.urdf.xacro" />
+  <xacro:include filename="$(find arm_description)/urdf/arm.urdf.xacro" />
+  <xacro:include filename="$(find pollen_generic_description)/urdf/inertial_primitives.urdf.xacro" />
+  <xacro:include filename="$(find pollen_generic_description)/urdf/materials.urdf.xacro" />
+  <xacro:include filename="$(find orbita2d_description)/urdf/orbita2d.urdf.xacro" />
   <!-- config  -->
-  <xacro:arg name="neck_config" default="$(find orbita3d_description)/config/fake.yaml"/>
-  <xacro:arg name="r_shoulder_config" default="$(find orbita2d_description)/config/fake.yaml"/>
-  <xacro:arg name="r_elbow_config" default="$(find orbita2d_description)/config/fake.yaml"/>
-  <xacro:arg name="r_wrist_config" default="$(find orbita3d_description)/config/fake.yaml"/>
-  <xacro:property name="right_gripper_id" value="11"/>
-  <xacro:property name="right_gripper_port" value="/dev/right_gripper"/>
-  <xacro:arg name="l_shoulder_config" default="$(find orbita2d_description)/config/fake.yaml"/>
-  <xacro:arg name="l_elbow_config" default="$(find orbita2d_description)/config/fake.yaml"/>
-  <xacro:arg name="l_wrist_config" default="$(find orbita3d_description)/config/fake.yaml"/>
-  <xacro:property name="left_gripper_id" value="12"/>
-  <xacro:property name="left_gripper_port" value="/dev/left_gripper"/>
- <xacro:include filename="$(find pollen_generic_description)/urdf/inertial_primitives.urdf.xacro" />
-  <xacro:include filename="$(find orbita2d_description)/urdf/orbita2d.urdf.xacro" />
-  <xacro:include filename="$(find arm_description)/urdf/arm.urdf.xacro" />
-  <!-- Orbita2d config -->
-  <!-- <xacro:arg name="config_file" default="fake.yaml"/> -->
-  <xacro:arg name="right_arm_config" default="fake.yaml" />
-  <xacro:arg name="left_arm_config" default="fake.yaml" />
+  <xacro:arg name="neck_config" default="$(find orbita3d_description)/config/fake.yaml" />
+  <xacro:arg name="right_arm_config" default="$(find arm_controller)/config/fake_arm.yaml" />
+  <xacro:arg name="left_arm_config" default="$(find arm_controller)/config/fake_arm.yaml" />
   <!-- config  -->
   <!-- MODEL PARAMETERS -->
-  <xacro:property name="base_collision" value="true"/>
-  <xacro:property name="base_visual" value="true"/>
-  <xacro:property name="damping" value="0.1"/>
-  <xacro:property name="friction" value="0.1"/>
-  <xacro:property name="arm_length" value="0.28"/>
-  <xacro:property name="forearm_length" value="0.28"/>
+  <xacro:property name="base_collision" value="true" />
+  <xacro:property name="base_visual" value="true" />
+  <xacro:property name="damping" value="0.1" />
+  <xacro:property name="friction" value="0.1" />
+  <xacro:property name="arm_length" value="0.28" />
+  <xacro:property name="forearm_length" value="0.28" />
   <!-- MODEL PARAMETERS -->
   <!-- <material name="torsoblack"> -->
   <!--     <color rgba="0.5 0.5 0.5 1.0"/> -->
   <!-- </material> -->
-  <link name="world"/>
+  <link name="world" />
   <joint name="world_joint" type="fixed">
-    <origin xyz="0 0 1.0" rpy="0 0 0"/>
-    <parent link="world"/>
-    <child link="torso"/>
+    <origin xyz="0 0 1.0" rpy="0 0 0" />
+    <parent link="world" />
+    <child link="torso" />
   </joint>
   <!-- TORSO -->
@@ -49,7 +35,7 @@
     <xacro:if value="${base_collision}">
       <collision>
-        <origin xyz="-0.05 0 -0.05" rpy="0 0.0 0"/>
+        <origin xyz="-0.05 0 -0.05" rpy="0 0.0 0" />
         <geometry>
-          <box size="0.1 0.2 0.22"/>
+          <box size="0.1 0.2 0.22" />
         </geometry>
         <!-- <origin xyz="0 0 -0.5" rpy="0 0 0"/> -->
@@ -59,7 +45,7 @@
       </collision>
       <collision>
-        <origin xyz="-0.15 0 -0.5" rpy="0 0 0"/>
+        <origin xyz="-0.15 0 -0.5" rpy="0 0 0" />
         <geometry>
-          <cylinder length="1" radius="0.03"/>
+          <cylinder length="1" radius="0.03" />
         </geometry>
       </collision>
@@ -67,20 +53,21 @@
     <xacro:if value="${base_visual}">
       <visual>
-        <origin xyz="-0.05 0 -0.05" rpy="0 0.0 0"/>
+        <origin xyz="-0.05 0 -0.05" rpy="0 0.0 0" />
         <geometry>
-          <box size="0.1 0.2 0.22"/>
+          <box size="0.1 0.2 0.22" />
         </geometry>
         <!-- <material name="torsoblack"/> -->
-        <xacro:torsoblack/>
+        <xacro:torsoblack />
       </visual>
       <visual>
-        <origin xyz="-0.15 0 -0.5" rpy="0 0 0"/>
+        <origin xyz="-0.15 0 -0.5" rpy="0 0 0" />
         <geometry>
-          <cylinder length="1" radius="0.03"/>
+          <cylinder length="1" radius="0.03" />
         </geometry>
-        <xacro:torsoblack/>
+        <xacro:torsoblack />
       </visual>
     </xacro:if>
-    <xacro:inertial_cuboid mass="10" xyz="0 0 0.5"  rpy="0 0 0" x_length="0.05" y_length="0.05" z_length="1"/>
+    <xacro:inertial_cuboid mass="10" xyz="0 0 0.5" rpy="0 0 0" x_length="0.05" y_length="0.05"
+      z_length="1" />
   </link>
   <gazebo reference="torso">
@@ -90,14 +77,15 @@
   <!-- TORSO -->
   <xacro:head
-          parent="torso"
-          damping="${damping}" friction="${friction}"
-          neck_config="$(arg neck_config)"
+    parent="torso"
+    damping="${damping}" friction="${friction}"
+    neck_config="$(arg neck_config)"
   />
-  <!-- <xacro:macro name="arm" params="prefix parent side damping friction orbita2d_shoulder_config orbita2d_elbow_config orbita3d_wrist_config gripper_port gripper_id"> -->
- <xacro:arm
+  <!-- RIGHT ARM -->
+  <xacro:arm
     prefix="r" parent="torso" side="right"
     damping="${damping}" friction="${friction}"
     config_file="$(arg right_arm_config)"
   />
+  <!-- LEFT ARM -->
   <xacro:arm
     prefix="l" parent="torso" side="left"
@@ -105,24 +93,4 @@
     config_file="$(arg left_arm_config)"
   />
-  <!-- RIGHT ARM -->
-  <!-- <xacro:arm
-          prefix="r" parent="torso" side="right"
-          damping="${damping}" friction="${friction}"
-          orbita2d_shoulder_config="$(arg r_shoulder_config)"
-          orbita2d_elbow_config="$(arg r_elbow_config)"
-          orbita3d_wrist_config="$(arg r_wrist_config)"
-          gripper_id="${right_gripper_id}"
-          gripper_port="${right_gripper_port}"
-  /> -->
-  <!-- LEFT ARM -->
-  <!-- <xacro:arm
-          prefix="l" parent="torso" side="left"
-          damping="${damping}" friction="${friction}"
-          orbita2d_shoulder_config="$(arg l_shoulder_config)"
-          orbita2d_elbow_config="$(arg l_elbow_config)"
-          orbita3d_wrist_config="$(arg l_wrist_config)"
-          gripper_id="${left_gripper_id}"
-          gripper_port="${left_gripper_port}"
-  /> -->
   <!-- <link name="r_wrist_cam_frame"/> -->
   <!-- <joint name="r_wrist_cam_frame_joint" type="fixed"> -->
@@ -140,7 +108,10 @@
     <gazebo>
       <plugin name="gazebo_ros2_control" filename="libgazebo_ros2_control.so">
-        <!-- <parameters>$(find reachy_bringup)/config/reachy_${robot_config}_controllers.yaml</parameters> -->
-<!--                  <parameters>$(find reachy_bringup)/config/reachy_full_kit_controllers.yaml</parameters>-->
+        <!-- <parameters>$(find
+        reachy_bringup)/config/reachy_${robot_config}_controllers.yaml</parameters> -->
+        <!--                  <parameters>$(find
+        reachy_bringup)/config/reachy_full_kit_controllers.yaml</parameters>-->
         <parameters>$(find reachy_bringup)/config/ros2_controllers_ultimate_combo_top_moumoute.yaml</parameters>
+        <!-- TODO FIX ME PROPER controller import  -->
         <robotNamespace>/reachy</robotNamespace>
       </plugin>

Commit message: wip

File: reachy_description/urdf/reachy.urdf.xacro (robot description, xacro)
@@ -143,4 +143,5 @@
 	<!-- <mesh filename="package://reachy_description/meshes/torso_visual_high.dae" /> -->
 	<mesh filename="file://$(find reachy_description)/meshes/torso_visual_high.dae" />
+	<!-- <mesh filename="file://$(find reachy_description)/meshes/torso_visual_high2.dae" /> -->
       </geometry>
     </visual>
@@ -256,7 +257,7 @@
           <update_rate>30</update_rate>
           <camera name="sr_cam_l">
-            <horizontal_fov>1.3962634</horizontal_fov>
+            <horizontal_fov>${77.0*pi/180}</horizontal_fov>
             <image>
-              <width>800</width>
+              <width>1280</width>
               <height>800</height>
               <format>R8G8B8</format>
@@ -306,7 +307,7 @@
           <update_rate>30</update_rate>
           <camera name="sr_cam_r">
-            <horizontal_fov>1.3962634</horizontal_fov>
+            <horizontal_fov>${77.0*pi/180}</horizontal_fov>
             <image>
-              <width>800</width>
+              <width>1280</width>
               <height>800</height>
               <format>R8G8B8</format>
@@ -354,8 +355,8 @@
             <pose>0 0 0 0 0 0</pose>
             <camera name="realsense_depth_camera">
-              <horizontal_fov>1.46608</horizontal_fov>
+              <horizontal_fov>${77.0*pi/180}</horizontal_fov>
               <image>
-                <width>424</width>
-                <height>240</height>
+                <width>1280</width>
+                <height>800</height>
                 <format>B8G8R8</format>
               </image>
@@ -364,4 +365,9 @@
                 <far>8</far>
               </clip>
+            <noise>
+              <type>gaussian</type>
+              <mean>0.0</mean>
+              <stddev>0.7</stddev>
+            </noise>
             </camera>
             <!-- https://github.com/mlherd/ros2_turtlebot3_waffle_intel_realsense -->

Commit message: wip

File: reachy_description/urdf/reachy.urdf.xacro (robot description, xacro)
@@ -19,5 +19,5 @@
   <xacro:property name="friction" value="0.1" />
   <!-- Height of the Torso Origin Min=0.9 Max=1.3 (TODO: make it a parameter at launch)  -->
-  <xacro:property name="base_height" value="1.0" />
+  <xacro:property name="base_height" value="1.2" />
   <!-- Parameters for the 3 bar base height -->
   <xacro:property name="back_bar_min_length" value="0.536" />

Commit message: minor cleanup

File: reachy_description/urdf/reachy.urdf.xacro (robot description, xacro)
@@ -97,11 +97,6 @@
 	       iyx="-0.00167148" iyy="0.4236827" iyz="0.00026596"
 	       izx="-0.00178789" izy="0.00026596" izz="0.70990763"/>
-    </inertial>
+  </inertial>
 </link>
-<!-- <joint name="base_link_joint" type="fixed"> -->
-<!-- 	<origin xyz="1 0 0" rpy="0 0 0"/> -->
-<!-- 	<parent link="world"/> -->
-<!-- 	<child link="base_link"/> -->
-<!-- </joint> -->
 <link name="back_bar">
 	<visual>

Commit message: base_footprint and base_link are now defined in zuuu_description

File: reachy_description/urdf/reachy.urdf.xacro (robot description, xacro)
@@ -68,35 +68,4 @@
     <child link="base_link" />
   </joint> -->
-<!-- Robot Footprint. The robot's root link -->
-<link name="base_footprint"/>
-<joint name="base_footprint_joint" type="fixed">
-  <origin rpy="0 0 0" xyz="0 0 0"/>
-  <axis xyz="0 0 0"/>
-  <!-- <joint_properties damping="${global_damping}" friction="${global_friction}"/> -->
-  <parent link="base_footprint"/>
-  <child link="base_link"/>
-</joint>
-<link name="base_link">
-	<visual>
-	  <origin xyz="0 0 0" rpy="0 0 0"/>
-	  <geometry>
-	    <mesh filename="file://$(find reachy_description)/meshes/mobile_base_visual.dae" />
-	  </geometry>
-	  <xacro:reachy_grey/>
-	</visual>
-	<collision>
-	  <origin xyz="0 0 0.13045" rpy="0 0 0"/>
-	  <geometry>
-	    <cylinder radius="0.245" length="0.2609"/>
-	  </geometry>
-	</collision>
-	<inertial>
-      <origin xyz="0.008 -0.00048 0.112" rpy="0 0 0"/>
-      <mass value="24.0"/>
-      <inertia ixx="0.40791094" ixy="-0.00167148" ixz="-0.00178789"
-	       iyx="-0.00167148" iyy="0.4236827" iyz="0.00026596"
-	       izx="-0.00178789" izy="0.00026596" izz="0.70990763"/>
-  </inertial>
-</link>
 <link name="back_bar">
 	<visual>
