Commit message: add configurable urdf

File: reachy_description/urdf/reachy.urdf.xacro (robot description, xacro)
@@ -9,17 +9,17 @@
   <xacro:include filename="$(find pollen_generic_description)/urdf/materials.urdf.xacro" />
   <!-- Zuuu mobile base -->
-  <xacro:arg name="zuuu_prefix" default=""/>
+  <xacro:arg name="zuuu_prefix" default="" />
   <xacro:arg name="model" default="zuuu" />
-  <xacro:arg name="use_fake_components" default="true"/>
-  <xacro:arg name="use_fixed_wheels" default="true"/>
-  <xacro:arg name="use_ros_control" default="true"/>
+  <xacro:arg name="use_fake_components" default="true" />
+  <xacro:arg name="use_fixed_wheels" default="true" />
+  <xacro:arg name="use_ros_control" default="true" />
   <!-- Import zuuu macro -->
-  <xacro:include filename="$(find zuuu_description)/urdf/zuuu_description.urdf.xacro"/>
+  <xacro:include filename="$(find zuuu_description)/urdf/zuuu_description.urdf.xacro" />
   <!-- Import Gazebo macro -->
-  <xacro:include filename="$(find zuuu_description)/urdf/zuuu.gazebo.xacro"/>
+  <xacro:include filename="$(find zuuu_description)/urdf/zuuu.gazebo.xacro" />
   <!-- Import Zuuu ros2_control description -->
-  <xacro:include filename="$(find zuuu_description)/urdf/zuuu.ros2_control.xacro"/>
+  <xacro:include filename="$(find zuuu_description)/urdf/zuuu.ros2_control.xacro" />
   <xacro:zuuu
-      model="$(arg model)" prefix="$(arg zuuu_prefix)">
+    model="$(arg model)" prefix="$(arg zuuu_prefix)">
   </xacro:zuuu>
   <xacro:if value="$(arg use_gazebo)">
@@ -27,5 +27,5 @@
   </xacro:if>
   <xacro:if value="$(arg use_ros_control)">
-    <xacro:zuuu_ros2_control model="$(arg model)" prefix="$(arg zuuu_prefix)"/>
+    <xacro:zuuu_ros2_control model="$(arg model)" prefix="$(arg zuuu_prefix)" />
   </xacro:if>
   <!-- End of Zuuu mobile base -->
@@ -34,4 +34,5 @@
   <xacro:arg name="right_arm_config" default="$(find arm_description)/config/fake_arm.yaml" />
   <xacro:arg name="left_arm_config" default="$(find arm_description)/config/fake_arm.yaml" />
+  <xacro:arg name="robot_model" default="none" />
   <!-- config  -->
   <!-- MODEL PARAMETERS -->
@@ -55,5 +56,6 @@
   <xacro:property name="right_bar_y" value="-0.117182" />
   <xacro:property name="back_bar_length" value="${base_height-0.2-back_bar_z}" />
-  <xacro:property name="front_bar_length" value="${sqrt(back_bar_length*back_bar_length+bar_small_triangle_base*bar_small_triangle_base)}" />
+  <xacro:property name="front_bar_length"
+    value="${sqrt(back_bar_length*back_bar_length+bar_small_triangle_base*bar_small_triangle_base)}" />
   <!-- <link name="world" /> -->
   <!-- <joint name="world_joint" type="fixed"> -->
@@ -68,90 +70,94 @@
     <child link="base_link" />
   </joint> -->
-<link name="back_bar">
-	<visual>
-	  <origin xyz="0 0 ${back_bar_length/2}" rpy="0 0 0"/>
-	  <geometry>
-	    <box size="0.04 0.04 ${back_bar_length}"/>
-	  </geometry>
-	  <xacro:reachy_grey/>
-	</visual>
-	<collision>
-	  <origin xyz="0 0 ${back_bar_length/2}" rpy="0 0 0"/>
-	  <geometry>
-	    <box size="0.04 0.04 ${back_bar_length}"/>
-	  </geometry>
-	</collision>
-</link>
-<link name="left_bar">
-	<visual>
-	  <origin xyz="0.0 0 ${front_bar_length/2}" rpy="0 0 0"/>
-	  <geometry>
-	    <box size="0.04 0.04 ${front_bar_length}"/>
-	  </geometry>
-	  <xacro:reachy_grey/>
-	</visual>
-	<collision>
-	  <origin xyz="0.0 0 ${front_bar_length/2}" rpy="0 0 0"/>
-	  <geometry>
-	    <box size="0.04 0.04 ${front_bar_length}"/>
-	  </geometry>
-	</collision>
-</link>
-<link name="right_bar">
-	<visual>
-	  <origin xyz="0.0 0 ${front_bar_length/2}" rpy="0 0 0"/>
-	  <geometry>
-	    <box size="0.04 0.04 ${front_bar_length}"/>
-	  </geometry>
-	  <xacro:reachy_grey/>
-	</visual>
-	<collision>
-	  <origin xyz="0.0 0 ${front_bar_length/2}" rpy="0 0 0"/>
-	  <geometry>
-	    <box size="0.04 0.04 ${front_bar_length}"/>
-	  </geometry>
-	</collision>
-</link>
-<joint name="back_bar_joint" type="fixed">
-	<!-- <origin xyz="-0.122 0 0.057" rpy="0 0 0"/> -->
-	<origin xyz="${back_bar_x} 0 ${back_bar_z}" rpy="0 0 0"/>
-	<parent link="base_link"/>
-	<child link="back_bar"/>
-</joint>
-<joint name="left_bar_joint" type="fixed">
-	<!-- <origin xyz="0.080966 0.11718 0.057" rpy="0 ${-pi/2+atan2(back_bar_length,bar_small_triangle_base)} ${bar_angle}"/> -->
-	<origin xyz="${left_bar_x} ${left_bar_y} ${back_bar_z}" rpy="0 ${-pi/2+atan2(back_bar_length,bar_small_triangle_base)} ${bar_angle}"/>
-	<parent link="base_link"/>
-	<child link="left_bar"/>
-</joint>
-<joint name="right_bar_joint" type="fixed">
-	<!-- <origin xyz="0.080966 -0.11718 0.057" rpy="0 ${-pi/2+atan2(back_bar_length,bar_small_triangle_base)} ${-bar_angle}"/> -->
-	<origin xyz="${right_bar_x} ${right_bar_y} ${back_bar_z}" rpy="0 ${-pi/2+atan2(back_bar_length,bar_small_triangle_base)} ${-bar_angle}"/>
-	<parent link="base_link"/>
-	<child link="right_bar"/>
-</joint>
+  <link name="back_bar">
+    <visual>
+      <origin xyz="0 0 ${back_bar_length/2}" rpy="0 0 0" />
+      <geometry>
+        <box size="0.04 0.04 ${back_bar_length}" />
+      </geometry>
+      <xacro:reachy_grey />
+    </visual>
+    <collision>
+      <origin xyz="0 0 ${back_bar_length/2}" rpy="0 0 0" />
+      <geometry>
+        <box size="0.04 0.04 ${back_bar_length}" />
+      </geometry>
+    </collision>
+  </link>
+  <link name="left_bar">
+    <visual>
+      <origin xyz="0.0 0 ${front_bar_length/2}" rpy="0 0 0" />
+      <geometry>
+        <box size="0.04 0.04 ${front_bar_length}" />
+      </geometry>
+      <xacro:reachy_grey />
+    </visual>
+    <collision>
+      <origin xyz="0.0 0 ${front_bar_length/2}" rpy="0 0 0" />
+      <geometry>
+        <box size="0.04 0.04 ${front_bar_length}" />
+      </geometry>
+    </collision>
+  </link>
+  <link name="right_bar">
+    <visual>
+      <origin xyz="0.0 0 ${front_bar_length/2}" rpy="0 0 0" />
+      <geometry>
+        <box size="0.04 0.04 ${front_bar_length}" />
+      </geometry>
+      <xacro:reachy_grey />
+    </visual>
+    <collision>
+      <origin xyz="0.0 0 ${front_bar_length/2}" rpy="0 0 0" />
+      <geometry>
+        <box size="0.04 0.04 ${front_bar_length}" />
+      </geometry>
+    </collision>
+  </link>
+  <joint name="back_bar_joint" type="fixed">
+    <!-- <origin xyz="-0.122 0 0.057" rpy="0 0 0"/> -->
+    <origin xyz="${back_bar_x} 0 ${back_bar_z}" rpy="0 0 0" />
+    <parent link="base_link" />
+    <child link="back_bar" />
+  </joint>
+  <joint name="left_bar_joint" type="fixed">
+    <!-- <origin xyz="0.080966 0.11718 0.057" rpy="0
+    ${-pi/2+atan2(back_bar_length,bar_small_triangle_base)} ${bar_angle}"/> -->
+    <origin xyz="${left_bar_x} ${left_bar_y} ${back_bar_z}"
+      rpy="0 ${-pi/2+atan2(back_bar_length,bar_small_triangle_base)} ${bar_angle}" />
+    <parent link="base_link" />
+    <child link="left_bar" />
+  </joint>
+  <joint name="right_bar_joint" type="fixed">
+    <!-- <origin xyz="0.080966 -0.11718 0.057" rpy="0
+    ${-pi/2+atan2(back_bar_length,bar_small_triangle_base)} ${-bar_angle}"/> -->
+    <origin xyz="${right_bar_x} ${right_bar_y} ${back_bar_z}"
+      rpy="0 ${-pi/2+atan2(back_bar_length,bar_small_triangle_base)} ${-bar_angle}" />
+    <parent link="base_link" />
+    <child link="right_bar" />
+  </joint>
   <!-- TORSO -->
   <link name="torso">
     <visual>
-      <origin xyz="0 0 0 " rpy="0 0 0"/>
-      <geometry>
-	<!-- <mesh filename="package://reachy_description/meshes/torso_visual_high.dae" /> -->
-	<mesh filename="file://$(find reachy_description)/meshes/torso_visual_high.dae" />
-	<!-- <mesh filename="file://$(find reachy_description)/meshes/torso_visual_high2.dae" /> -->
+      <origin xyz="0 0 0 " rpy="0 0 0" />
+      <geometry>
+        <!-- <mesh filename="package://reachy_description/meshes/torso_visual_high.dae" /> -->
+        <mesh filename="file://$(find reachy_description)/meshes/torso_visual_high.dae" />
+        <!-- <mesh filename="file://$(find reachy_description)/meshes/torso_visual_high2.dae" /> -->
       </geometry>
     </visual>
     <inertial>
       <!-- <origin xyz="-0.098614 -0.000471 -0.018363" rpy="0 0 0"/> -->
-      <origin xyz="-0.051614 -0.000471 -0.018363" rpy="0 0 0"/>
-      <mass value="6.314"/>
+      <origin xyz="-0.051614 -0.000471 -0.018363" rpy="0 0 0" />
+      <mass value="6.314" />
       <inertia ixx="0.07397673" ixy="-4.624e-4" ixz="-0.00175905"
-	       iyx="-0.00046237" iyy="0.04454533" iyz="0.00008675"
-	       izx="-0.00175905" izy="0.00008675" izz="0.05494939"/>
+        iyx="-0.00046237" iyy="0.04454533" iyz="0.00008675"
+        izx="-0.00175905" izy="0.00008675" izz="0.05494939" />
     </inertial>
     <collision>
-      <origin xyz="0 0 0 " rpy="0 0 0"/>
-      <geometry>
-	<!-- <mesh filename="package://reachy_description/meshes/torso_collider_no_cone.dae" /> -->
-	<mesh filename="file://$(find reachy_description)/meshes/torso_collider_no_cone.dae" />
+      <origin xyz="0 0 0 " rpy="0 0 0" />
+      <geometry>
+        <!-- <mesh filename="package://reachy_description/meshes/torso_collider_no_cone.dae" /> -->
+        <mesh filename="file://$(find reachy_description)/meshes/torso_collider_no_cone.dae" />
       </geometry>
     </collision>
@@ -163,9 +169,9 @@
   </joint>
   <link name="logo">
-            <inertial>
-                <origin xyz="0.0 0.0 0.0" rpy="0.0 0.0 0.0"/>
-                <mass value="0.001"/>
-                <inertia ixx="1.0e-6" ixy="1.0e-8" ixz="1.0e-8" iyy="1.0e-6" iyz="1.0e-8" izz="1.0e-6"/>
-            </inertial>
+    <inertial>
+      <origin xyz="0.0 0.0 0.0" rpy="0.0 0.0 0.0" />
+      <mass value="0.001" />
+      <inertia ixx="1.0e-6" ixy="1.0e-8" ixz="1.0e-8" iyy="1.0e-6" iyz="1.0e-8" izz="1.0e-6" />
+    </inertial>
   </link>
   <joint name="logo_joint" type="fixed">
@@ -189,4 +195,5 @@
     damping="${damping}" friction="${friction}"
     config_file="$(arg right_arm_config)"
+    robot_model="$(arg robot_model)"
   />
   <!-- LEFT ARM -->
@@ -195,207 +202,208 @@
     damping="${damping}" friction="${friction}"
     config_file="$(arg left_arm_config)"
+    robot_model="$(arg robot_model)"
   />
   <link name="depth_cam_l_optical">
     <inertial>
-      <origin xyz="0.0 0.0 0.0" rpy="0.0 0.0 0.0"/>
-      <mass value="0.001"/>
-                <inertia ixx="1.0e-6" ixy="1.0e-8" ixz="1.0e-8" iyy="1.0e-6" iyz="1.0e-8" izz="1.0e-6"/>
+      <origin xyz="0.0 0.0 0.0" rpy="0.0 0.0 0.0" />
+      <mass value="0.001" />
+      <inertia ixx="1.0e-6" ixy="1.0e-8" ixz="1.0e-8" iyy="1.0e-6" iyz="1.0e-8" izz="1.0e-6" />
     </inertial>
   </link>
   <link name="depth_cam_l_frame">
     <inertial>
-      <origin xyz="0.0 0.0 0.0" rpy="0.0 0.0 0.0"/>
-      <mass value="0.001"/>
-                <inertia ixx="1.0e-6" ixy="1.0e-8" ixz="1.0e-8" iyy="1.0e-6" iyz="1.0e-8" izz="1.0e-6"/>
+      <origin xyz="0.0 0.0 0.0" rpy="0.0 0.0 0.0" />
+      <mass value="0.001" />
+      <inertia ixx="1.0e-6" ixy="1.0e-8" ixz="1.0e-8" iyy="1.0e-6" iyz="1.0e-8" izz="1.0e-6" />
     </inertial>
   </link>
   <joint name="depth_cam_l_optical_joint" type="fixed">
-    <origin xyz="0.002597 0.009989 0.038089" rpy="${radians(-48.0-90.0)} 0.0 ${-pi/2}"/>
-    <parent link="logo"/>
-    <child link="depth_cam_l_optical"/>
+    <origin xyz="0.002597 0.009989 0.038089" rpy="${radians(-48.0-90.0)} 0.0 ${-pi/2}" />
+    <parent link="logo" />
+    <child link="depth_cam_l_optical" />
   </joint>
   <joint name="depth_cam_l_frame_joint" type="fixed">
-    <origin xyz="0.002597 0.009989 0.038089" rpy="0.0 ${radians(48.0)} 0.0"/>
-    <parent link="logo"/>
-    <child link="depth_cam_l_frame"/>
+    <origin xyz="0.002597 0.009989 0.038089" rpy="0.0 ${radians(48.0)} 0.0" />
+    <parent link="logo" />
+    <child link="depth_cam_l_frame" />
   </joint>
   <link name="depth_cam_r_optical">
-            <inertial>
-                <origin xyz="0.0 0.0 0.0" rpy="0.0 0.0 0.0"/>
-                <mass value="0.001"/>
-                <inertia ixx="1.0e-6" ixy="1.0e-8" ixz="1.0e-8" iyy="1.0e-6" iyz="1.0e-8" izz="1.0e-6"/>
-            </inertial>
+    <inertial>
+      <origin xyz="0.0 0.0 0.0" rpy="0.0 0.0 0.0" />
+      <mass value="0.001" />
+      <inertia ixx="1.0e-6" ixy="1.0e-8" ixz="1.0e-8" iyy="1.0e-6" iyz="1.0e-8" izz="1.0e-6" />
+    </inertial>
   </link>
   <link name="depth_cam_r_frame">
-            <inertial>
-                <origin xyz="0.0 0.0 0.0" rpy="0.0 0.0 0.0"/>
-                <mass value="0.001"/>
-                <inertia ixx="1.0e-6" ixy="1.0e-8" ixz="1.0e-8" iyy="1.0e-6" iyz="1.0e-8" izz="1.0e-6"/>
-            </inertial>
+    <inertial>
+      <origin xyz="0.0 0.0 0.0" rpy="0.0 0.0 0.0" />
+      <mass value="0.001" />
+      <inertia ixx="1.0e-6" ixy="1.0e-8" ixz="1.0e-8" iyy="1.0e-6" iyz="1.0e-8" izz="1.0e-6" />
+    </inertial>
   </link>
   <joint name="depth_cam_r_optical_joint" type="fixed">
-    <origin xyz="0.002597 -0.009989 0.038089" rpy="${radians(-48.0-90.0)} 0.0 ${-pi/2}"/>
-    <parent link="logo"/>
-    <child link="depth_cam_r_optical"/>
+    <origin xyz="0.002597 -0.009989 0.038089" rpy="${radians(-48.0-90.0)} 0.0 ${-pi/2}" />
+    <parent link="logo" />
+    <child link="depth_cam_r_optical" />
   </joint>
   <joint name="depth_cam_r_frame_joint" type="fixed">
-    <origin xyz="0.002597 -0.009989 0.038089" rpy="0.0 ${radians(48.0)} 0.0 "/>
-    <parent link="logo"/>
-    <child link="depth_cam_r_frame"/>
-  </joint>
-      <gazebo reference="depth_cam_l_frame">
-	<!-- <link name="left_camera"> -->
-	<sensor type="camera" name="left_camera">
-          <!-- Set always_on only sensor, not on plugin -->
-          <always_on>0</always_on>
-          <!-- Set update_rate only sensor, not on plugin -->
-          <update_rate>30</update_rate>
-          <camera name="depth_cam_l">
-            <horizontal_fov>${90.0*pi/180}</horizontal_fov>
-            <image>
-              <width>1280</width>
-              <height>800</height>
-              <format>B8G8R8</format>
-            </image>
-            <distortion>
-              <k1>0.006059</k1>
-              <k2>-0.048786</k2>
-              <k3>0.033282</k3>
-              <p1>-0.000877</p1>
-              <p2>-0.000732</p2>
-              <center>0.5 0.5</center>
-            </distortion>
-            <noise>
-              <type>gaussian</type>
-              <mean>0.0</mean>
-              <stddev>0.007</stddev>
-            </noise>
-          </camera>
-          <!-- Use camera, not camera_triggered -->
-          <plugin name="depth_left_camera_controller" filename="libgazebo_ros_camera.so">
-              <ros>
-                <namespace>camera</namespace>
-                <remapping>left/image_raw:=/camera/left/color/image_raw</remapping>
-                <remapping>left/image_raw/compressed:=/camera/left/color/image_raw/compressed</remapping>
-                <remapping>left/camera_info:=/camera/left/color/camera_info</remapping>
-              </ros>
-              <camera_name>left</camera_name>
-            <!-- <ros> -->
-            <!--   <namespace>custom_ns</namespace> -->
-            <!--   <argument>image_raw:=custom_img</argument> -->
-            <!--   <argument>camera_info:=custom_info</argument> -->
-            <!-- </ros> -->
-            <!-- Set camera name. If empty, defaults to sensor name (i.e. "sensor_name") -->
-            <!-- <camera_name>left_camera</camera_name> -->
-            <!-- Set TF frame name. If empty, defaults to link name (i.e. "link_name") -->
-            <frame_name>depth_cam_l_optical</frame_name>
-            <hack_baseline>0.07</hack_baseline>
-            <!-- No need to repeat distortion parameters or to set autoDistortion -->
-          </plugin>
-        </sensor>
-      </gazebo>
-      <gazebo reference="depth_cam_r_frame">
-	<!-- <link name="left_camera"> -->
-	<sensor type="camera" name="right_camera">
-          <!-- Set always_on only sensor, not on plugin -->
-          <always_on>0</always_on>
-          <!-- Set update_rate only sensor, not on plugin -->
-          <update_rate>30</update_rate>
-          <camera name="depth_cam_r">
-            <horizontal_fov>${90.0*pi/180}</horizontal_fov>
-            <image>
-              <width>1280</width>
-              <height>800</height>
-              <format>B8G8R8</format>
-            </image>
-            <distortion>
-              <k1>0.006059</k1>
-              <k2>-0.048786</k2>
-              <k3>0.033282</k3>
-              <p1>-0.000877</p1>
-              <p2>-0.000732</p2>
-              <center>0.5 0.5</center>
-            </distortion>
-            <noise>
-              <type>gaussian</type>
-              <mean>0.0</mean>
-              <stddev>0.007</stddev>
-            </noise>
-          </camera>
-          <!-- Use camera, not camera_triggered -->
-          <plugin name="depth_right_camera_controller" filename="libgazebo_ros_camera.so">
-              <ros>
-                <namespace>camera</namespace>
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
Commit message: update mesh

File: reachy_description/urdf/reachy.urdf.xacro (robot description, xacro)
@@ -143,5 +143,5 @@
       <geometry>
         <!-- <mesh filename="package://reachy_description/meshes/torso_visual_high.dae" /> -->
-        <mesh filename="file://$(find reachy_description)/meshes/torso_visual_high.dae" />
+        <mesh filename="file://$(find reachy_description)/meshes/torso_visual.dae" />
         <!-- <mesh filename="file://$(find reachy_description)/meshes/torso_visual_high2.dae" /> -->
       </geometry>
@@ -159,5 +159,5 @@
       <geometry>
         <!-- <mesh filename="package://reachy_description/meshes/torso_collider_no_cone.dae" /> -->
-        <mesh filename="file://$(find reachy_description)/meshes/torso_collider_no_cone.dae" />
+        <mesh filename="file://$(find reachy_description)/meshes/torso_collider.dae" />
       </geometry>
     </collision>
