Commit message: wip

File: reachy_description/urdf/reachy.urdf.xacro (robot description, xacro)
@@ -1 +1,790 @@
-reachy.urdf.xacro.test
+<?xml version="1.0"?>
+<robot xmlns:xacro="http://www.ros.org/wiki/xacro" name="reachy2">
+  <xacro:arg name="use_fake_hardware" default="false" />
+  <xacro:arg name="use_gazebo" default="false" />
+  <xacro:arg name="use_moveit_gazebo" default="false" />
+  <xacro:include filename="$(find reachy_description)/urdf/head.urdf.xacro" />
+  <xacro:include filename="$(find reachy_description)/urdf/arm.urdf.xacro" />
+  <xacro:include filename="$(find dynamixel_description)/urdf/dynamixel_gripper.urdf.xacro" />
+  <xacro:include filename="$(find dynamixel_description)/ros2_control/dynamixel_gripper.ros2_control.xacro" />
+  <xacro:include filename="$(find pollen_generic_description)/urdf/inertial_primitives.urdf.xacro" />
+  <xacro:include filename="$(find pollen_generic_description)/urdf/materials.urdf.xacro" />
+  <xacro:include filename="$(find reachy_description)/urdf/gz_mimic.urdf.xacro" />
+  <!-- Zuuu mobile base -->
+  <xacro:arg name="zuuu_prefix" default="" />
+  <xacro:arg name="model" default="zuuu" />
+  <xacro:arg name="use_fake_components" default="true" />
+  <xacro:arg name="use_fixed_wheels" default="true" />
+  <xacro:arg name="use_ros_control" default="true" />
+  <!-- Import zuuu macro -->
+  <xacro:include filename="$(find zuuu_description)/urdf/zuuu_description.urdf.xacro" />
+  <!-- Import Gazebo macro -->
+  <xacro:include filename="$(find zuuu_description)/urdf/zuuu.gazebo.xacro" />
+  <!-- Import Zuuu ros2_control description -->
+  <xacro:include filename="$(find zuuu_description)/urdf/zuuu.ros2_control.xacro" />
+  <xacro:zuuu
+    model="$(arg model)" prefix="$(arg zuuu_prefix)">
+  </xacro:zuuu>
+  <xacro:if value="$(arg use_gazebo)">
+    <xacro:zuuu_gazebo model="$(arg model)" prefix="$(arg zuuu_prefix)" />
+  </xacro:if>
+  <xacro:if value="$(arg use_ros_control)">
+    <xacro:zuuu_ros2_control model="$(arg model)" prefix="$(arg zuuu_prefix)" />
+  </xacro:if>
+  <!-- End of Zuuu mobile base -->
+  <!-- config  -->
+  <xacro:arg name="antenna_config" default="$(find dynamixel_description)/config/two_fake.yaml"/>
+  <xacro:arg name="neck_config" default="$(find orbita3d_description)/config/fake_neck.yaml" />
+  <xacro:arg name="right_shoulder_config" default="$(find orbita2d_description)/config/fake.yaml" />
+  <xacro:arg name="right_elbow_config" default="$(find orbita2d_description)/config/fake.yaml" />
+  <xacro:arg name="right_wrist_config" default="$(find orbita3d_description)/config/fake.yaml" />
+  <xacro:arg name="left_shoulder_config" default="$(find orbita2d_description)/config/fake.yaml" />
+  <xacro:arg name="left_elbow_config" default="$(find orbita2d_description)/config/fake.yaml" />
+  <xacro:arg name="left_wrist_config" default="$(find orbita3d_description)/config/fake.yaml" />
+  <!-- <xacro:arg name="right_arm_config" default="$(find arm_description)/config/fake_r_arm.yaml" /> -->
+  <!-- <xacro:arg name="left_arm_config" default="$(find arm_description)/config/fake_l_arm.yaml" /> -->
+  <xacro:arg name="grippers_config" default="$(find dynamixel_description)/config/two_fake.yaml"/>
+  <xacro:arg name="robot_model" default="none" />
+  <xacro:arg name="robot_config" default="full_kit" />
+  <!-- all the robot configurations -->
+  <xacro:property name="mobile_base" value="false" />
+  <xacro:property name="left_arm" value="false" />
+  <xacro:property name="right_arm" value="false" />
+  <xacro:property name="left_gripper" value="false" />
+  <xacro:property name="right_gripper" value="false" />
+  <!-- <xacro:property name="config" value="$(arg robot_config)" /> -->
+  <xacro:property name="config" value="full_kit" />
+  <xacro:if value="${config == 'full_kit'}">
+      <xacro:property name="mobile_base" value="true" />
+      <xacro:property name="left_arm" value="true" />
+      <xacro:property name="left_gripper" value="true" />
+      <xacro:property name="right_arm" value="true" />
+      <xacro:property name="right_gripper" value="true" />
+  </xacro:if>
+  <xacro:if value="${config == 'full_kit_no_gripper'}">
+      <xacro:property name="mobile_base" value="true" />
+      <xacro:property name="left_arm" value="true" />
+      <xacro:property name="right_arm" value="true" />
+  </xacro:if>
+  <xacro:if value="${config == 'left_arm'}">
+      <xacro:property name="mobile_base" value="true" />
+      <xacro:property name="left_arm" value="true" />
+      <xacro:property name="left_gripper" value="true" />
+  </xacro:if>
+  <xacro:if value="${config == 'right_arm'}">
+      <xacro:property name="mobile_base" value="true" />
+      <xacro:property name="right_arm" value="true" />
+      <xacro:property name="right_gripper" value="true" />
+  </xacro:if>
+  <xacro:if value="${config == 'left_arm_no_gripper'}">
+      <xacro:property name="mobile_base" value="true" />
+      <xacro:property name="left_arm" value="true" />
+  </xacro:if>
+  <xacro:if value="${config == 'right_arm_no_gripper'}">
+      <xacro:property name="mobile_base" value="true" />
+      <xacro:property name="right_arm" value="true" />
+  </xacro:if>
+  <!-- config  -->
+  <!-- MODEL PARAMETERS -->
+  <xacro:property name="base_collision" value="true" />
+  <xacro:property name="base_visual" value="true" />
+  <xacro:property name="damping" value="0.01" />
+  <xacro:property name="friction" value="0.1" />
+  <!-- Base height (torso) = 1000mm when back bar joint=525mm -->
+  <!-- Parameters for the 3 bar base height -->
+  <xacro:property name="back_bar_min_length" value="0.520" />
+  <xacro:property name="back_bar_max_length" value="${back_bar_min_length+0.210}" />
+  <!-- <xacro:property name="bar_angle" value="${radians(27.458)}" /> -->
+  <xacro:property name="bar_angle" value="${radians(10.937)}" />
+  <xacro:property name="bar_angle_offset" value="${pi/2-atan2(back_bar_min_length-0.03-0.018,bar_small_triangle_base-0.09)}" />
+  <xacro:property name="bar_small_triangle_base" value="0.186" />
+  <xacro:property name="back_bar_z" value="0.241" />
+  <xacro:property name="back_bar_x" value="-0.09" />
+  <xacro:property name="left_bar_x" value="0.084" />
+  <xacro:property name="left_bar_y" value="0.066" />
+  <xacro:property name="right_bar_x" value="0.084" />
+  <xacro:property name="right_bar_y" value="-0.066" />
+  <xacro:property name="right_bar_anchor" value="0.03" />
+  <!-- <xacro:property name="back_bar_length" value="${base_height-0.2-back_bar_z}" /> -->
+  <xacro:property name="back_bar_length" value="0.485" />
+  <!-- TODO: replace by primitives -->
+    <xacro:macro name="box_inertia" params="m w h d">
+      <inertial>
+        <origin xyz="0 0 0" rpy="${pi/2} 0 ${pi/2}" />
+        <mass value="${m}" />
+        <inertia ixx="${(m/12) * (h*h + d*d)}" ixy="0.0" ixz="0.0" iyy="${(m/12) * (w*w + d*d)}"
+          iyz="0.0" izz="${(m/12) * (w*w + h*h)}" />
+      </inertial>
+    </xacro:macro>
+  <link name="back_bar_base">
+   <visual>
+      <origin xyz="0 0 ${back_bar_length/2}" rpy="0 0 0" />
+      <geometry>
+        <box size="0.04 0.04 ${back_bar_length}" />
+      </geometry>
+      <xacro:reachy_grey />
+    </visual>
+    <collision>
+      <origin xyz="0 0 ${back_bar_length/2}" rpy="0 0 0" />
+      <geometry>
+        <box size="0.05 0.05 ${back_bar_length}" />
+      </geometry>
+    </collision>
+    <xacro:box_inertia m="0.759" w="0.04" h="0.04" d="0.04"/>
+  </link>
+  <joint name="back_bar_joint" type="fixed">
+    <origin xyz="${back_bar_x} 0 ${back_bar_z}" rpy="0 0 0" />
+    <parent link="base_link" />
+    <child link="back_bar_base" />
+  </joint>
+  <link name="back_bar_inner">
+   <visual>
+      <origin xyz="0 0 ${back_bar_length/2}" rpy="0 0 0" />
+      <geometry>
+        <box size="0.03 0.03 ${back_bar_length}" />
+      </geometry>
+      <xacro:reachy_grey />
+    </visual>
+    <collision>
+      <origin xyz="0 0 ${back_bar_length/2}" rpy="0 0 0" />
+      <geometry>
+        <box size="0.05 0.05 ${back_bar_length}" />
+      </geometry>
+    </collision>
+    <xacro:box_inertia m="0.759" w="0.04" h="0.04" d="0.04"/>
+  </link>
+  <joint name="tripod_joint" type="prismatic">
+    <origin xyz="0 0 0.035" rpy="0 0 0" />
+    <parent link="back_bar_base" />
+    <child link="back_bar_inner" />
+    <limit effort="1.0" lower="0.0" upper="0.210" velocity="0.1"/>
+    <axis xyz="0 0 1"/>
+    <dynamics damping="${damping}" friction="${friction}"/>
+  </joint>
+<link name="left_bar_base">
+   <visual>
+      <origin xyz="0 0 ${-back_bar_length/2}" rpy="0 0 0" />
+      <!-- <origin xyz="0 0 0" rpy="0 0 0" /> -->
+      <geometry>
+        <box size="0.04 0.04 ${back_bar_length}" />
+      </geometry>
+      <xacro:reachy_grey />
+    </visual>
+    <collision>
+      <origin xyz="0 0 ${-back_bar_length/2}" rpy="0 0 0" />
+      <geometry>
+        <box size="0.05 0.05 ${back_bar_length}" />
+      </geometry>
+    </collision>
+    <xacro:box_inertia m="1.759" w="0.04" h="0.04" d="0.04"/>
+</link>
+<link name="left_bar_anchor">
+   <visual>
+      <origin xyz="0 0 ${right_bar_anchor/2}" rpy="0 0 ${bar_angle}" />
+      <geometry>
+        <box size="0.03 0.03 ${right_bar_anchor}" />
+      </geometry>
+      <xacro:reachy_grey />
+    </visual>
+    <collision>
+      <origin xyz="0 0 ${right_bar_anchor/2}" rpy="0 0 ${bar_angle}" />
+      <geometry>
+        <box size="0.03 0.03 ${right_bar_anchor}" />
+      </geometry>
+    </collision>
+    <xacro:box_inertia m="1.759" w="0.03" h="0.03" d="0.03"/>
+</link>
+<joint name="left_bar_anchor_to_base" type="fixed">
+    <origin xyz="${left_bar_x} ${left_bar_y} ${back_bar_z}" rpy="0 0 0" />
+    <parent link="base_link" />
+    <child link="left_bar_anchor" />
+</joint>
+  <joint name="left_bar_joint_mimic" type="revolute">
+    <origin xyz="0 0.048 -0.258" rpy="0 0 ${bar_angle}" />
+    <parent link="torso" />
+    <child link="left_bar_inner" />
+    <limit effort="0.01" lower="-1.0" upper="1.0" velocity="0.01"/>
+    <axis xyz="0 1 0"/>
+    <mimic joint="tripod_joint" multiplier="0.2864183599287582" offset="-0.1967146343049915" />
+    <!-- <mimic joint="tripod_joint" multiplier="0" offset="0" /> -->
+    <dynamics damping="${damping}" friction="${friction}"/>
+  </joint>
+  <link name="left_bar_inner">
+   <visual>
+      <origin xyz="0 0 ${-back_bar_length/2}" rpy="0 0 0" />
+      <geometry>
+        <box size="0.03 0.03 ${back_bar_length}" />
+      </geometry>
+      <xacro:reachy_grey />
+    </visual>
+    <collision>
+      <origin xyz="0 0 ${-back_bar_length/2}" rpy="0 0 0" />
+      <geometry>
+        <box size="0.05 0.05 ${back_bar_length}" />
+      </geometry>
+    </collision>
+    <xacro:box_inertia m="0.759" w="0.04" h="0.04" d="0.04"/>
+  </link>
+  <joint name="left_bar_prism_joint_mimic" type="prismatic">
+    <origin xyz="0 0 ${-back_bar_length}" rpy="0 0 0" />
+    <parent link="left_bar_inner" />
+    <child link="left_bar_base" />
+    <limit effort="1.0" lower="-1.0" upper="1.0" velocity="0.5"/>
+    <axis xyz="0 0 1"/>
+    <mimic joint="tripod_joint" multiplier="-0.9861535348976198" offset="0.4814718126556904" />
+    <dynamics damping="${damping}" friction="${friction}"/>
+  </joint>
+  <!-- right bar -->
+<link name="right_bar_base">
+   <visual>
+      <origin xyz="0 0 ${-back_bar_length/2}" rpy="0 0 0" />
+      <!-- <origin xyz="0 0 0" rpy="0 0 0" /> -->
+      <geometry>
+        <box size="0.04 0.04 ${back_bar_length}" />
+      </geometry>
+      <xacro:reachy_grey />
+    </visual>
+    <collision>
+      <origin xyz="0 0 ${-back_bar_length/2}" rpy="0 0 0" />
+      <geometry>
+        <box size="0.05 0.05 ${back_bar_length}" />
+      </geometry>
+    </collision>
+    <!-- <xacro:box_inertia m="1.759" w="0.04" h="0.04" d="0.04"/> -->
+    <xacro:box_inertia m="1.759" w="0.04" h="0.04" d="0.04"/>
+</link>
+<link name="right_bar_anchor">
+   <visual>
+      <origin xyz="0 0 ${right_bar_anchor/2}" rpy="0 0 ${-bar_angle}" />
+      <geometry>
+        <box size="0.03 0.03 ${right_bar_anchor}" />
+      </geometry>
+      <xacro:reachy_grey />
+    </visual>
+    <collision>
+      <origin xyz="0 0 ${right_bar_anchor/2}" rpy="0 0 ${-bar_angle}" />
+      <geometry>
+        <box size="0.03 0.03 ${right_bar_anchor}" />
+      </geometry>
+    </collision>
+    <xacro:box_inertia m="1.759" w="0.03" h="0.03" d="0.03"/>
+</link>
+<joint name="right_bar_anchor_to_base" type="fixed">
+    <origin xyz="${right_bar_x} ${right_bar_y} ${back_bar_z}" rpy="0 0 0" />
+    <parent link="base_link" />
+    <child link="right_bar_anchor" />
+</joint>
+  <joint name="right_bar_joint_mimic" type="revolute">
+    <origin xyz="0 -0.048 -0.258" rpy="0 0 ${-bar_angle}" />
+    <parent link="torso" />
+    <child link="right_bar_inner" />
+    <limit effort="0.01" lower="-1.0" upper="1.0" velocity="0.01"/>
+    <axis xyz="0 1 0"/>
+    <mimic joint="tripod_joint" multiplier="0.2864183599287582" offset="-0.1967146343049915" />
+    <!-- <mimic joint="tripod_joint" multiplier="0" offset="0" /> -->
+    <dynamics damping="${damping}" friction="${friction}"/>
+  </joint>
+  <link name="right_bar_inner">
+   <visual>
+      <origin xyz="0 0 ${-back_bar_length/2}" rpy="0 0 0" />
+      <geometry>
+        <box size="0.03 0.03 ${back_bar_length}" />
+      </geometry>
+      <xacro:reachy_grey />
+    </visual>
+    <collision>
+      <origin xyz="0 0 ${-back_bar_length/2}" rpy="0 0 0" />
+      <geometry>
+        <box size="0.05 0.05 ${back_bar_length}" />
+      </geometry>
+    </collision>
+    <xacro:box_inertia m="0.759" w="0.04" h="0.04" d="0.04"/>
+  </link>
+  <joint name="right_bar_prism_joint_mimic" type="prismatic">
+    <origin xyz="0 0 ${-back_bar_length}" rpy="0 0 0" />
+    <parent link="right_bar_inner" />
+    <child link="right_bar_base" />
+    <limit effort="1.0" lower="-1.0" upper="1.0" velocity="0.5"/>
+    <axis xyz="0 0 1"/>
+    <mimic joint="tripod_joint" multiplier="-0.9861535348976198" offset="0.4814718126556904" />
+    <dynamics damping="${damping}" friction="${friction}"/>
+  </joint>
+<xacro:if value="$(arg use_gazebo)">
+      <!-- 3rd order poly fit (pretty good): -0.82037152*x**3 + 0.74428024*x**2 -0.40967047*x + 0.20061291 -->
+  <!-- <xacro:mimic_joint_plugin_gazebo name_prefix="tripod_left_rev" following_joint="tripod_joint" mimic_joint="left_bar_joint_mimic" multiplier="0.2864183599287582" offset="-0.1967146343049915"/> -->
+  <xacro:mimic_joint_plugin_gazebo name_prefix="tripod_left_rev" following_joint="tripod_joint" mimic_joint="left_bar_joint_mimic" multiplier="0.40967047" offset="-0.20061291" k2="-0.74428024," k3="0.82037152"/>
+  <xacro:mimic_joint_plugin_gazebo name_prefix="tripod_left_prism" following_joint="tripod_joint" mimic_joint="left_bar_prism_joint_mimic" multiplier="-0.9861535348976198" offset="0.4814718126556904"/>
+  <!-- <xacro:mimic_joint_plugin_gazebo name_prefix="tripod_right_rev" following_joint="tripod_joint" mimic_joint="right_bar_joint_mimic" multiplier="0.2864183599287582" offset="-0.1967146343049915"/> -->
+  <xacro:mimic_joint_plugin_gazebo name_prefix="tripod_right_rev" following_joint="tripod_joint" mimic_joint="right_bar_joint_mimic" multiplier="0.40967047" offset="-0.20061291" k2="-0.74428024," k3="0.82037152"/>
+  <xacro:mimic_joint_plugin_gazebo name_prefix="tripod_right_prism" following_joint="tripod_joint" mimic_joint="right_bar_prism_joint_mimic" multiplier="-0.9861535348976198" offset="0.4814718126556904"/>
+</xacro:if>
+  <ros2_control name="tripod" type="system">
+    <hardware>
+      <!-- Use gazebo as hardware simulation. -->
+      <xacro:if value="$(arg use_gazebo)">
+        <plugin>gazebo_ros2_control/GazeboSystem</plugin>
+      </xacro:if>
+      <!-- Use fake components. -->
+      <xacro:unless value="$(arg use_gazebo)">
+        <plugin>fake_components/GenericSystem</plugin>
+      </xacro:unless>
+    </hardware>
+    <joint name="tripod_joint">
+      <state_interface name="position">
+        <param name="initial_value">0.0</param>
+      </state_interface>
+      <state_interface name="velocity">
+        <param name="initial_value">0.0</param>
+      </state_interface>
+      <state_interface name="effort">
+        <param name="initial_value">0.0</param>
+      </state_interface>
+      <!-- <command_interface name="position"> -->
+      <!--   <param name="min">0.0</param> -->
+      <!--   <param name="max">0.21</param> -->
+      <!-- </command_interface> -->
+      <command_interface name="position"/>
+    </joint>
+      <xacro:if value="$(arg use_gazebo)">
+        <joint name="left_bar_joint_mimic">
+          <!-- <param name="mimic">tripod_joint</param> -->
+          <!-- <param name="multiplier">0.2864183599287582</param> -->
+          <command_interface name="position"/>
+          <state_interface name="position"/>
+          <state_interface name="velocity"/>
+          <state_interface name="effort"/>
+        </joint>
+        <joint name="left_bar_prism_joint_mimic">
+          <!-- <param name="mimic">tripod_joint</param> -->
+          <!-- <param name="multiplier">0.9861535348976198</param> -->
+          <command_interface name="position"/>
+          <state_interface name="position"/>
+          <state_interface name="velocity"/>
+          <state_interface name="effort"/>
+        </joint>
+        <joint name="right_bar_joint_mimic">
+          <!-- <param name="mimic">tripod_joint</param> -->
+          <!-- <param name="multiplier">0.2864183599287582</param> -->
+          <command_interface name="position"/>
+          <state_interface name="position"/>
+          <state_interface name="velocity"/>
+          <state_interface name="effort"/>
+        </joint>
+        <joint name="right_bar_prism_joint_mimic">
+          <!-- <param name="mimic">tripod_joint</param> -->
+          <!-- <param name="multiplier">0.9861535348976198</param> -->
+          <command_interface name="position"/>
+          <state_interface name="position"/>
+          <state_interface name="velocity"/>
+          <state_interface name="effort"/>
+        </joint>
+      </xacro:if>
+  </ros2_control>
+  <!-- TORSO -->
+  <link name="torso">
+    <visual>
+      <origin xyz="0 0 0 " rpy="0 0 0" />
+      <geometry>
+        <!-- <mesh filename="file://$(find reachy_description)/meshes/torso_visual_high.dae" /> -->
+        <mesh filename="file://$(find reachy_description)/meshes/torso_visual.dae" />
+      </geometry>
+    </visual>
+    <inertial>
+      <!-- <origin xyz="-0.098614 -0.000471 -0.018363" rpy="0 0 0"/> -->
+      <origin xyz="-0.051614 -0.000471 -0.018363" rpy="0 0 0" />
+      <mass value="6.314" />
+      <inertia ixx="0.07397673" ixy="-4.624e-4" ixz="-0.00175905"
+        iyx="-0.00046237" iyy="0.04454533" iyz="0.00008675"
+        izx="-0.00175905" izy="0.00008675" izz="0.05494939" />
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