Commit message: tune head urdf

File: reachy_description/urdf/head.urdf.xacro (robot description, xacro)
@@ -6,4 +6,10 @@
   <xacro:property name="neck_orbita_reduction" value="4.266667"/>
   <xacro:property name="neck_orbita_alpha" value="0.9424777960769379"/>
+    <material name="camblack">
+        <color rgba="0.2 0.2 0.2 1"/>
+    </material>
+    <material name="neckwhite">
+        <color rgba="0.9 0.9 0.9 1"/>
+    </material>
   <xacro:macro name="head" params="parent damping friction neck_orbita_serial_port neck_orbita_id neck_orbita_hardware_zero">
     <xacro:include filename="$(find reachy_description)/ros2_control/head.ros2_control.xacro"/>
@@ -139,21 +145,37 @@
       </inertial>
       <visual name="">
-        <origin xyz="0.0 0.0 0.0" rpy="0.0 0.0 0.0"/>
+        <origin xyz="0.0075 0.0 0.085" rpy="0.0 0.0 0.0"/>
         <geometry>
-          <mesh filename="file://$(find reachy_description)/meshes/head.dae"/>
+          <!-- <mesh filename="file://$(find reachy_description)/meshes/head.dae"/> -->
+	  <box size="0.015 0.1245 0.0265"/>
         </geometry>
+	<material name="camblack"/>
       </visual>
       <collision>
-        <origin xyz="-0.009 -0.002 0.059" rpy="1.57 0.0 0.0"/>
+	<origin xyz="0.0075 0.0 0.085" rpy="0.0 0.0 0.0"/>
         <geometry>
-          <cylinder length="0.15" radius="0.06" />
+	  <box size="0.015 0.1245 0.0265"/>
         </geometry>
       </collision>
     </link>
+    <link name="head_base">
+      <visual name="">
+        <origin xyz="0.00 0.0 0.0425" rpy="0.0 0.0 0.0"/>
+        <geometry>
+	  <cylinder length="0.07" radius="0.0225"/>
+        </geometry>
+	<material name="neckwhite"/>
+      </visual>
+    </link>
+    <joint name="head_base_fixed" type="fixed">
+      <origin xyz="0.0 0 0.0" rpy="0.0 0.0 0"/>
+      <parent link="head" />
+      <child link="head_base" />
+    </joint>
     <link name="head_tip" >
     </link>
     <joint name="head_tip_fixed" type="fixed">
       <!-- between the cameras -->
-      <origin xyz="0.02 0 0.06105" rpy="0.0 0.0 0"/>
+      <origin xyz="0.015 0 0.085" rpy="0.0 0.0 0"/>
       <!-- Rotation center -->
       <!-- <origin xyz="0.0 0 0.0" rpy="0.0 0.0 0"/> -->
@@ -230,249 +252,210 @@
     orbita_reduction="${neck_orbita_reduction}"
   /> -->
-    <!-- Cameras -->
-    <xacro:if value="$(arg use_gazebo)">
-      <joint name="left_cam_fixed" type="fixed">
-	<origin xyz="0.02 0.03625 0.06105" rpy="0.0 0.0  ${-camera_convergence/2.0}"/>
-	<parent link="head" />
-	<child link="left_camera" />
-      </joint>
-      <link name="left_camera" >
-	<!-- <collision> -->
-	<!--     <origin xyz="0 0 0" rpy="0 0 0"/> -->
-	<!--     <geometry> -->
-	<!--   <box size="${camera_link} ${camera_link} ${camera_link}"/> -->
-	<!--     </geometry> -->
-	<!--   </collision> -->
-	<!-- <visual> -->
-	<!--   <origin xyz="0 0 0" rpy="0 0 0"/> -->
-	<!--   <geometry> -->
-	<!-- <box size="${camera_link} ${camera_link} ${camera_link}"/> -->
-	<!--   </geometry> -->
-	<!--   <material name="red"/> -->
-	<!-- </visual> -->
-	<inertial>
-	  <mass value="1e-5" />
-	  <origin xyz="0 0 0" rpy="0 0 0"/>
-	  <inertia ixx="1e-6" ixy="0" ixz="0" iyy="1e-6" iyz="0" izz="1e-6" />
-	</inertial>
-      </link>
-      <link name="left_camera_optical">
-      </link>
-      <joint name="left_camera_optical_joint" type="fixed">
-	<!-- these values have to be these values otherwise the gazebo camera
-             image won't be aligned properly with the frame it is supposedly
-             originating from -->
-	<origin xyz="0 0 0" rpy="${-pi/2.0} 0 ${-pi/2.0}"/>
-	<parent link="left_camera"/>
-	<child link="left_camera_optical"/>
-      </joint>
-      <joint name="right_cam_fixed" type="fixed">
-	<origin xyz="0.02 -0.03625 0.06105" rpy="0.0 0.0 ${camera_convergence/2.0}"/>
-	<parent link="head" />
-	<child link="right_camera" />
-      </joint>
-      <link name="right_camera" >
-	<!-- <collision> -->
-	<!--     <origin xyz="0 0 0" rpy="0 0 0"/> -->
-	<!--     <geometry> -->
-	<!--   <box size="${camera_link} ${camera_link} ${camera_link}"/> -->
-	<!--     </geometry> -->
-	<!--   </collision> -->
-	<!-- <visual> -->
-	<!--   <origin xyz="0 0 0" rpy="0 0 0"/> -->
-	<!--   <geometry> -->
-	<!-- <box size="${camera_link} ${camera_link} ${camera_link}"/> -->
-	<!--   </geometry> -->
-	<!--   <material name="red"/> -->
-	<!-- </visual> -->
-	<inertial>
-	  <mass value="1e-5" />
-	  <origin xyz="0 0 0" rpy="0 0 0"/>
-	  <inertia ixx="1e-6" ixy="0" ixz="0" iyy="1e-6" iyz="0" izz="1e-6" />
-	</inertial>
-      </link>
-      <link name="right_camera_optical">
-      </link>
-      <joint name="right_camera_optical_joint" type="fixed">
-	<!-- these values have to be these values otherwise the gazebo camera
-             image won't be aligned properly with the frame it is supposedly
-             originating from -->
-	<origin xyz="0 0 0" rpy="${-pi/2.0} 0 ${-pi/2.0}"/>
-	<parent link="right_camera"/>
-	<child link="right_camera_optical"/>
-      </joint>
-      <gazebo reference="left_camera">
-	<!-- <link name="left_camera"> -->
-	<sensor type="camera" name="left_camera">
-          <!-- Set always_on only sensor, not on plugin -->
-          <always_on>0</always_on>
-          <!-- Set update_rate only sensor, not on plugin -->
-          <update_rate>30</update_rate>
-          <camera name="left_camera">
-            <horizontal_fov>1.3962634</horizontal_fov>
-            <image>
-              <width>800</width>
-              <height>800</height>
-              <format>R8G8B8</format>
-            </image>
-            <distortion>
-              <k1>0.0</k1>
-              <k2>0.0</k2>
-              <k3>0.0</k3>
-              <p1>0.0</p1>
-              <p2>0.0</p2>
-              <center>0.5 0.5</center>
-            </distortion>
-            <noise>
-              <type>gaussian</type>
-              <mean>0.0</mean>
-              <stddev>0.007</stddev>
-            </noise>
-          </camera>
-          <!-- Use camera, not camera_triggered -->
-          <plugin name="left_camera_controller" filename="libgazebo_ros_camera.so">
-              <ros>
-                <namespace>/</namespace>
-                <remapping>image_raw:=image_raw</remapping>
-                <remapping>camera_info:=camera_info</remapping>
-              </ros>
-              <camera_name>left_image</camera_name>
-            <!-- <ros> -->
-            <!--   <namespace>custom_ns</namespace> -->
-            <!--   <argument>image_raw:=custom_img</argument> -->
-            <!--   <argument>camera_info:=custom_info</argument> -->
-            <!-- </ros> -->
-            <!-- Set camera name. If empty, defaults to sensor name (i.e. "sensor_name") -->
-            <!-- <camera_name>left_camera</camera_name> -->
-            <!-- Set TF frame name. If empty, defaults to link name (i.e. "link_name") -->
-            <frame_name>left_camera_optical</frame_name>
-            <hack_baseline>0.07</hack_baseline>
-            <!-- No need to repeat distortion parameters or to set autoDistortion -->
-          </plugin>
-        </sensor>
-      </gazebo>
-      <gazebo reference="right_camera">
-	<sensor type="camera" name="right_camera">
-          <!-- Set always_on only sensor, not on plugin -->
-          <always_on>0</always_on>
-          <!-- Set update_rate only sensor, not on plugin -->
-          <update_rate>30</update_rate>
-          <camera name="right_camera">
-            <horizontal_fov>1.3962634</horizontal_fov>
-            <image>
-              <width>800</width>
-              <height>800</height>
-              <format>R8G8B8</format>
-            </image>
-            <distortion>
-              <k1>0.0</k1>
-              <k2>0.0</k2>
-              <k3>0.0</k3>
-              <p1>0.0</p1>
-              <p2>0.0</p2>
-              <center>0.5 0.5</center>
-            </distortion>
-            <noise>
-              <type>gaussian</type>
-              <mean>0.0</mean>
-              <stddev>0.007</stddev>
-            </noise>
-          </camera>
-          <!-- Use camera, not camera_triggered -->
-          <plugin name="right_camera_controller" filename="libgazebo_ros_camera.so">
-              <ros>
-                <namespace>/</namespace>
-                <remapping>image_raw:=image_raw</remapping>
-                <remapping>camera_info:=camera_info</remapping>
-              </ros>
-              <camera_name>right_image</camera_name>
-            <!-- <ros> -->
-            <!--   <namespace>custom_ns</namespace> -->
-            <!--   <argument>image_raw:=custom_img</argument> -->
-            <!--   <argument>camera_info:=custom_info</argument> -->
-            <!-- </ros> -->
-            <!-- Set camera name. If empty, defaults to sensor name (i.e. "sensor_name") -->
-            <!-- <camera_name>right_camera</camera_name> -->
-            <!-- Set TF frame name. If empty, defaults to link name (i.e. "link_name") -->
-            <frame_name>right_camera_optical</frame_name>
-            <hack_baseline>0.07</hack_baseline>
-            <!-- No need to repeat distortion parameters or to set autoDistortion -->
-          </plugin>
-        </sensor>
-      </gazebo>
-      <link name="depth_camera_link" >
-	<!-- <collision> -->
-	<!--     <origin xyz="0 0 0" rpy="0 0 0"/> -->
-	<!--     <geometry> -->
-	<!--   <box size="${camera_link} ${camera_link} ${camera_link}"/> -->
-	<!--     </geometry> -->
-	<!--   </collision> -->
-	<!-- <visual> -->
-	<!--   <origin xyz="0 0 0" rpy="0 0 0"/> -->
-	<!--   <geometry> -->
-	<!-- <box size="${camera_link} ${camera_link} ${camera_link}"/> -->
-	<!--   </geometry> -->
-	<!--   <material name="red"/> -->
-	<!-- </visual> -->
-	<inertial>
-	  <mass value="1e-5" />
-	  <origin xyz="0 0 0" rpy="0 0 0"/>
-	  <inertia ixx="1e-6" ixy="0" ixz="0" iyy="1e-6" iyz="0" izz="1e-6" />
-	</inertial>
-      </link>
-      <joint name="depth_cam_fixed" type="fixed">
-	<origin xyz="0.02 0 0.06105" rpy="0.0 0.0 0"/>
-	<parent link="head" />
-	<child link="depth_camera_link" />
-      </joint>
-      <link name="depth_camera_optical">
-      </link>
-      <joint name="depth_camera_optical_joint" type="fixed">
-	<!-- these values have to be these values otherwise the gazebo camera
-             image won't be aligned properly with the frame it is supposedly
-             originating from -->
-	<origin xyz="0 0 0" rpy="${-pi/2.0} 0 ${-pi/2.0}"/>
-	<parent link="depth_camera_link"/>
-	<child link="depth_camera_optical"/>
-      </joint>
-      <xacro:if value="$(arg depth_camera)">
-	<gazebo reference="depth_camera_link">
-	  <sensor name="depth_camera" type="depth">
-            <always_on>true</always_on>
-            <update_rate>15</update_rate>
-            <pose>0 0 0 0 0 0</pose>
-            <camera name="realsense_depth_camera">
-              <horizontal_fov>1.46608</horizontal_fov>
-              <image>
-                <width>424</width>
-                <height>240</height>
-                <format>B8G8R8</format>
-              </image>
-              <clip>
-                <near>0.05</near>
-                <far>8</far>
-              </clip>
-            </camera>
-            <!-- https://github.com/mlherd/ros2_turtlebot3_waffle_intel_realsense -->
-            <!-- <plugin name="intel_realsense_d430_depth_driver" filename="libgazebo_ros_camera.so"> -->
-            <plugin name="intel_realsense_r200_depth_driver" filename="libgazebo_ros_camera.so">
-              <ros>
-                <namespace>depth_camera</namespace>
-                <remapping>depth_camera/image_raw:=color/image_raw</remapping>
-                <remapping>depth_camera/depth/image_raw:=depth/image_rect_raw</remapping>
-                <remapping>depth_camera/camera_info:=camera_info</remapping>
-                <remapping>depth_camera/depth/camera_info:=depth/camera_info</remapping>
-                <remapping>depth_camera/points:=depth/points</remapping>
-              </ros>
-              <camera_name>depth_camera</camera_name>
-              <frame_name>depth_camera_optical</frame_name>
-              <hack_baseline>0.07</hack_baseline>
-              <min_depth>0.05</min_depth>
-              <max_depth>8.0</max_depth>
-            </plugin>
-	  </sensor>
-	</gazebo>
-      </xacro:if>
-</xacro:if>
+    <!-- Reachy Cameras -->
+<!--     <xacro:if value="$(arg use_gazebo)"> -->
+<!--       <joint name="left_cam_fixed" type="fixed"> -->
+<!-- 	<origin xyz="0.02 0.03625 0.06105" rpy="0.0 0.0  ${-camera_convergence/2.0}"/> -->
+<!-- 	<parent link="head" /> -->
+<!-- 	<child link="left_camera" /> -->
+<!--       </joint> -->
+<!--       <link name="left_camera" > -->
+<!-- 	<inertial> -->
+<!-- 	  <mass value="1e-5" /> -->
+<!-- 	  <origin xyz="0 0 0" rpy="0 0 0"/> -->
+<!-- 	  <inertia ixx="1e-6" ixy="0" ixz="0" iyy="1e-6" iyz="0" izz="1e-6" /> -->
+<!-- 	</inertial> -->
+<!--       </link> -->
+<!--       <link name="left_camera_optical"> -->
+<!--       </link> -->
+<!--       <joint name="left_camera_optical_joint" type="fixed"> -->
+<!-- 	<!-\- these values have to be these values otherwise the gazebo camera -->
+<!--              image won't be aligned properly with the frame it is supposedly -->
+<!--              originating from -\-> -->
+<!-- 	<origin xyz="0 0 0" rpy="${-pi/2.0} 0 ${-pi/2.0}"/> -->
+<!-- 	<parent link="left_camera"/> -->
+<!-- 	<child link="left_camera_optical"/> -->
+<!--       </joint> -->
+<!--       <joint name="right_cam_fixed" type="fixed"> -->
+<!-- 	<origin xyz="0.02 -0.03625 0.06105" rpy="0.0 0.0 ${camera_convergence/2.0}"/> -->
+<!-- 	<parent link="head" /> -->
+<!-- 	<child link="right_camera" /> -->
+<!--       </joint> -->
+<!--       <link name="right_camera" > -->
+<!-- 	<inertial> -->
+<!-- 	  <mass value="1e-5" /> -->
+<!-- 	  <origin xyz="0 0 0" rpy="0 0 0"/> -->
+<!-- 	  <inertia ixx="1e-6" ixy="0" ixz="0" iyy="1e-6" iyz="0" izz="1e-6" /> -->
+<!-- 	</inertial> -->
+<!--       </link> -->
+<!--       <link name="right_camera_optical"> -->
+<!--       </link> -->
+<!--       <joint name="right_camera_optical_joint" type="fixed"> -->
+<!-- 	<!-\- these values have to be these values otherwise the gazebo camera -->
+<!--              image won't be aligned properly with the frame it is supposedly -->
+<!--              originating from -\-> -->
+<!-- 	<origin xyz="0 0 0" rpy="${-pi/2.0} 0 ${-pi/2.0}"/> -->
+<!-- 	<parent link="right_camera"/> -->
+<!-- 	<child link="right_camera_optical"/> -->
+<!--       </joint> -->
+<!--       <gazebo reference="left_camera"> -->
+<!-- 	<!-\- <link name="left_camera"> -\-> -->
+<!-- 	<sensor type="camera" name="left_camera"> -->
+<!--           <!-\- Set always_on only sensor, not on plugin -\-> -->
+<!--           <always_on>0</always_on> -->
+<!--           <!-\- Set update_rate only sensor, not on plugin -\-> -->
+<!--           <update_rate>30</update_rate> -->
+<!--           <camera name="left_camera"> -->
+<!--             <horizontal_fov>1.3962634</horizontal_fov> -->
+<!--             <image> -->
+<!--               <width>800</width> -->
+<!--               <height>800</height> -->
+<!--               <format>R8G8B8</format> -->
+<!--             </image> -->
+<!--             <distortion> -->
+<!--               <k1>0.0</k1> -->
+<!--               <k2>0.0</k2> -->
+<!--               <k3>0.0</k3> -->
+<!--               <p1>0.0</p1> -->
+<!--               <p2>0.0</p2> -->
+<!--               <center>0.5 0.5</center> -->
+<!--             </distortion> -->
+<!--             <noise> -->
+<!--               <type>gaussian</type> -->
+<!--               <mean>0.0</mean> -->
+<!--               <stddev>0.007</stddev> -->
+<!--             </noise> -->
+<!--           </camera> -->
+<!--           <!-\- Use camera, not camera_triggered -\-> -->
+<!--           <plugin name="left_camera_controller" filename="libgazebo_ros_camera.so"> -->
+<!--               <ros> -->
+<!--                 <namespace>/</namespace> -->
+<!--                 <remapping>image_raw:=image_raw</remapping> -->
+<!--                 <remapping>camera_info:=camera_info</remapping> -->
+<!--               </ros> -->
+<!--               <camera_name>left_image</camera_name> -->
+<!--             <!-\- <ros> -\-> -->
+<!--             <!-\-   <namespace>custom_ns</namespace> -\-> -->
+<!--             <!-\-   <argument>image_raw:=custom_img</argument> -\-> -->
+<!--             <!-\-   <argument>camera_info:=custom_info</argument> -\-> -->
+<!--             <!-\- </ros> -\-> -->
+<!--             <!-\- Set camera name. If empty, defaults to sensor name (i.e. "sensor_name") -\-> -->
+<!--             <!-\- <camera_name>left_camera</camera_name> -\-> -->
+<!--             <!-\- Set TF frame name. If empty, defaults to link name (i.e. "link_name") -\-> -->
+<!--             <frame_name>left_camera_optical</frame_name> -->
+<!--             <hack_baseline>0.07</hack_baseline> -->
+<!--             <!-\- No need to repeat distortion parameters or to set autoDistortion -\-> -->
+<!--           </plugin> -->
+<!--         </sensor> -->
+<!--       </gazebo> -->
+<!--       <gazebo reference="right_camera"> -->
+<!-- 	<sensor type="camera" name="right_camera"> -->
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
File: reachy_description/urdf/orbita.urdf.xacro (robot description, xacro)
@@ -6,4 +6,10 @@
     <!-- 54°?? -->
   <xacro:property name="orbita_alpha" value="0.9424777960769379"/>
+    <material name="orbitayellow">
+        <color rgba="0.8 0.8 0.0 1"/>
+    </material>
+    <material name="orbitagrey">
+        <color rgba="0.8 0.8 0.8 1"/>
+    </material>
     <!--
       Orbita
@@ -24,4 +30,11 @@
     </link>
     <link name="${name}_link">
+      <visual>
+      	<origin xyz="0 0 ${length/2}" rpy="0 0 0"/>
+      	<geometry>
+          <cylinder length="${length}" radius="${radius}"/>
+      	</geometry>
+      	<material name="orbitayellow"/>
+      </visual>
       <collision>
       	<origin xyz="0 0 ${length/2}" rpy="0 0 0"/>
@@ -30,11 +43,4 @@
       	</geometry>
       </collision>
-      <visual>
-      	<origin xyz="0 0 ${length/2}" rpy="0 0 0"/>
-      	<geometry>
-          <cylinder length="${length}" radius="${radius}"/>
-      	</geometry>
-      	<material name="yellow"/>
-      </visual>
       <xacro:inertial_cuboid mass="${mass*0.48}" xyz="0 0 ${-length/2}"  rpy="0 0 0" x_length="${radius*2}" y_length="${radius*2}" z_length="${length}">
       </xacro:inertial_cuboid>
@@ -46,5 +52,5 @@
           <sphere radius="${radius*1.2}"/>
       	</geometry>
-      	<!-- <material name="grey"/> -->
+      	<material name="orbitagrey"/>
       </visual>
       <collision>

File: reachy_description/urdf/orbita2dof.urdf.xacro (robot description, xacro)
@@ -3,4 +3,10 @@
   <xacro:include filename="$(find reachy_description)/urdf/inertial_primitives.urdf.xacro"/>
   <xacro:include filename="$(find reachy_description)/ros2_control/orbita2dof.ros2_control.xacro"/>
+    <material name="orbita2dmetal">
+        <color rgba="0.85 0.85 0.85 1"/>
+    </material>
+    <material name="orbita2dgrey">
+        <color rgba="0.8 0.8 0.8 1"/>
+    </material>
   <xacro:macro name="joint2axis" params="joint">
     <xacro:if value="${joint == 'roll'}">
@@ -39,5 +45,6 @@
       	<origin xyz="0 0 ${-length/2}" rpy="0 0 0"/>
       	<geometry>
-          <cylinder length="${length}" radius="${radius}"/>
+          <!-- <cylinder length="${length}" radius="${radius}"/> -->
+	  <box size="${radius*2.5} ${radius*2.0} ${length}"/>
       	</geometry>
       </collision>
@@ -45,7 +52,8 @@
       	<origin xyz="0 0 ${-length/2}" rpy="0 0 0"/>
       	<geometry>
-          <cylinder length="${length}" radius="${radius}"/>
+          <!-- <cylinder length="${length}" radius="${radius}"/> -->
+	  <box size="${radius*2.5} ${radius*2.0} ${length}"/>
       	</geometry>
-      	<material name="yellow"/>
+      	<material name= "orbita2dmetal"/>
       </visual>
       <xacro:inertial_cuboid mass="${mass*0.49}" xyz="0 0 ${-length/2}"  rpy="0 0 0" x_length="${radius*2}" y_length="${radius*2}" z_length="${length}"/>
@@ -69,5 +77,5 @@
           <sphere radius="${radius*1.2}"/>
       	</geometry>
-      	<!-- <material name="grey"/> -->
+      	<material name="orbita2dgrey"/>
       </visual>
       <collision>

File: reachy_description/urdf/reachy.urdf.xacro (robot description, xacro)
@@ -43,4 +43,7 @@
   <xacro:property name="forearm_length" value="0.28"/>
   <!-- MODEL PARAMETERS -->
+    <material name="torsoblack">
+        <color rgba="0.5 0.5 0.5 1"/>
+    </material>
   <link name="world"/>
   <joint name="world_joint" type="fixed">
@@ -69,5 +72,5 @@
         <!--   <cylinder length="1" radius="0.03"/> -->
         <!-- </geometry> -->
-        <material name="black"/>
+        <material name="torsoblack"/>
       </visual>
     </xacro:if>

File: reachy_description/urdf/smartgripper.urdf.xacro (robot description, xacro)
@@ -16,4 +16,10 @@
     <xacro:property name="max_grasping_finger" value="2.094"/>
   </xacro:if>
+    <material name="gripperblack">
+        <color rgba="0.4 0.4 0.4 1"/>
+    </material>
+    <material name="gripperwhite">
+        <color rgba="0.9 0.9 0.9 1"/>
+    </material>
   <xacro:property name="p" value="${prefix}_gripper"/>
   <link name="${p}_palm_link">
@@ -29,5 +35,5 @@
         <box size="${gripper_radius} ${gripper_radius*2} ${gripper_length/2}"/>
       </geometry>
-      <material name="yellow"/>
+      <material name="gripperblack"/>
     </visual>
     <xacro:inertial_cuboid mass="${gripper_mass*0.85}" xyz="0 0 ${gripper_length/4}"  rpy="0 0 0" x_length="${gripper_radius}" y_length="${gripper_radius*2}" z_length="${gripper_length/2}"/>
@@ -50,5 +56,5 @@
         <box size="${gripper_radius} 0.01 ${gripper_length/2}"/>
       </geometry>
-      <material name="yellow"/>
+      <material name="gripperwhite"/>
     </visual>
     <xacro:inertial_cuboid mass="${gripper_mass*0.1}" xyz="0 ${gripper_radius} ${gripper_length/4}"  rpy="0 0 0" x_length="${gripper_radius}" y_length="0.01" z_length="${gripper_length/2}"/>
@@ -66,5 +72,5 @@
         <box size="${gripper_radius} 0.01 ${gripper_length/2}"/>
       </geometry>
-      <material name="yellow"/>
+      <material name="gripperwhite"/>
     </visual>
     <xacro:inertial_cuboid mass="${gripper_mass*0.1}" xyz="0 ${gripper_radius} ${gripper_length/4}"  rpy="0 0 0" x_length="${gripper_radius}" y_length="0.01" z_length="${gripper_length/2}"/>

Commit message: add head tracker

File: reachy_description/urdf/head.urdf.xacro (robot description, xacro)
@@ -172,4 +172,18 @@
       <parent link="head" />
       <child link="head_base" />
+    </joint>
+    <link name="head_tracker">
+      <visual name="">
+        <origin xyz="0 0 0" rpy="0.0 0.0 0.0"/>
+        <geometry>
+	  <cylinder length="0.04" radius="0.04"/>
+        </geometry>
+	<material name="camblack"/>
+      </visual>
+    </link>
+    <joint name="head_tracker_fixed" type="fixed">
+      <origin xyz="-0.035 0.0 0.108" rpy="0.0 0.0 0"/>
+      <parent link="head" />
+      <child link="head_tracker" />
     </joint>
     <link name="head_tip" >
