Commit message: updating urdf

File: reachy_description/urdf/head.urdf.xacro (robot description, xacro)
@@ -15,5 +15,5 @@
     <xacro:include filename="$(find reachy_description)/ros2_control/head.ros2_control.xacro"/>
     <joint name="neck_roll" type="revolute">
-      <origin xyz="-0.032893 0.0 0.110675" rpy="-0.15105105 0.08669986 -1.05356462"/>
+      <origin xyz="-0.032893 0.0 0.110675" rpy="0.0 0.17453293 0.0"/>
       <parent link="${parent}"/>
       <child link="head_x"/>
@@ -60,5 +60,5 @@
     </link>
     <joint name="neck_fixed" type="fixed">
-      <origin xyz="0 0 0" rpy="0.0 0.0 1.047"/>
+      <origin xyz="0 0 0" rpy="0.0 0.0 0.0"/>
       <parent link="head_z" />
       <child link="head" />
@@ -183,5 +183,5 @@
     </link>
     <joint name="head_tracker_fixed" type="fixed">
-      <origin xyz="-0.035 0.0 0.108" rpy="0.0 0.0 0"/>
+      <origin xyz="-0.030 0.0 0.111" rpy="0.0 0.0 0"/>
       <parent link="head" />
       <child link="head_tracker" />
@@ -191,5 +191,5 @@
     <joint name="head_tip_fixed" type="fixed">
       <!-- between the cameras -->
-      <origin xyz="0.015 0 0.085" rpy="0.0 0.0 0"/>
+      <origin xyz="0.030 0.022 0.085" rpy="-1.57 0.0 -1.57"/>
       <!-- Rotation center -->
       <!-- <origin xyz="0.0 0 0.0" rpy="0.0 0.0 0"/> -->

Commit message: urdf correction

File: reachy_description/urdf/head.urdf.xacro (robot description, xacro)
@@ -191,9 +191,19 @@
     <joint name="head_tip_fixed" type="fixed">
       <!-- between the cameras -->
+      <origin xyz="0.030 0.022 0.085" rpy="0 0.0 0"/>
+      <!-- Rotation center -->
+      <!-- <origin xyz="0.0 0 0.0" rpy="0.0 0.0 0"/> -->
+      <parent link="head" />
+      <child link="head_tip" />
+    </joint>
+    <link name="camera_optical_left" >
+    </link>
+    <joint name="camera_optical_left" type="fixed">
+      <!-- between the cameras -->
       <origin xyz="0.030 0.022 0.085" rpy="-1.57 0.0 -1.57"/>
       <!-- Rotation center -->
       <!-- <origin xyz="0.0 0 0.0" rpy="0.0 0.0 0"/> -->
       <parent link="head" />
-      <child link="head_tip" />
+      <child link="camera_optical_left" />
     </joint>
     <!-- <link name="l_antenna_link"> -->

Commit message: add cameras

File: reachy_description/urdf/head.urdf.xacro (robot description, xacro)
@@ -1,5 +1,5 @@
 <?xml version="1.0"?>
 <robot xmlns:xacro="http://www.ros.org/wiki/xacro">
-  <xacro:arg name="depth_camera" default="false"/>
+  <xacro:arg name="depth_camera" default="true"/>
   <xacro:property name="camera_link" value="0.05" /> <!-- Size of square 'camera' box -->
   <xacro:property name="camera_convergence" value="0.0" /> <!-- convergence angle (rad) of the cameras. 0=parallel-->
@@ -103,209 +103,209 @@
     </joint>
     <!-- Reachy Cameras -->
-<!--     <xacro:if value="$(arg use_gazebo)"> -->
-<!--       <joint name="left_cam_fixed" type="fixed"> -->
-<!-- 	<origin xyz="0.02 0.03625 0.06105" rpy="0.0 0.0  ${-camera_convergence/2.0}"/> -->
-<!-- 	<parent link="head" /> -->
-<!-- 	<child link="left_camera" /> -->
-<!--       </joint> -->
-<!--       <link name="left_camera" > -->
-<!-- 	<inertial> -->
-<!-- 	  <mass value="1e-5" /> -->
-<!-- 	  <origin xyz="0 0 0" rpy="0 0 0"/> -->
-<!-- 	  <inertia ixx="1e-6" ixy="0" ixz="0" iyy="1e-6" iyz="0" izz="1e-6" /> -->
-<!-- 	</inertial> -->
-<!--       </link> -->
-<!--       <link name="left_camera_optical"> -->
-<!--       </link> -->
-<!--       <joint name="left_camera_optical_joint" type="fixed"> -->
-<!-- 	<!-\- these values have to be these values otherwise the gazebo camera -->
-<!--              image won't be aligned properly with the frame it is supposedly -->
-<!--              originating from -\-> -->
-<!-- 	<origin xyz="0 0 0" rpy="${-pi/2.0} 0 ${-pi/2.0}"/> -->
-<!-- 	<parent link="left_camera"/> -->
-<!-- 	<child link="left_camera_optical"/> -->
-<!--       </joint> -->
-<!--       <joint name="right_cam_fixed" type="fixed"> -->
-<!-- 	<origin xyz="0.02 -0.03625 0.06105" rpy="0.0 0.0 ${camera_convergence/2.0}"/> -->
-<!-- 	<parent link="head" /> -->
-<!-- 	<child link="right_camera" /> -->
-<!--       </joint> -->
-<!--       <link name="right_camera" > -->
-<!-- 	<inertial> -->
-<!-- 	  <mass value="1e-5" /> -->
-<!-- 	  <origin xyz="0 0 0" rpy="0 0 0"/> -->
-<!-- 	  <inertia ixx="1e-6" ixy="0" ixz="0" iyy="1e-6" iyz="0" izz="1e-6" /> -->
-<!-- 	</inertial> -->
-<!--       </link> -->
-<!--       <link name="right_camera_optical"> -->
-<!--       </link> -->
-<!--       <joint name="right_camera_optical_joint" type="fixed"> -->
-<!-- 	<!-\- these values have to be these values otherwise the gazebo camera -->
-<!--              image won't be aligned properly with the frame it is supposedly -->
-<!--              originating from -\-> -->
-<!-- 	<origin xyz="0 0 0" rpy="${-pi/2.0} 0 ${-pi/2.0}"/> -->
-<!-- 	<parent link="right_camera"/> -->
-<!-- 	<child link="right_camera_optical"/> -->
-<!--       </joint> -->
-<!--       <gazebo reference="left_camera"> -->
-<!-- 	<!-\- <link name="left_camera"> -\-> -->
-<!-- 	<sensor type="camera" name="left_camera"> -->
-<!--           <!-\- Set always_on only sensor, not on plugin -\-> -->
-<!--           <always_on>0</always_on> -->
-<!--           <!-\- Set update_rate only sensor, not on plugin -\-> -->
-<!--           <update_rate>30</update_rate> -->
-<!--           <camera name="left_camera"> -->
-<!--             <horizontal_fov>1.3962634</horizontal_fov> -->
-<!--             <image> -->
-<!--               <width>800</width> -->
-<!--               <height>800</height> -->
-<!--               <format>R8G8B8</format> -->
-<!--             </image> -->
-<!--             <distortion> -->
-<!--               <k1>0.0</k1> -->
-<!--               <k2>0.0</k2> -->
-<!--               <k3>0.0</k3> -->
-<!--               <p1>0.0</p1> -->
-<!--               <p2>0.0</p2> -->
-<!--               <center>0.5 0.5</center> -->
-<!--             </distortion> -->
-<!--             <noise> -->
-<!--               <type>gaussian</type> -->
-<!--               <mean>0.0</mean> -->
-<!--               <stddev>0.007</stddev> -->
-<!--             </noise> -->
-<!--           </camera> -->
-<!--           <!-\- Use camera, not camera_triggered -\-> -->
-<!--           <plugin name="left_camera_controller" filename="libgazebo_ros_camera.so"> -->
-<!--               <ros> -->
-<!--                 <namespace>/</namespace> -->
-<!--                 <remapping>image_raw:=image_raw</remapping> -->
-<!--                 <remapping>camera_info:=camera_info</remapping> -->
-<!--               </ros> -->
-<!--               <camera_name>left_image</camera_name> -->
-<!--             <!-\- <ros> -\-> -->
-<!--             <!-\-   <namespace>custom_ns</namespace> -\-> -->
-<!--             <!-\-   <argument>image_raw:=custom_img</argument> -\-> -->
-<!--             <!-\-   <argument>camera_info:=custom_info</argument> -\-> -->
-<!--             <!-\- </ros> -\-> -->
-<!--             <!-\- Set camera name. If empty, defaults to sensor name (i.e. "sensor_name") -\-> -->
-<!--             <!-\- <camera_name>left_camera</camera_name> -\-> -->
-<!--             <!-\- Set TF frame name. If empty, defaults to link name (i.e. "link_name") -\-> -->
-<!--             <frame_name>left_camera_optical</frame_name> -->
-<!--             <hack_baseline>0.07</hack_baseline> -->
-<!--             <!-\- No need to repeat distortion parameters or to set autoDistortion -\-> -->
-<!--           </plugin> -->
-<!--         </sensor> -->
-<!--       </gazebo> -->
-<!--       <gazebo reference="right_camera"> -->
-<!-- 	<sensor type="camera" name="right_camera"> -->
-<!--           <!-\- Set always_on only sensor, not on plugin -\-> -->
-<!--           <always_on>0</always_on> -->
-<!--           <!-\- Set update_rate only sensor, not on plugin -\-> -->
-<!--           <update_rate>30</update_rate> -->
-<!--           <camera name="right_camera"> -->
-<!--             <horizontal_fov>1.3962634</horizontal_fov> -->
-<!--             <image> -->
-<!--               <width>800</width> -->
-<!--               <height>800</height> -->
-<!--               <format>R8G8B8</format> -->
-<!--             </image> -->
-<!--             <distortion> -->
-<!--               <k1>0.0</k1> -->
-<!--               <k2>0.0</k2> -->
-<!--               <k3>0.0</k3> -->
-<!--               <p1>0.0</p1> -->
-<!--               <p2>0.0</p2> -->
-<!--               <center>0.5 0.5</center> -->
-<!--             </distortion> -->
-<!--             <noise> -->
-<!--               <type>gaussian</type> -->
-<!--               <mean>0.0</mean> -->
-<!--               <stddev>0.007</stddev> -->
-<!--             </noise> -->
-<!--           </camera> -->
-<!--           <!-\- Use camera, not camera_triggered -\-> -->
-<!--           <plugin name="right_camera_controller" filename="libgazebo_ros_camera.so"> -->
-<!--               <ros> -->
-<!--                 <namespace>/</namespace> -->
-<!--                 <remapping>image_raw:=image_raw</remapping> -->
-<!--                 <remapping>camera_info:=camera_info</remapping> -->
-<!--               </ros> -->
-<!--               <camera_name>right_image</camera_name> -->
-<!--             <!-\- <ros> -\-> -->
-<!--             <!-\-   <namespace>custom_ns</namespace> -\-> -->
-<!--             <!-\-   <argument>image_raw:=custom_img</argument> -\-> -->
-<!--             <!-\-   <argument>camera_info:=custom_info</argument> -\-> -->
-<!--             <!-\- </ros> -\-> -->
-<!--             <!-\- Set camera name. If empty, defaults to sensor name (i.e. "sensor_name") -\-> -->
-<!--             <!-\- <camera_name>right_camera</camera_name> -\-> -->
-<!--             <!-\- Set TF frame name. If empty, defaults to link name (i.e. "link_name") -\-> -->
-<!--             <frame_name>right_camera_optical</frame_name> -->
-<!--             <hack_baseline>0.07</hack_baseline> -->
-<!--             <!-\- No need to repeat distortion parameters or to set autoDistortion -\-> -->
-<!--           </plugin> -->
-<!--         </sensor> -->
-<!--       </gazebo> -->
-<!--       <link name="depth_camera_link" > -->
-<!-- 	<inertial> -->
-<!-- 	  <mass value="1e-5" /> -->
-<!-- 	  <origin xyz="0 0 0" rpy="0 0 0"/> -->
-<!-- 	  <inertia ixx="1e-6" ixy="0" ixz="0" iyy="1e-6" iyz="0" izz="1e-6" /> -->
-<!-- 	</inertial> -->
-<!--       </link> -->
-<!--       <joint name="depth_cam_fixed" type="fixed"> -->
-<!-- 	<origin xyz="0.02 0 0.06105" rpy="0.0 0.0 0"/> -->
-<!-- 	<parent link="head" /> -->
-<!-- 	<child link="depth_camera_link" /> -->
-<!--       </joint> -->
-<!--       <link name="depth_camera_optical"> -->
-<!--       </link> -->
-<!--       <joint name="depth_camera_optical_joint" type="fixed"> -->
-<!-- 	<!-\- these values have to be these values otherwise the gazebo camera -->
-<!--              image won't be aligned properly with the frame it is supposedly -->
-<!--              originating from -\-> -->
-<!-- 	<origin xyz="0 0 0" rpy="${-pi/2.0} 0 ${-pi/2.0}"/> -->
-<!-- 	<parent link="depth_camera_link"/> -->
-<!-- 	<child link="depth_camera_optical"/> -->
-<!--       </joint> -->
-<!--       <xacro:if value="$(arg depth_camera)"> -->
-<!-- 	<gazebo reference="depth_camera_link"> -->
-<!-- 	  <sensor name="depth_camera" type="depth"> -->
-<!--             <always_on>true</always_on> -->
-<!--             <update_rate>15</update_rate> -->
-<!--             <pose>0 0 0 0 0 0</pose> -->
-<!--             <camera name="realsense_depth_camera"> -->
-<!--               <horizontal_fov>1.46608</horizontal_fov> -->
-<!--               <image> -->
-<!--                 <width>424</width> -->
-<!--                 <height>240</height> -->
-<!--                 <format>B8G8R8</format> -->
-<!--               </image> -->
-<!--               <clip> -->
-<!--                 <near>0.05</near> -->
-<!--                 <far>8</far> -->
-<!--               </clip> -->
-<!--             </camera> -->
-<!--             <!-\- https://github.com/mlherd/ros2_turtlebot3_waffle_intel_realsense -\-> -->
-<!--             <!-\- <plugin name="intel_realsense_d430_depth_driver" filename="libgazebo_ros_camera.so"> -\-> -->
-<!--             <plugin name="intel_realsense_r200_depth_driver" filename="libgazebo_ros_camera.so"> -->
-<!--               <ros> -->
-<!--                 <namespace>depth_camera</namespace> -->
-<!--                 <remapping>depth_camera/image_raw:=color/image_raw</remapping> -->
-<!--                 <remapping>depth_camera/depth/image_raw:=depth/image_rect_raw</remapping> -->
-<!--                 <remapping>depth_camera/camera_info:=camera_info</remapping> -->
-<!--                 <remapping>depth_camera/depth/camera_info:=depth/camera_info</remapping> -->
-<!--                 <remapping>depth_camera/points:=depth/points</remapping> -->
-<!--               </ros> -->
-<!--               <camera_name>depth_camera</camera_name> -->
-<!--               <frame_name>depth_camera_optical</frame_name> -->
-<!--               <hack_baseline>0.07</hack_baseline> -->
-<!--               <min_depth>0.05</min_depth> -->
-<!--               <max_depth>8.0</max_depth> -->
-<!--             </plugin> -->
-<!-- 	  </sensor> -->
-<!-- 	</gazebo> -->
-<!--       </xacro:if> -->
-<!-- </xacro:if> -->
+    <xacro:if value="$(arg use_gazebo)">
+      <joint name="left_cam_fixed" type="fixed">
+	<origin xyz="0.02 0.03625 0.06105" rpy="0.0 0.0  ${-camera_convergence/2.0}"/>
+	<parent link="head" />
+	<child link="left_camera" />
+      </joint>
+      <link name="left_camera" >
+	<inertial>
+	  <mass value="1e-5" />
+	  <origin xyz="0 0 0" rpy="0 0 0"/>
+	  <inertia ixx="1e-6" ixy="0" ixz="0" iyy="1e-6" iyz="0" izz="1e-6" />
+	</inertial>
+      </link>
+      <link name="left_camera_optical">
+      </link>
+      <joint name="left_camera_optical_joint" type="fixed">
+	<!-- these values have to be these values otherwise the gazebo camera
+             image won't be aligned properly with the frame it is supposedly
+             originating from -->
+	<origin xyz="0 0 0" rpy="${-pi/2.0} 0 ${-pi/2.0}"/>
+	<parent link="left_camera"/>
+	<child link="left_camera_optical"/>
+      </joint>
+      <joint name="right_cam_fixed" type="fixed">
+	<origin xyz="0.02 -0.03625 0.06105" rpy="0.0 0.0 ${camera_convergence/2.0}"/>
+	<parent link="head" />
+	<child link="right_camera" />
+      </joint>
+      <link name="right_camera" >
+	<inertial>
+	  <mass value="1e-5" />
+	  <origin xyz="0 0 0" rpy="0 0 0"/>
+	  <inertia ixx="1e-6" ixy="0" ixz="0" iyy="1e-6" iyz="0" izz="1e-6" />
+	</inertial>
+      </link>
+      <link name="right_camera_optical">
+      </link>
+      <joint name="right_camera_optical_joint" type="fixed">
+	<!-- these values have to be these values otherwise the gazebo camera
+             image won't be aligned properly with the frame it is supposedly
+             originating from -->
+	<origin xyz="0 0 0" rpy="${-pi/2.0} 0 ${-pi/2.0}"/>
+	<parent link="right_camera"/>
+	<child link="right_camera_optical"/>
+      </joint>
+      <gazebo reference="left_camera">
+	<!-- <link name="left_camera"> -->
+	<sensor type="camera" name="left_camera">
+          <!-- Set always_on only sensor, not on plugin -->
+          <always_on>0</always_on>
+          <!-- Set update_rate only sensor, not on plugin -->
+          <update_rate>30</update_rate>
+          <camera name="left_camera">
+            <horizontal_fov>1.3962634</horizontal_fov>
+            <image>
+              <width>800</width>
+              <height>800</height>
+              <format>R8G8B8</format>
+            </image>
+            <distortion>
+              <k1>0.0</k1>
+              <k2>0.0</k2>
+              <k3>0.0</k3>
+              <p1>0.0</p1>
+              <p2>0.0</p2>
+              <center>0.5 0.5</center>
+            </distortion>
+            <noise>
+              <type>gaussian</type>
+              <mean>0.0</mean>
+              <stddev>0.007</stddev>
+            </noise>
+          </camera>
+          <!-- Use camera, not camera_triggered -->
+          <plugin name="left_camera_controller" filename="libgazebo_ros_camera.so">
+              <ros>
+                <namespace>/</namespace>
+                <remapping>image_raw:=image_raw</remapping>
+                <remapping>camera_info:=camera_info</remapping>
+              </ros>
+              <camera_name>left_image</camera_name>
+            <!-- <ros> -->
+            <!--   <namespace>custom_ns</namespace> -->
+            <!--   <argument>image_raw:=custom_img</argument> -->
+            <!--   <argument>camera_info:=custom_info</argument> -->
+            <!-- </ros> -->
+            <!-- Set camera name. If empty, defaults to sensor name (i.e. "sensor_name") -->
+            <!-- <camera_name>left_camera</camera_name> -->
+            <!-- Set TF frame name. If empty, defaults to link name (i.e. "link_name") -->
+            <frame_name>left_camera_optical</frame_name>
+            <hack_baseline>0.07</hack_baseline>
+            <!-- No need to repeat distortion parameters or to set autoDistortion -->
+          </plugin>
+        </sensor>
+      </gazebo>
+      <gazebo reference="right_camera">
+	<sensor type="camera" name="right_camera">
+          <!-- Set always_on only sensor, not on plugin -->
+          <always_on>0</always_on>
+          <!-- Set update_rate only sensor, not on plugin -->
+          <update_rate>30</update_rate>
+          <camera name="right_camera">
+            <horizontal_fov>1.3962634</horizontal_fov>
+            <image>
+              <width>800</width>
+              <height>800</height>
+              <format>R8G8B8</format>
+            </image>
+            <distortion>
+              <k1>0.0</k1>
+              <k2>0.0</k2>
+              <k3>0.0</k3>
+              <p1>0.0</p1>
+              <p2>0.0</p2>
+              <center>0.5 0.5</center>
+            </distortion>
+            <noise>
+              <type>gaussian</type>
+              <mean>0.0</mean>
+              <stddev>0.007</stddev>
+            </noise>
+          </camera>
+          <!-- Use camera, not camera_triggered -->
+          <plugin name="right_camera_controller" filename="libgazebo_ros_camera.so">
+              <ros>
+                <namespace>/</namespace>
+                <remapping>image_raw:=image_raw</remapping>
+                <remapping>camera_info:=camera_info</remapping>
+              </ros>
+              <camera_name>right_image</camera_name>
+            <!-- <ros> -->
+            <!--   <namespace>custom_ns</namespace> -->
+            <!--   <argument>image_raw:=custom_img</argument> -->
+            <!--   <argument>camera_info:=custom_info</argument> -->
+            <!-- </ros> -->
+            <!-- Set camera name. If empty, defaults to sensor name (i.e. "sensor_name") -->
+            <!-- <camera_name>right_camera</camera_name> -->
+            <!-- Set TF frame name. If empty, defaults to link name (i.e. "link_name") -->
+            <frame_name>right_camera_optical</frame_name>
+            <hack_baseline>0.07</hack_baseline>
+            <!-- No need to repeat distortion parameters or to set autoDistortion -->
+          </plugin>
+        </sensor>
+      </gazebo>
+      <link name="depth_camera_link" >
+	<inertial>
+	  <mass value="1e-5" />
+	  <origin xyz="0 0 0" rpy="0 0 0"/>
+	  <inertia ixx="1e-6" ixy="0" ixz="0" iyy="1e-6" iyz="0" izz="1e-6" />
+	</inertial>
+      </link>
+      <joint name="depth_cam_fixed" type="fixed">
+	<origin xyz="0.02 0 0.06105" rpy="0.0 0.0 0"/>
+	<parent link="head" />
+	<child link="depth_camera_link" />
+      </joint>
+      <link name="depth_camera_optical">
+      </link>
+      <joint name="depth_camera_optical_joint" type="fixed">
+	<!-- these values have to be these values otherwise the gazebo camera
+             image won't be aligned properly with the frame it is supposedly
+             originating from -->
+	<origin xyz="0 0 0" rpy="${-pi/2.0} 0 ${-pi/2.0}"/>
+	<parent link="depth_camera_link"/>
+	<child link="depth_camera_optical"/>
+      </joint>
+      <xacro:if value="$(arg depth_camera)">
+	<gazebo reference="depth_camera_link">
+	  <sensor name="depth_camera" type="depth">
+            <always_on>true</always_on>
+            <update_rate>15</update_rate>
+            <pose>0 0 0 0 0 0</pose>
+            <camera name="realsense_depth_camera">
+              <horizontal_fov>1.46608</horizontal_fov>
+              <image>
+                <width>424</width>
+                <height>240</height>
+                <format>B8G8R8</format>
+              </image>
+              <clip>
+                <near>0.05</near>
+                <far>8</far>
+              </clip>
+            </camera>
+            <!-- https://github.com/mlherd/ros2_turtlebot3_waffle_intel_realsense -->
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