Commit message: wip

File: reachy_description/urdf/head.urdf.xacro (robot description, xacro)
@@ -7,8 +7,8 @@
   <xacro:property name="neck_radius" value="0.03"/>
   <xacro:property name="neck_mass" value="0.5"/>
-  <xacro:property name="neck_offset_x" value="-0.032893"/>
+  <xacro:property name="neck_offset_x" value="-0.0465"/>
   <xacro:property name="neck_offset_y" value="0"/>
-  <xacro:property name="neck_offset_z" value="0.110675"/>
-  <xacro:property name="neck_offset_pitch" value="0.17453293"/>
+  <xacro:property name="neck_offset_z" value="0.125"/>
+  <xacro:property name="neck_offset_pitch" value="${radians(10)}"/> <!-- 10 degrees -->
   <xacro:property name="neck_offset_yaw" value="0.0"/>
   <xacro:include filename="$(find orbita3d_description)/urdf/orbita3d.urdf.xacro"/>
@@ -21,13 +21,13 @@
   <xacro:macro name="head" params="parent damping friction neck_config">
   <xacro:orbita3d
-    name="neck" parent="torso"
+    name="neck" parent="${parent}"
     length="${neck_length}" radius="${neck_radius}" mass="${neck_mass}"
-    xyz="${neck_offset_x} ${neck_offset_y} ${neck_offset_z}" rpy="0 0 ${neck_offset_yaw}"
+    xyz="${neck_offset_x} ${neck_offset_y} ${neck_offset_z}" rpy="${pi} ${neck_offset_pitch} ${neck_offset_yaw}"
     damping="${damping}" friction="${friction}"
     config_file="${neck_config}"
-  />
+    />
     <joint name="neck_fixed" type="fixed">
       <origin xyz="0 0 0" rpy="0.0 0.0 0.0"/>
-      <parent link="neck_ball_link" />
+      <parent link="neck_out_link" />
       <child link="head" />
     </joint>
@@ -35,31 +35,24 @@
     <link name="head">
       <inertial>
-        <origin xyz="-0.009 -0.002 0.059" rpy="0.0 0.0 0.0"/>
-        <mass value="0.237"/>
-        <inertia ixx="1.676e-3" ixy="3.068e-6" ixz="1.2449e-4" iyy="1.368e-3" iyz="3.360e-5" izz="8.425e-4"/>
+        <origin xyz="0.0116978 -0.00022144 0.0611705" rpy="0.0 0.0 0.0"/>
+        <mass value="0.325"/>
+	 <inertia ixx="0.00085265" ixy="-0.00000298" ixz="0.00000932"
+		  iyx="-0.00000298" iyy="0.00063136" iyz="-0.000000039"
+		  izx="0.00000932" izy="-0.000000039" izz="0.0008951"/>
       </inertial>
-      <visual name="">
-        <origin xyz="0.0075 0.0 0.085" rpy="0.0 0.0 0.0"/>
+      <visual>
+        <origin xyz="0.00 0.0 0.0" rpy="0.0 0.0 0.0"/>
         <geometry>
-          <!-- <mesh filename="file://$(find reachy_description)/meshes/head.dae"/> -->
-	  <box size="0.015 0.1245 0.0265"/>
+          <mesh filename="file://$(find reachy_description)/meshes/R2B_head.dae"/>
         </geometry>
-	<material name="camblack"/>
       </visual>
       <collision>
-	<origin xyz="0.0075 0.0 0.085" rpy="0.0 0.0 0.0"/>
+	<origin xyz="0.0 0.0 0.05" rpy="0.0 0.0 0.0"/>
         <geometry>
-	  <box size="0.015 0.1245 0.0265"/>
+	  <box size="0.12 0.162 0.1"/>
         </geometry>
       </collision>
     </link>
     <link name="head_base">
-      <visual name="">
-        <origin xyz="0.00 0.0 0.0425" rpy="0.0 0.0 0.0"/>
-        <geometry>
-	  <cylinder length="0.07" radius="0.0225"/>
-        </geometry>
-	<material name="neckwhite"/>
-      </visual>
     </link>
     <joint name="head_base_fixed" type="fixed">
@@ -86,5 +79,5 @@
     <joint name="head_tip_fixed" type="fixed">
       <!-- between the cameras -->
-      <origin xyz="0.030 0.022 0.085" rpy="0 0.0 0"/>
+      <origin xyz="0.057 0.0 0.056" rpy="0 0.0 0"/>
       <!-- Rotation center -->
       <!-- <origin xyz="0.0 0 0.0" rpy="0.0 0.0 0"/> -->
@@ -92,27 +85,27 @@
       <child link="head_tip" />
     </joint>
-    <link name="camera_optical_left" >
-    </link>
-    <joint name="camera_optical_left" type="fixed">
-      <!-- between the cameras -->
-      <origin xyz="0.030 0.022 0.085" rpy="-1.57 0.0 -1.57"/>
-      <!-- Rotation center -->
-      <!-- <origin xyz="0.0 0 0.0" rpy="0.0 0.0 0"/> -->
-      <parent link="head" />
-      <child link="camera_optical_left" />
-    </joint>
+    <!-- <link name="camera_optical_left" > -->
+    <!-- </link> -->
+    <!-- <joint name="camera_optical_left" type="fixed"> -->
+    <!--   <!-\- between the cameras -\-> -->
+    <!--   <!-\- <origin xyz="0.030 0.022 0.085" rpy="-1.57 0.0 -1.57"/> -\-> -->
+    <!--   <origin xyz="0.03531 0.0325 0.056" rpy="${-pi/2.0} 0 ${-pi/2.0}"/> -->
+    <!--   <!-\- Rotation center -\-> -->
+    <!--   <!-\- <origin xyz="0.0 0 0.0" rpy="0.0 0.0 0"/> -\-> -->
+    <!--   <parent link="head" /> -->
+    <!--   <child link="camera_optical_left" /> -->
+    <!-- </joint> -->
     <!-- Reachy Cameras -->
-    <xacro:if value="$(arg use_gazebo)">
       <joint name="left_cam_fixed" type="fixed">
-	<origin xyz="0.02 0.03625 0.06105" rpy="0.0 0.0  ${-camera_convergence/2.0}"/>
+	<origin xyz="0.03531 0.0325 0.056" rpy="0.0 0.0  ${-camera_convergence/2.0}"/>
 	<parent link="head" />
 	<child link="left_camera" />
       </joint>
       <link name="left_camera" >
-	<inertial>
-	  <mass value="1e-5" />
-	  <origin xyz="0 0 0" rpy="0 0 0"/>
-	  <inertia ixx="1e-6" ixy="0" ixz="0" iyy="1e-6" iyz="0" izz="1e-6" />
-	</inertial>
+	<!-- <inertial> -->
+	<!--   <mass value="1e-5" /> -->
+	<!--   <origin xyz="0 0 0" rpy="0 0 0"/> -->
+	<!--   <inertia ixx="1e-6" ixy="0" ixz="0" iyy="1e-6" iyz="0" izz="1e-6" /> -->
+	<!-- </inertial> -->
       </link>
       <link name="left_camera_optical">
@@ -127,14 +120,14 @@
       </joint>
       <joint name="right_cam_fixed" type="fixed">
-	<origin xyz="0.02 -0.03625 0.06105" rpy="0.0 0.0 ${camera_convergence/2.0}"/>
+	<origin xyz="0.03531 -0.0325 0.056" rpy="0.0 0.0 ${camera_convergence/2.0}"/>
 	<parent link="head" />
 	<child link="right_camera" />
       </joint>
       <link name="right_camera" >
-	<inertial>
-	  <mass value="1e-5" />
-	  <origin xyz="0 0 0" rpy="0 0 0"/>
-	  <inertia ixx="1e-6" ixy="0" ixz="0" iyy="1e-6" iyz="0" izz="1e-6" />
-	</inertial>
+	<!-- <inertial> -->
+	<!--   <mass value="1e-5" /> -->
+	<!--   <origin xyz="0 0 0" rpy="0 0 0"/> -->
+	<!--   <inertia ixx="1e-6" ixy="0" ixz="0" iyy="1e-6" iyz="0" izz="1e-6" /> -->
+	<!-- </inertial> -->
       </link>
       <link name="right_camera_optical">
@@ -145,7 +138,9 @@
              originating from -->
 	<origin xyz="0 0 0" rpy="${-pi/2.0} 0 ${-pi/2.0}"/>
+	<!-- <origin xyz="0.03531 -0.0325 0.056" rpy="${-pi/2.0} 0 ${-pi/2.0}"/> -->
 	<parent link="right_camera"/>
 	<child link="right_camera_optical"/>
       </joint>
+    <xacro:if value="$(arg use_gazebo)">
       <gazebo reference="left_camera">
 	<!-- <link name="left_camera"> -->
@@ -247,64 +242,64 @@
         </sensor>
       </gazebo>
-      <link name="depth_camera_link" >
-	<inertial>
-	  <mass value="1e-5" />
-	  <origin xyz="0 0 0" rpy="0 0 0"/>
-	  <inertia ixx="1e-6" ixy="0" ixz="0" iyy="1e-6" iyz="0" izz="1e-6" />
-	</inertial>
-      </link>
-      <joint name="depth_cam_fixed" type="fixed">
-	<origin xyz="0.02 0 0.06105" rpy="0.0 0.0 0"/>
-	<parent link="head" />
-	<child link="depth_camera_link" />
-      </joint>
-      <link name="depth_camera_optical">
-      </link>
-      <joint name="depth_camera_optical_joint" type="fixed">
-	<!-- these values have to be these values otherwise the gazebo camera
-             image won't be aligned properly with the frame it is supposedly
-             originating from -->
-	<origin xyz="0 0 0" rpy="${-pi/2.0} 0 ${-pi/2.0}"/>
-	<parent link="depth_camera_link"/>
-	<child link="depth_camera_optical"/>
-      </joint>
-      <xacro:if value="$(arg depth_camera)">
-	<gazebo reference="depth_camera_link">
-	  <sensor name="depth_camera" type="depth">
-            <always_on>true</always_on>
-            <update_rate>15</update_rate>
-            <pose>0 0 0 0 0 0</pose>
-            <camera name="realsense_depth_camera">
-              <horizontal_fov>1.46608</horizontal_fov>
-              <image>
-                <width>424</width>
-                <height>240</height>
-                <format>B8G8R8</format>
-              </image>
-              <clip>
-                <near>0.05</near>
-                <far>8</far>
-              </clip>
-            </camera>
-            <!-- https://github.com/mlherd/ros2_turtlebot3_waffle_intel_realsense -->
-            <!-- <plugin name="intel_realsense_d430_depth_driver" filename="libgazebo_ros_camera.so"> -->
-            <plugin name="intel_realsense_r200_depth_driver" filename="libgazebo_ros_camera.so">
-              <ros>
-                <namespace>depth_camera</namespace>
-                <remapping>depth_camera/image_raw:=color/image_raw</remapping>
-                <remapping>depth_camera/depth/image_raw:=depth/image_rect_raw</remapping>
-                <remapping>depth_camera/camera_info:=camera_info</remapping>
-                <remapping>depth_camera/depth/camera_info:=depth/camera_info</remapping>
-                <remapping>depth_camera/points:=depth/points</remapping>
-              </ros>
-              <camera_name>depth_camera</camera_name>
-              <frame_name>depth_camera_optical</frame_name>
-              <hack_baseline>0.07</hack_baseline>
-              <min_depth>0.05</min_depth>
-              <max_depth>8.0</max_depth>
-            </plugin>
-	  </sensor>
-	</gazebo>
-      </xacro:if>
+      <!-- <link name="depth_camera_link" > -->
+      <!-- 	<inertial> -->
+      <!-- 	  <mass value="1e-5" /> -->
+      <!-- 	  <origin xyz="0 0 0" rpy="0 0 0"/> -->
+      <!-- 	  <inertia ixx="1e-6" ixy="0" ixz="0" iyy="1e-6" iyz="0" izz="1e-6" /> -->
+      <!-- 	</inertial> -->
+      <!-- </link> -->
+      <!-- <joint name="depth_cam_fixed" type="fixed"> -->
+      <!-- 	<origin xyz="0.02 0 0.06105" rpy="0.0 0.0 0"/> -->
+      <!-- 	<parent link="head" /> -->
+      <!-- 	<child link="depth_camera_link" /> -->
+      <!-- </joint> -->
+      <!-- <link name="depth_camera_optical"> -->
+      <!-- </link> -->
+      <!-- <joint name="depth_camera_optical_joint" type="fixed"> -->
+      <!-- 	<!-\- these values have to be these values otherwise the gazebo camera -->
+      <!--        image won't be aligned properly with the frame it is supposedly -->
+      <!--        originating from -\-> -->
+      <!-- 	<origin xyz="0 0 0" rpy="${-pi/2.0} 0 ${-pi/2.0}"/> -->
+      <!-- 	<parent link="depth_camera_link"/> -->
+      <!-- 	<child link="depth_camera_optical"/> -->
+      <!-- </joint> -->
+      <!-- <xacro:if value="$(arg depth_camera)"> -->
+      <!-- 	<gazebo reference="depth_camera_link"> -->
+      <!-- 	  <sensor name="depth_camera" type="depth"> -->
+      <!--       <always_on>true</always_on> -->
+      <!--       <update_rate>15</update_rate> -->
+      <!--       <pose>0 0 0 0 0 0</pose> -->
+      <!--       <camera name="realsense_depth_camera"> -->
+      <!--         <horizontal_fov>1.46608</horizontal_fov> -->
+      <!--         <image> -->
+      <!--           <width>424</width> -->
+      <!--           <height>240</height> -->
+      <!--           <format>B8G8R8</format> -->
+      <!--         </image> -->
+      <!--         <clip> -->
+      <!--           <near>0.05</near> -->
+      <!--           <far>8</far> -->
+      <!--         </clip> -->
+      <!--       </camera> -->
+      <!--       <!-\- https://github.com/mlherd/ros2_turtlebot3_waffle_intel_realsense -\-> -->
+      <!--       <!-\- <plugin name="intel_realsense_d430_depth_driver" filename="libgazebo_ros_camera.so"> -\-> -->
+      <!--       <plugin name="intel_realsense_r200_depth_driver" filename="libgazebo_ros_camera.so"> -->
+      <!--         <ros> -->
+      <!--           <namespace>depth_camera</namespace> -->
+      <!--           <remapping>depth_camera/image_raw:=color/image_raw</remapping> -->
+      <!--           <remapping>depth_camera/depth/image_raw:=depth/image_rect_raw</remapping> -->
+      <!--           <remapping>depth_camera/camera_info:=camera_info</remapping> -->
+      <!--           <remapping>depth_camera/depth/camera_info:=depth/camera_info</remapping> -->
+      <!--           <remapping>depth_camera/points:=depth/points</remapping> -->
+      <!--         </ros> -->
+      <!--         <camera_name>depth_camera</camera_name> -->
+      <!--         <frame_name>depth_camera_optical</frame_name> -->
+      <!--         <hack_baseline>0.07</hack_baseline> -->
+      <!--         <min_depth>0.05</min_depth> -->
+      <!--         <max_depth>8.0</max_depth> -->
+      <!--       </plugin> -->
+      <!-- 	  </sensor> -->
+      <!-- 	</gazebo> -->
+      <!-- </xacro:if> -->
 </xacro:if>
 </xacro:macro>

File: reachy_description/urdf/reachy.urdf.xacro (robot description, xacro)
@@ -8,5 +8,5 @@
   <xacro:include filename="$(find pollen_generic_description)/urdf/inertial_primitives.urdf.xacro" />
   <xacro:include filename="$(find pollen_generic_description)/urdf/materials.urdf.xacro" />
-  <xacro:include filename="$(find orbita2d_description)/urdf/orbita2d.urdf.xacro" />
+  <!-- <xacro:include filename="$(find orbita2d_description)/urdf/orbita2d.urdf.xacro" /> -->
   <!-- config  -->
   <xacro:arg name="neck_config" default="$(find orbita3d_description)/config/fake.yaml" />
@@ -21,59 +21,128 @@
   <xacro:property name="arm_length" value="0.28" />
   <xacro:property name="forearm_length" value="0.28" />
+  <xacro:property name="base_height" value="0.7" />
+  <!-- <xacro:property name="base_height" value="1.1" /> -->
+  <xacro:property name="back_bar_min_length" value="0.536" />
+  <xacro:property name="back_bar_max_length" value="0.936" />
+  <xacro:property name="bar_angle" value="${radians(27.458)}" />
+  <xacro:property name="bar_triangle_base" value="0.226186" />
+  <xacro:property name="bar_small_triangle_base" value="0.13857" />
+  <xacro:property name="back_bar_length" value="0.6" />
+  <!-- <xacro:property name="front_bar_length" value="${sqrt(back_bar_length*back_bar_length+bar_triangle_base*bar_triangle_base)}" /> -->
+  <xacro:property name="front_bar_length" value="${sqrt(back_bar_length*back_bar_length+bar_small_triangle_base*bar_small_triangle_base)}" />
   <!-- MODEL PARAMETERS -->
-  <!-- <material name="torsoblack"> -->
-  <!--     <color rgba="0.5 0.5 0.5 1.0"/> -->
-  <!-- </material> -->
+  <!-- <link name="world" /> -->
+  <!-- <joint name="world_joint" type="fixed"> -->
+  <!--   <origin xyz="0 0 1.0" rpy="0 0 0" /> -->
+  <!--   <parent link="world" /> -->
+  <!--   <child link="torso" /> -->
+  <!-- </joint> -->
   <link name="world" />
   <joint name="world_joint" type="fixed">
     <origin xyz="0 0 1.0" rpy="0 0 0" />
     <parent link="world" />
-    <child link="torso" />
-  </joint>
+    <child link="base_link" />
+  </joint>
+<link name="base_link">
+	<visual>
+	  <origin xyz="0 0 0" rpy="0 0 0"/>
+	  <geometry>
+	    <!-- <cylinder radius="0.1" length="0.1"/> -->
+	    <mesh filename="package://reachy_description/meshes/zuuu.dae" />
+	  </geometry>
+	</visual>
+	<!-- <collision> -->
+	<!--   <origin xyz="0 0 0" rpy="0 0 0"/> -->
+	<!--   <geometry> -->
+	<!--     <cylinder radius="0.1" length="0.1"/> -->
+	<!--   </geometry> -->
+	<!-- </collision> -->
+	<!-- <inertial> -->
+	<!--   <origin xyz="0 0 0" rpy="0 0 0"/> -->
+	<!--   <mass value="1"/> -->
+	<!--   <inertia ixx="0.1" ixy="0" ixz="0" iyy="0.1" iyz="0" izz="0.1"/> -->
+	<!-- </inertial> -->
+</link>
+<!-- <joint name="base_link_joint" type="fixed"> -->
+<!-- 	<origin xyz="1 0 0" rpy="0 0 0"/> -->
+<!-- 	<parent link="world"/> -->
+<!-- 	<child link="base_link"/> -->
+<!-- </joint> -->
+<link name="back_bar">
+	<visual>
+	  <origin xyz="0 0 ${back_bar_length/2}" rpy="0 0 0"/>
+	  <geometry>
+	    <box size="0.04 0.04 ${back_bar_length}"/>
+	  </geometry>
+	</visual>
+</link>
+<link name="left_bar">
+	<visual>
+	  <origin xyz="0.0 0 ${front_bar_length/2}" rpy="0 0 0"/>
+	  <geometry>
+	    <box size="0.04 0.04 ${front_bar_length}"/>
+	  </geometry>
+	</visual>
+</link>
+<link name="right_bar">
+	<visual>
+	  <origin xyz="0.0 0 ${front_bar_length/2}" rpy="0 0 0"/>
+	  <geometry>
+	    <box size="0.04 0.04 ${front_bar_length}"/>
+	  </geometry>
+	</visual>
+</link>
+<joint name="back_bar_joint" type="fixed">
+	<origin xyz="-0.122 0 0.057" rpy="0 0 0"/>
+	<parent link="base_link"/>
+	<child link="back_bar"/>
+</joint>
+<joint name="left_bar_joint" type="fixed">
+	<!-- <origin xyz="0.203 0.11718 0.01" rpy="0 ${-pi/2+atan2(back_bar_length,bar_small_triangle_base)} ${bar_angle}"/> -->
+	<origin xyz="0.080966 0.11718 0.057" rpy="0 ${-pi/2+atan2(back_bar_length,bar_small_triangle_base)} ${bar_angle}"/>
+	<parent link="base_link"/>
+	<child link="left_bar"/>
+</joint>
+<joint name="right_bar_joint" type="fixed">
+	<!-- <origin xyz="0.203 -0.11718 0.01" rpy="0 ${-pi/2+atan2(back_bar_length,bar_small_triangle_base)} ${-bar_angle}"/> -->
+	<origin xyz="0.080966 -0.11718 0.057" rpy="0 ${-pi/2+atan2(back_bar_length,bar_small_triangle_base)} ${-bar_angle}"/>
+	<parent link="base_link"/>
+	<child link="right_bar"/>
+</joint>
   <!-- TORSO -->
   <link name="torso">
-    <xacro:if value="${base_collision}">
-      <collision>
-        <origin xyz="-0.05 0 -0.05" rpy="0 0.0 0" />
-        <geometry>
-          <box size="0.1 0.2 0.22" />
-        </geometry>
-        <!-- <origin xyz="0 0 -0.5" rpy="0 0 0"/> -->
-        <!-- <geometry> -->
-        <!--   <cylinder length="1" radius="0.03"/> -->
-        <!-- </geometry> -->
-      </collision>
-      <collision>
-        <origin xyz="-0.15 0 -0.5" rpy="0 0 0" />
-        <geometry>
-          <cylinder length="1" radius="0.03" />
-        </geometry>
-      </collision>
-    </xacro:if>
-    <xacro:if value="${base_visual}">
-      <visual>
-        <origin xyz="-0.05 0 -0.05" rpy="0 0.0 0" />
-        <geometry>
-          <box size="0.1 0.2 0.22" />
-        </geometry>
-        <!-- <material name="torsoblack"/> -->
-        <xacro:torsoblack />
-      </visual>
-      <visual>
-        <origin xyz="-0.15 0 -0.5" rpy="0 0 0" />
-        <geometry>
-          <cylinder length="1" radius="0.03" />
-        </geometry>
-        <xacro:torsoblack />
-      </visual>
-    </xacro:if>
-    <xacro:inertial_cuboid mass="10" xyz="0 0 0.5" rpy="0 0 0" x_length="0.05" y_length="0.05"
-      z_length="1" />
+    <visual>
+      <origin xyz="0 0 0 " rpy="0 0 0"/>
+      <geometry>
+	<!-- <mesh filename="package://reachy_description/meshes/Torso.dae" /> -->
+	<mesh filename="package://reachy_description/meshes/Torso_visual_simplify.dae" />
+	<!-- <mesh filename="package://reachy_description/meshes/Torso_nobedrock_nocam.dae" /> -->
+      </geometry>
+    </visual>
+    <inertial>
+      <origin xyz="-0.098614 -0.000471 -0.018363" rpy="0 0 0"/>
+      <mass value="6.314"/>
+      <inertia ixx="0.07397673" ixy="-4.624e-4" ixz="-0.00175905"
+	       iyx="-0.00046237" iyy="0.04454533" iyz="0.00008675"
+	       izx="-0.00175905" izy="0.00008675" izz="0.05494939"/>
+    </inertial>
+    <collision>
+      <origin xyz="0 0 0 " rpy="0 0 0"/>
+      <geometry>
+	<!-- <mesh filename="package://reachy_description/meshes/Torso_convex.dae" /> -->
+	<mesh filename="package://reachy_description/meshes/Torso_double_convex_simplify.dae" />
+      </geometry>
+    </collision>
   </link>
-  <gazebo reference="torso">
-    <material>Gazebo/Black</material>
-    <static>true</static>
-  </gazebo>
-  <!-- TORSO -->
+  <joint name="torso_base" type="fixed">
+    <origin xyz="0.1265 0 ${0.2+back_bar_length}" rpy="0 0 0" />
+    <parent link="back_bar" />
+    <child link="torso" />
+  </joint>
+  <!-- <gazebo reference="torso"> -->
+  <!--   <!-\- <material>Gazebo/Black</material> -\-> -->
+  <!--   <static>true</static> -->
+  <!-- </gazebo> -->
+  <!-- Head -->
   <xacro:head
     parent="torso"
@@ -93,4 +162,16 @@
     config_file="$(arg left_arm_config)"
   />
+  <link name="sr_cam_l_frame"/>
+  <joint name="sr_cam_l_frame_joint" type="fixed">
+    <origin xyz="0.002597 0.009989 0.038089" rpy="${radians(-48.0-90.0)} 0.0 ${-pi/2}"/>
+    <parent link="torso"/>
+    <child link="sr_cam_l_frame"/>
+  </joint>
+  <link name="sr_cam_r_frame"/>
+  <joint name="sr_cam_r_frame_joint" type="fixed">
+    <origin xyz="0.002597 -0.009989 0.038089" rpy="${radians(-48.0-90.0)} 0.0 ${-pi/2}"/>
+    <parent link="torso"/>
+    <child link="sr_cam_r_frame"/>
+  </joint>
   <!-- <link name="r_wrist_cam_frame"/> -->
   <!-- <joint name="r_wrist_cam_frame_joint" type="fixed"> -->
