Commit message: meshes

File: reachy_description/urdf/head.urdf.xacro (robot description, xacro)
@@ -7,5 +7,6 @@
   <xacro:property name="neck_radius" value="0.03"/>
   <xacro:property name="neck_mass" value="0.5"/>
-  <xacro:property name="neck_offset_x" value="-0.0465"/>
+  <!-- <xacro:property name="neck_offset_x" value="-0.0465"/> -->
+  <xacro:property name="neck_offset_x" value="0.0"/>
   <xacro:property name="neck_offset_y" value="0"/>
   <xacro:property name="neck_offset_z" value="0.125"/>
@@ -44,11 +45,14 @@
         <origin xyz="0.00 0.0 0.0" rpy="0.0 0.0 0.0"/>
         <geometry>
-          <mesh filename="file://$(find reachy_description)/meshes/R2B_head.dae"/>
+          <!-- <mesh filename="file://$(find reachy_description)/meshes/R2B_head.dae"/> -->
+          <mesh filename="file://$(find reachy_description)/meshes/head_visual.dae"/>
         </geometry>
       </visual>
       <collision>
-	<origin xyz="0.0 0.0 0.05" rpy="0.0 0.0 0.0"/>
+	<!-- <origin xyz="0.0 0.0 0.05" rpy="0.0 0.0 0.0"/> -->
+	<origin xyz="0.0 0.0 0.0" rpy="0.0 0.0 0.0"/>
         <geometry>
-	  <box size="0.12 0.162 0.1"/>
+	  <!-- <box size="0.12 0.162 0.1"/> -->
+          <mesh filename="file://$(find reachy_description)/meshes/head_collider.dae"/>
         </geometry>
       </collision>

File: reachy_description/urdf/reachy.urdf.xacro (robot description, xacro)
@@ -28,5 +28,11 @@
   <xacro:property name="bar_triangle_base" value="0.226186" />
   <xacro:property name="bar_small_triangle_base" value="0.13857" />
-  <xacro:property name="back_bar_length" value="0.6" />
+  <xacro:property name="back_bar_length" value="0.720" />
+  <xacro:property name="back_bar_z" value="0.164" />
+  <xacro:property name="back_bar_x" value="-0.122" />
+  <xacro:property name="left_bar_x" value="0.080966" />
+  <xacro:property name="left_bar_y" value="0.117182" />
+  <xacro:property name="right_bar_x" value="0.080966" />
+  <xacro:property name="right_bar_y" value="-0.117182" />
   <!-- <xacro:property name="front_bar_length" value="${sqrt(back_bar_length*back_bar_length+bar_triangle_base*bar_triangle_base)}" /> -->
   <xacro:property name="front_bar_length" value="${sqrt(back_bar_length*back_bar_length+bar_small_triangle_base*bar_small_triangle_base)}" />
@@ -40,27 +46,31 @@
   <link name="world" />
   <joint name="world_joint" type="fixed">
-    <origin xyz="0 0 1.0" rpy="0 0 0" />
+    <origin xyz="0 0 0.0" rpy="0 0 0" />
     <parent link="world" />
     <child link="base_link" />
   </joint>
-<link name="base_link">
+  <link name="base_link">
 	<visual>
 	  <origin xyz="0 0 0" rpy="0 0 0"/>
 	  <geometry>
 	    <!-- <cylinder radius="0.1" length="0.1"/> -->
-	    <mesh filename="package://reachy_description/meshes/zuuu.dae" />
-	  </geometry>
-	</visual>
-	<!-- <collision> -->
-	<!--   <origin xyz="0 0 0" rpy="0 0 0"/> -->
-	<!--   <geometry> -->
-	<!--     <cylinder radius="0.1" length="0.1"/> -->
-	<!--   </geometry> -->
-	<!-- </collision> -->
-	<!-- <inertial> -->
-	<!--   <origin xyz="0 0 0" rpy="0 0 0"/> -->
-	<!--   <mass value="1"/> -->
-	<!--   <inertia ixx="0.1" ixy="0" ixz="0" iyy="0.1" iyz="0" izz="0.1"/> -->
-	<!-- </inertial> -->
+	    <!-- <mesh filename="package://reachy_description/meshes/zuuu.dae" /> -->
+	    <mesh filename="package://reachy_description/meshes/mobile_base_visual.dae" />
+	  </geometry>
+	  <xacro:reachy_grey/>
+	</visual>
+	<collision>
+	  <origin xyz="0 0 0.13045" rpy="0 0 0"/>
+	  <geometry>
+	    <cylinder radius="0.245" length="0.2609"/>
+	  </geometry>
+	</collision>
+	<inertial>
+      <origin xyz="0.008 -0.00048 0.112" rpy="0 0 0"/>
+      <mass value="24.0"/>
+      <inertia ixx="0.40791094" ixy="-0.00167148" ixz="-0.00178789"
+	       iyx="-0.00167148" iyy="0.4236827" iyz="0.00026596"
+	       izx="-0.00178789" izy="0.00026596" izz="0.70990763"/>
+    </inertial>
 </link>
 <!-- <joint name="base_link_joint" type="fixed"> -->
@@ -75,5 +85,12 @@
 	    <box size="0.04 0.04 ${back_bar_length}"/>
 	  </geometry>
-	</visual>
+	  <xacro:reachy_grey/>
+	</visual>
+	<collision>
+	  <origin xyz="0 0 ${back_bar_length/2}" rpy="0 0 0"/>
+	  <geometry>
+	    <box size="0.04 0.04 ${back_bar_length}"/>
+	  </geometry>
+	</collision>
 </link>
 <link name="left_bar">
@@ -83,5 +100,12 @@
 	    <box size="0.04 0.04 ${front_bar_length}"/>
 	  </geometry>
-	</visual>
+	  <xacro:reachy_grey/>
+	</visual>
+	<collision>
+	  <origin xyz="0.0 0 ${front_bar_length/2}" rpy="0 0 0"/>
+	  <geometry>
+	    <box size="0.04 0.04 ${front_bar_length}"/>
+	  </geometry>
+	</collision>
 </link>
 <link name="right_bar">
@@ -91,20 +115,28 @@
 	    <box size="0.04 0.04 ${front_bar_length}"/>
 	  </geometry>
-	</visual>
+	  <xacro:reachy_grey/>
+	</visual>
+	<collision>
+	  <origin xyz="0.0 0 ${front_bar_length/2}" rpy="0 0 0"/>
+	  <geometry>
+	    <box size="0.04 0.04 ${front_bar_length}"/>
+	  </geometry>
+	</collision>
 </link>
 <joint name="back_bar_joint" type="fixed">
-	<origin xyz="-0.122 0 0.057" rpy="0 0 0"/>
+	<!-- <origin xyz="-0.122 0 0.057" rpy="0 0 0"/> -->
+	<origin xyz="${back_bar_x} 0 ${back_bar_z}" rpy="0 0 0"/>
 	<parent link="base_link"/>
 	<child link="back_bar"/>
 </joint>
 <joint name="left_bar_joint" type="fixed">
-	<!-- <origin xyz="0.203 0.11718 0.01" rpy="0 ${-pi/2+atan2(back_bar_length,bar_small_triangle_base)} ${bar_angle}"/> -->
-	<origin xyz="0.080966 0.11718 0.057" rpy="0 ${-pi/2+atan2(back_bar_length,bar_small_triangle_base)} ${bar_angle}"/>
+	<!-- <origin xyz="0.080966 0.11718 0.057" rpy="0 ${-pi/2+atan2(back_bar_length,bar_small_triangle_base)} ${bar_angle}"/> -->
+	<origin xyz="${left_bar_x} ${left_bar_y} ${back_bar_z}" rpy="0 ${-pi/2+atan2(back_bar_length,bar_small_triangle_base)} ${bar_angle}"/>
 	<parent link="base_link"/>
 	<child link="left_bar"/>
 </joint>
 <joint name="right_bar_joint" type="fixed">
-	<!-- <origin xyz="0.203 -0.11718 0.01" rpy="0 ${-pi/2+atan2(back_bar_length,bar_small_triangle_base)} ${-bar_angle}"/> -->
-	<origin xyz="0.080966 -0.11718 0.057" rpy="0 ${-pi/2+atan2(back_bar_length,bar_small_triangle_base)} ${-bar_angle}"/>
+	<!-- <origin xyz="0.080966 -0.11718 0.057" rpy="0 ${-pi/2+atan2(back_bar_length,bar_small_triangle_base)} ${-bar_angle}"/> -->
+	<origin xyz="${right_bar_x} ${right_bar_y} ${back_bar_z}" rpy="0 ${-pi/2+atan2(back_bar_length,bar_small_triangle_base)} ${-bar_angle}"/>
 	<parent link="base_link"/>
 	<child link="right_bar"/>
@@ -116,10 +148,11 @@
       <geometry>
 	<!-- <mesh filename="package://reachy_description/meshes/Torso.dae" /> -->
-	<mesh filename="package://reachy_description/meshes/Torso_visual_simplify.dae" />
+	<mesh filename="package://reachy_description/meshes/torso_visual_high.dae" />
 	<!-- <mesh filename="package://reachy_description/meshes/Torso_nobedrock_nocam.dae" /> -->
       </geometry>
     </visual>
     <inertial>
-      <origin xyz="-0.098614 -0.000471 -0.018363" rpy="0 0 0"/>
+      <!-- <origin xyz="-0.098614 -0.000471 -0.018363" rpy="0 0 0"/> -->
+      <origin xyz="-0.051614 -0.000471 -0.018363" rpy="0 0 0"/>
       <mass value="6.314"/>
       <inertia ixx="0.07397673" ixy="-4.624e-4" ixz="-0.00175905"
@@ -131,12 +164,20 @@
       <geometry>
 	<!-- <mesh filename="package://reachy_description/meshes/Torso_convex.dae" /> -->
-	<mesh filename="package://reachy_description/meshes/Torso_double_convex_simplify.dae" />
+	<!-- <mesh filename="package://reachy_description/meshes/torso_collider.dae" /> -->
+	<mesh filename="package://reachy_description/meshes/torso_collider_no_cone.dae" />
       </geometry>
     </collision>
   </link>
   <joint name="torso_base" type="fixed">
-    <origin xyz="0.1265 0 ${0.2+back_bar_length}" rpy="0 0 0" />
+    <origin xyz="0.0768 0 ${0.2+back_bar_length}" rpy="0 0 0" />
     <parent link="back_bar" />
     <child link="torso" />
+  </joint>
+  <link name="logo">
+  </link>
+  <joint name="logo_joint" type="fixed">
+    <origin xyz="0.047 0 0.0" rpy="0 0 0" />
+    <parent link="torso" />
+    <child link="logo" />
   </joint>
   <!-- <gazebo reference="torso"> -->
