Commit message: Gazebo support, modify simulated cameras

File: reachy_description/urdf/head.urdf.xacro (robot description, xacro)
@@ -193,9 +193,9 @@
           <plugin name="left_camera_controller" filename="libgazebo_ros_camera.so">
               <ros>
-                <namespace>/</namespace>
+                <namespace>/teleop_camera</namespace>
                 <remapping>image_raw:=image_raw</remapping>
                 <remapping>camera_info:=camera_info</remapping>
               </ros>
-              <camera_name>teleop_camera/left_image</camera_name>
+              <camera_name>left_image</camera_name>
             <!-- <ros> -->
             <!--   <namespace>custom_ns</namespace> -->
@@ -242,9 +242,9 @@
           <plugin name="right_camera_controller" filename="libgazebo_ros_camera.so">
               <ros>
-                <namespace>/</namespace>
+                <namespace>/teleop_camera</namespace>
                 <remapping>image_raw:=image_raw</remapping>
                 <remapping>camera_info:=camera_info</remapping>
               </ros>
-              <camera_name>teleop_camera/right_image</camera_name>
+              <camera_name>right_image</camera_name>
             <!-- <ros> -->
             <!--   <namespace>custom_ns</namespace> -->

File: reachy_description/urdf/reachy.urdf.xacro (robot description, xacro)
@@ -227,5 +227,5 @@
     config_file="$(arg left_arm_config)"
   />
-  <link name="sr_cam_l_optical">
+  <link name="depth_cam_l_optical">
     <inertial>
       <origin xyz="0.0 0.0 0.0" rpy="0.0 0.0 0.0"/>
@@ -234,5 +234,5 @@
     </inertial>
   </link>
-  <link name="sr_cam_l_frame">
+  <link name="depth_cam_l_frame">
     <inertial>
       <origin xyz="0.0 0.0 0.0" rpy="0.0 0.0 0.0"/>
@@ -241,15 +241,15 @@
     </inertial>
   </link>
-  <joint name="sr_cam_l_optical_joint" type="fixed">
+  <joint name="depth_cam_l_optical_joint" type="fixed">
     <origin xyz="0.002597 0.009989 0.038089" rpy="${radians(-48.0-90.0)} 0.0 ${-pi/2}"/>
     <parent link="logo"/>
-    <child link="sr_cam_l_optical"/>
-  </joint>
-  <joint name="sr_cam_l_frame_joint" type="fixed">
+    <child link="depth_cam_l_optical"/>
+  </joint>
+  <joint name="depth_cam_l_frame_joint" type="fixed">
     <origin xyz="0.002597 0.009989 0.038089" rpy="0.0 ${radians(48.0)} 0.0"/>
     <parent link="logo"/>
-    <child link="sr_cam_l_frame"/>
-  </joint>
-  <link name="sr_cam_r_optical">
+    <child link="depth_cam_l_frame"/>
+  </joint>
+  <link name="depth_cam_r_optical">
             <inertial>
                 <origin xyz="0.0 0.0 0.0" rpy="0.0 0.0 0.0"/>
@@ -258,5 +258,5 @@
             </inertial>
   </link>
-  <link name="sr_cam_r_frame">
+  <link name="depth_cam_r_frame">
             <inertial>
                 <origin xyz="0.0 0.0 0.0" rpy="0.0 0.0 0.0"/>
@@ -265,15 +265,15 @@
             </inertial>
   </link>
-  <joint name="sr_cam_r_optical_joint" type="fixed">
+  <joint name="depth_cam_r_optical_joint" type="fixed">
     <origin xyz="0.002597 -0.009989 0.038089" rpy="${radians(-48.0-90.0)} 0.0 ${-pi/2}"/>
     <parent link="logo"/>
-    <child link="sr_cam_r_optical"/>
-  </joint>
-  <joint name="sr_cam_r_frame_joint" type="fixed">
+    <child link="depth_cam_r_optical"/>
+  </joint>
+  <joint name="depth_cam_r_frame_joint" type="fixed">
     <origin xyz="0.002597 -0.009989 0.038089" rpy="0.0 ${radians(48.0)} 0.0 "/>
     <parent link="logo"/>
-    <child link="sr_cam_r_frame"/>
-  </joint>
-      <gazebo reference="sr_cam_l_frame">
+    <child link="depth_cam_r_frame"/>
+  </joint>
+      <gazebo reference="depth_cam_l_frame">
 	<!-- <link name="left_camera"> -->
 	<sensor type="camera" name="left_camera">
@@ -282,5 +282,5 @@
           <!-- Set update_rate only sensor, not on plugin -->
           <update_rate>30</update_rate>
-          <camera name="sr_cam_l">
+          <camera name="depth_cam_l">
             <horizontal_fov>${77.0*pi/180}</horizontal_fov>
             <image>
@@ -304,11 +304,12 @@
           </camera>
           <!-- Use camera, not camera_triggered -->
-          <plugin name="sr_left_camera_controller" filename="libgazebo_ros_camera.so">
+          <plugin name="depth_left_camera_controller" filename="libgazebo_ros_camera.so">
               <ros>
-                <namespace>/</namespace>
-                <remapping>image_raw:=image_raw</remapping>
-                <remapping>camera_info:=camera_info</remapping>
+                <namespace>camera</namespace>
+                <remapping>left/image_raw:=/camera/left/color/image_raw</remapping>
+                <remapping>left/image_raw/compressed:=/camera/left/color/image_raw/compressed</remapping>
+                <remapping>left/camera_info:=/camera/left/color/camera_info</remapping>
               </ros>
-              <camera_name>sr_left_image</camera_name>
+              <camera_name>left</camera_name>
             <!-- <ros> -->
             <!--   <namespace>custom_ns</namespace> -->
@@ -319,5 +320,5 @@
             <!-- <camera_name>left_camera</camera_name> -->
             <!-- Set TF frame name. If empty, defaults to link name (i.e. "link_name") -->
-            <frame_name>sr_cam_l_optical</frame_name>
+            <frame_name>depth_cam_l_optical</frame_name>
             <hack_baseline>0.07</hack_baseline>
             <!-- No need to repeat distortion parameters or to set autoDistortion -->
@@ -325,5 +326,5 @@
         </sensor>
       </gazebo>
-      <gazebo reference="sr_cam_r_frame">
+      <gazebo reference="depth_cam_r_frame">
 	<!-- <link name="left_camera"> -->
 	<sensor type="camera" name="right_camera">
@@ -332,5 +333,5 @@
           <!-- Set update_rate only sensor, not on plugin -->
           <update_rate>30</update_rate>
-          <camera name="sr_cam_r">
+          <camera name="depth_cam_r">
             <horizontal_fov>${77.0*pi/180}</horizontal_fov>
             <image>
@@ -354,11 +355,14 @@
           </camera>
           <!-- Use camera, not camera_triggered -->
-          <plugin name="sr_right_camera_controller" filename="libgazebo_ros_camera.so">
+          <plugin name="depth_right_camera_controller" filename="libgazebo_ros_camera.so">
               <ros>
-                <namespace>/</namespace>
-                <remapping>image_raw:=image_raw</remapping>
-                <remapping>camera_info:=camera_info</remapping>
+                <namespace>camera</namespace>
+                <remapping>right/image_raw:=/camera/right/color/image_raw</remapping>
+                <remapping>right/image_raw/compressed:=/camera/right/color/image_raw/compressed</remapping>
+                <remapping>right/camera_info:=/camera/right/color/camera_info</remapping>
+                <!-- <remapping>image_raw:=image_raw</remapping> -->
+                <!-- <remapping>camera_info:=camera_info</remapping> -->
               </ros>
-              <camera_name>sr_right_image</camera_name>
+              <camera_name>right</camera_name>
             <!-- <ros> -->
             <!--   <namespace>custom_ns</namespace> -->
@@ -369,5 +373,5 @@
             <!-- <camera_name>left_camera</camera_name> -->
             <!-- Set TF frame name. If empty, defaults to link name (i.e. "link_name") -->
-            <frame_name>sr_cam_r_optical</frame_name>
+            <frame_name>depth_cam_r_optical</frame_name>
             <hack_baseline>0.07</hack_baseline>
             <!-- No need to repeat distortion parameters or to set autoDistortion -->
@@ -375,8 +379,8 @@
         </sensor>
       </gazebo>
-	<gazebo reference="sr_cam_l_frame">
+	<gazebo reference="depth_cam_l_frame">
 	  <sensor name="depth_camera" type="depth">
             <always_on>true</always_on>
-            <update_rate>15</update_rate>
+            <update_rate>30</update_rate>
             <pose>0 0 0 0 0 0</pose>
             <camera name="depth_camera">
@@ -401,13 +405,14 @@
             <plugin name="depth_driver" filename="libgazebo_ros_camera.so">
               <ros>
-                <namespace>camera</namespace>
-                <remapping>camera/image_raw:=color/image_raw</remapping>
-                <remapping>camera/depth/image_raw:=depth/image_rect_raw</remapping>
-                <remapping>camera/camera_info:=camera_info</remapping>
-                <remapping>camera/depth/camera_info:=depth/camera_info</remapping>
-                <remapping>camera/points:=depth/points</remapping>
+                <namespace>/</namespace>
+                <remapping>camera/image_raw:=camera/color/image_raw</remapping>
+                <remapping>camera/image_raw/compressed:=camera/color/image_raw/compressed</remapping>
+                <remapping>camera/camera_info:=camera/color/camera_info</remapping>
+                <remapping>camera/image_depth:=camera/depth/image_raw</remapping>
+                <remapping>camera/camera_info_depth:=camera/depth/camera_info</remapping>
+                <remapping>camera/points:=camera/depth/points</remapping>
               </ros>
-              <camera_name>depth_camera</camera_name>
-              <frame_name>sr_cam_l_optical</frame_name>
+              <camera_name>camera</camera_name>
+              <frame_name>depth_cam_l_optical</frame_name>
               <hack_baseline>0.07</hack_baseline>
               <min_depth>0.05</min_depth>

Commit message: works in fake

File: reachy_description/urdf/head.urdf.xacro (robot description, xacro)
@@ -14,4 +14,5 @@
   <xacro:property name="neck_offset_yaw" value="0.0"/>
   <xacro:include filename="$(find orbita3d_description)/urdf/orbita3d.urdf.xacro"/>
+  <xacro:include filename="$(find dynamixel_description)/ros2_control/dynamixel.ros2_control.xacro"/>
     <material name="camblack">
         <color rgba="0.2 0.2 0.2 1"/>
@@ -20,5 +21,5 @@
         <color rgba="0.9 0.9 0.9 1"/>
     </material>
-  <xacro:macro name="head" params="parent damping friction neck_config">
+  <xacro:macro name="head" params="parent damping friction neck_config antenna_config">
     <!-- xyz="${neck_offset_x} ${neck_offset_y} ${neck_offset_z}" rpy="${pi} ${neck_offset_pitch} ${neck_offset_yaw}" -->
   <xacro:orbita3d
@@ -99,15 +100,55 @@
       <child link="head_tip" />
     </joint>
-    <!-- <link name="camera_optical_left" > -->
-    <!-- </link> -->
-    <!-- <joint name="camera_optical_left" type="fixed"> -->
-    <!--   <!-\- between the cameras -\-> -->
-    <!--   <!-\- <origin xyz="0.030 0.022 0.085" rpy="-1.57 0.0 -1.57"/> -\-> -->
-    <!--   <origin xyz="0.03531 0.0325 0.056" rpy="${-pi/2.0} 0 ${-pi/2.0}"/> -->
-    <!--   <!-\- Rotation center -\-> -->
-    <!--   <!-\- <origin xyz="0.0 0 0.0" rpy="0.0 0.0 0"/> -\-> -->
-    <!--   <parent link="head" /> -->
-    <!--   <child link="camera_optical_left" /> -->
-    <!-- </joint> -->
+    <!-- test antennas -->
+    <link name="antenna_left" >
+      <inertial>
+	<origin xyz="0.0 0.0 0.0" rpy="0.0 0.0 0.0"/>
+	<mass value="0.001"/>
+	<inertia ixx="1.0e-6" ixy="1.0e-8" ixz="1.0e-8" iyy="1.0e-6" iyz="1.0e-8" izz="1.0e-6"/>
+      </inertial>
+      <!-- cylinder geometry -->
+      <visual>
+	<origin xyz="0 0 0" rpy="0 0 0"/>
+	<geometry>
+	  <cylinder length="0.1" radius="0.005"/>
+	</geometry>
+	<material name="neckwhite"/>
+      </visual>
+    </link>
+    <!-- revolute joint -->
+    <joint name="antenna_left_joint" type="revolute">
+      <origin xyz="0.0 0.1 0.1" rpy="0 0.0 0"/>
+      <parent link="head" />
+      <child link="antenna_left" />
+      <axis xyz="0 1 0"/>
+      <limit effort="0.0" velocity="0.0" lower="-0.5" upper="0.5"/>
+    </joint>
+    <link name="antenna_right" >
+      <inertial>
+	<origin xyz="0.0 0.0 0.0" rpy="0.0 0.0 0.0"/>
+	<mass value="0.001"/>
+	<inertia ixx="1.0e-6" ixy="1.0e-8" ixz="1.0e-8" iyy="1.0e-6" iyz="1.0e-8" izz="1.0e-6"/>
+      </inertial>
+      <!-- cylinder geometry -->
+      <visual>
+	<origin xyz="0 0 0" rpy="0 0 0"/>
+	<geometry>
+	  <cylinder length="0.1" radius="0.005"/>
+	</geometry>
+	<material name="neckwhite"/>
+      </visual>
+    </link>
+    <!-- revolute joint -->
+    <joint name="antenna_right_joint" type="revolute">
+      <origin xyz="0.0 -0.1 0.1" rpy="0 0.0 0"/>
+      <parent link="head" />
+      <child link="antenna_right" />
+      <axis xyz="0 1 0"/>
+      <limit effort="0.0" velocity="0.0" lower="-0.5" upper="0.5"/>
+    </joint>
+  <xacro:dynamixel_control
+    name="antenna"
+    config_file="${antenna_config}"
+    />
     <!-- Reachy Cameras -->
       <joint name="left_cam_fixed" type="fixed">

File: reachy_description/urdf/reachy.urdf.xacro (robot description, xacro)
@@ -31,4 +31,5 @@
   <!-- End of Zuuu mobile base -->
   <!-- config  -->
+  <xacro:arg name="antenna_config" default="$(find dynamixel_description)/config/two_fake.yaml"/>
   <xacro:arg name="neck_config" default="$(find orbita3d_description)/config/fake_neck.yaml" />
   <xacro:arg name="right_arm_config" default="$(find arm_description)/config/fake_r_arm.yaml" />
@@ -188,5 +189,5 @@
     parent="torso"
     damping="${damping}" friction="${friction}"
-    neck_config="$(arg neck_config)"
+    neck_config="$(arg neck_config)" antenna_config="$(arg antenna_config)"
   />
   <!-- RIGHT ARM -->

Commit message: move mujoco cam a bit further along to avoid seeing model

File: reachy_description/urdf/head.urdf.xacro (robot description, xacro)
@@ -199,8 +199,5 @@
     </link>
     <joint name="left_camera_optical_frame_joint" type="fixed">
-      <!-- these values have to be these values otherwise the gazebo camera
-             image won't be aligned properly with the frame it is supposedly
-             originating from -->
-      <origin xyz="0 0 0" rpy="${-pi/2.0} 0 ${-pi/2.0}" />
+      <origin xyz="0.01 0 0" rpy="${-pi/2.0} 0 ${-pi/2.0}" />
       <parent link="left_camera" />
       <child link="left_camera_optical_frame" />
@@ -232,8 +229,5 @@
     </link>
     <joint name="right_camera_optical_frame_joint" type="fixed">
-      <!-- these values have to be these values otherwise the gazebo camera
-             image won't be aligned properly with the frame it is supposedly
-             originating from -->
-      <origin xyz="0 0 0" rpy="${-pi/2.0} 0 ${-pi/2.0}" />
+      <origin xyz="0.01 0 0" rpy="${-pi/2.0} 0 ${-pi/2.0}" />
       <!-- <origin xyz="0.03531 -0.0325 0.056" rpy="${-pi/2.0} 0 ${-pi/2.0}"/> -->
       <parent link="right_camera" />

Commit message: tof mujoco joint needed

File: reachy_description/urdf/head.urdf.xacro (robot description, xacro)
@@ -248,4 +248,6 @@
     <link name="tof_camera_optical">
     </link>
+    <link name="tof_camera_optical_frame">
+    </link>
     <joint name="tof_camera_optical_joint" type="fixed">
       <!-- these values have to be these values otherwise the gazebo camera
@@ -256,4 +258,13 @@
       <parent link="tof_camera" />
       <child link="tof_camera_optical" />
+    </joint>
+    <joint name="tof_camera_optical_frame_joint" type="fixed">
+      <!-- these values have to be these values otherwise the gazebo camera
+             image won't be aligned properly with the frame it is supposedly
+             originating from -->
+      <origin xyz="0 0 0" rpy="${-pi/2.0} 0 ${-pi/2.0}" />
+      <!-- <origin xyz="0.03531 -0.0325 0.056" rpy="${-pi/2.0} 0 ${-pi/2.0}"/> -->
+      <parent link="tof_camera" />
+      <child link="tof_camera_optical_frame" />
     </joint>
     <xacro:if value="$(arg use_gazebo)">
