Commit message: Fix orbita zero.

File: reachy_description/urdf/arm.urdf.xacro (robot description, xacro)
@@ -24,5 +24,5 @@
   <xacro:property name="wrist_radius" value="0.02"/>
   <xacro:property name="wrist_mass" value="0.3"/>
-  <xacro:property name="wrist_reduction" value="4.0"/>
+  <xacro:property name="wrist_reduction" value="4.266667"/>
   <!-- ARM PARAMETERS -->
   <xacro:if value="${side == 'left'}">

File: reachy_description/urdf/head.urdf.xacro (robot description, xacro)
@@ -4,5 +4,5 @@
   <xacro:property name="camera_link" value="0.05" /> <!-- Size of square 'camera' box -->
   <xacro:property name="camera_convergence" value="0.0" /> <!-- convergence angle (rad) of the cameras. 0=parallel-->
-  <xacro:property name="neck_orbita_reduction" value="4.0"/>
+  <xacro:property name="neck_orbita_reduction" value="4.266667"/>
   <xacro:property name="neck_orbita_alpha" value="0.9424777960769379"/>
   <xacro:macro name="head" params="parent damping friction neck_orbita_serial_port neck_orbita_id neck_orbita_hardware_zero">

Commit message: Update arm.urdf.xacro

File: reachy_description/urdf/arm.urdf.xacro (robot description, xacro)
@@ -93,5 +93,5 @@
   <link name="${p}_arm_tip"/>
   <joint name="${p}_tip_joint" type="fixed">
-    <origin xyz="0 0 0.1" rpy="${pi+reflect*0.35} 0 0"/>
+    <origin xyz="0 0 0.1" rpy="${pi} 0 0"/>
     <parent link="${p}_gripper_palm_link"/>
     <child link="${p}_arm_tip"/>

Commit message: test with new orbita control

File: reachy_description/urdf/arm.urdf.xacro (robot description, xacro)
@@ -1,8 +1,13 @@
 <?xml version="1.0" ?>
 <robot xmlns:xacro="http://www.ros.org/wiki/xacro">
-<xacro:macro name="arm" params="prefix parent side damping friction shoulder_port_a shoulder_port_b shoulder_id_a shoulder_id_b elbow_port_a elbow_port_b elbow_id_a elbow_id_b wrist_port wrist_id wrist_hardware_zero gripper_port gripper_id">
-  <xacro:include filename="$(find reachy_description)/urdf/orbita.urdf.xacro"/>
-  <xacro:include filename="$(find reachy_description)/urdf/orbita2dof.urdf.xacro"/>
-  <xacro:include filename="$(find reachy_description)/urdf/smartgripper.urdf.xacro"/>
+<xacro:macro name="arm" params="prefix parent side damping friction orbita2d_shoulder_config orbita2d_elbow_config orbita3d_wrist_config">
+  <xacro:include filename="$(find orbita3d_description)/urdf/orbita3d.urdf.xacro"/>
+  <xacro:include filename="$(find orbita2d_description)/urdf/orbita2d.urdf.xacro"/>
+  <!-- <xacro:include filename="$(find reachy_description)/urdf/smartgripper.urdf.xacro"/> -->
+  <!-- <!-\- Orbita2d config -\-> -->
+  <!-- <xacro:arg name="orbita2d_shoulder_config" default="$(find orbita2d_description)/config/fake.yaml"/> -->
+  <!-- <xacro:arg name="orbita2d_elbow_config" default="$(find orbita2d_description)/config/fake.yaml"/> -->
+  <!-- <!-\- Orbita3d config -\-> -->
+  <!-- <xacro:arg name="orbita3d_wrist_config" default="$(find orbita3d_controller)/config/fake.yaml"/> -->
   <!-- ARM PARAMETERS -->
   <!-- TODO: USE REAL VALUES -->
@@ -45,5 +50,5 @@
   </xacro:if>
   <xacro:property name="p" value="${prefix}"/>
-  <xacro:orbita2dof
+  <xacro:orbita2d
     name="${p}_shoulder" parent="${parent}"
     length="${arm_length}" radius="${arm_radius}" mass="${arm_mass}"
@@ -52,13 +57,8 @@
     joint1="pitch" joint2="roll"
     joint1_min_angle="-${pi/2}" joint1_max_angle="${pi/2}"
-    joint2_min_angle="${min_shoulder_roll}" joint2_max_angle="${max_shoulder_roll}"
-    port_a="${shoulder_port_a}" port_b="${shoulder_port_b}"
-    id_a="${shoulder_id_a}" id_b="${shoulder_id_b}"
-    offset_a="0.0" offset_b="0.0"
-    ratio_a="${shoulder_ratio_a}" ratio_b="${shoulder_ratio_b}"
-    axis1_inverted="${shoulder_axis1_inverted}"
-    axis2_inverted="${shoulder_axis2_inverted}"
+    joint2_min_angle="-${pi/2}" joint2_max_angle="0.0"
+    config_file="${orbita2d_shoulder_config}"
   />
-   <xacro:orbita2dof
+   <xacro:orbita2d
     name="${p}_elbow" parent="${p}_shoulder_ball_link"
     length="${forearm_length}" radius="${forearm_radius}" mass="${forearm_mass}"
@@ -68,33 +68,25 @@
     joint1_min_angle="-${pi/2}" joint1_max_angle="${pi/2}"
     joint2_min_angle="-2.25" joint2_max_angle="0.1"
-    port_a="${elbow_port_a}" port_b="${elbow_port_b}"
-    id_a="${elbow_id_a}" id_b="${elbow_id_b}"
-    offset_a="0.0" offset_b="0.0"
-    ratio_a="${elbow_ratio_a}" ratio_b="${elbow_ratio_b}"
-    axis1_inverted="${elbow_axis1_inverted}"
-    axis2_inverted="${elbow_axis2_inverted}"
+    config_file="${orbita2d_elbow_config}"
   />
-  <xacro:orbita
+  <xacro:orbita3d
     name="${p}_wrist" parent="${p}_elbow_ball_link"
     length="${wrist_length}" radius="${wrist_radius}" mass="${wrist_mass}"
     xyz="0 0 -${forearm_length}" rpy="${pi} 0 0"
     damping="${damping}" friction="${friction}"
-    orbita_serial_port="${wrist_port}"
-    orbita_id="${wrist_id}"
-    orbita_hardware_zero="${wrist_hardware_zero}"
-    orbita_reduction="${wrist_reduction}"
+    config_file="${orbita3d_wrist_config}"
   />
-  <xacro:smartgripper
-    prefix="${p}" parent="${p}_wrist_ball_link" side="${side}"
-    damping="${damping}" friction="${friction}"
-    gripper_port="${gripper_port}"
-    gripper_id="${gripper_id}"
-  />
-  <link name="${p}_arm_tip"/>
-  <joint name="${p}_tip_joint" type="fixed">
-    <origin xyz="0 0 0.1" rpy="${pi} 0 0"/>
-    <parent link="${p}_gripper_palm_link"/>
-    <child link="${p}_arm_tip"/>
-  </joint>
+  <!-- <xacro:smartgripper -->
+  <!--   prefix="${p}" parent="${p}_wrist_ball_link" side="${side}" -->
+  <!--   damping="${damping}" friction="${friction}" -->
+  <!--   gripper_port="${gripper_port}" -->
+  <!--   gripper_id="${gripper_id}" -->
+  <!-- /> -->
+  <!-- <link name="${p}_arm_tip"/> -->
+  <!-- <joint name="${p}_tip_joint" type="fixed"> -->
+  <!--   <origin xyz="0 0 0.1" rpy="${pi} 0 0"/> -->
+  <!--   <parent link="${p}_gripper_palm_link"/> -->
+  <!--   <child link="${p}_arm_tip"/> -->
+  <!-- </joint> -->
 </xacro:macro>
 </robot>

File: reachy_description/urdf/head.urdf.xacro (robot description, xacro)
@@ -4,6 +4,13 @@
   <xacro:property name="camera_link" value="0.05" /> <!-- Size of square 'camera' box -->
   <xacro:property name="camera_convergence" value="0.0" /> <!-- convergence angle (rad) of the cameras. 0=parallel-->
-  <xacro:property name="neck_orbita_reduction" value="4.266667"/>
-  <xacro:property name="neck_orbita_alpha" value="0.9424777960769379"/>
+  <xacro:property name="neck_length" value="0.05"/>
+  <xacro:property name="neck_radius" value="0.03"/>
+  <xacro:property name="neck_mass" value="0.5"/>
+  <xacro:property name="neck_offset_x" value="-0.032893"/>
+  <xacro:property name="neck_offset_y" value="0"/>
+  <xacro:property name="neck_offset_z" value="0.110675"/>
+  <xacro:property name="neck_offset_pitch" value="0.17453293"/>
+  <xacro:property name="neck_offset_yaw" value="0.0"/>
+  <xacro:include filename="$(find orbita3d_description)/urdf/orbita3d.urdf.xacro"/>
     <material name="camblack">
         <color rgba="0.2 0.2 0.2 1"/>
@@ -12,129 +19,17 @@
         <color rgba="0.9 0.9 0.9 1"/>
     </material>
-  <xacro:macro name="head" params="parent damping friction neck_orbita_serial_port neck_orbita_id neck_orbita_hardware_zero">
-    <xacro:include filename="$(find reachy_description)/ros2_control/head.ros2_control.xacro"/>
-    <joint name="neck_roll" type="revolute">
-      <origin xyz="-0.032893 0.0 0.110675" rpy="0.0 0.17453293 0.0"/>
-      <parent link="${parent}"/>
-      <child link="head_x"/>
-      <axis xyz="1 0 0"/>
-      <limit lower="-0.8" upper="0.8" effort="10." velocity="0.0"/>
-      <dynamics damping="${damping}" friction="${friction}"/>
-    </joint>
-    <link name="head_x">
-      <inertial>
-        <origin xyz="0.0 0.0 0.0" rpy="0.0 0.0 0.0"/>
-        <mass value="0.001"/>
-        <inertia ixx="1.0e-6" ixy="1.0e-8" ixz="1.0e-8" iyy="1.0e-6" iyz="1.0e-8" izz="1.0e-6"/>
-      </inertial>
-    </link>
-    <joint name="neck_pitch" type="revolute">
-      <origin xyz="0 0 0" rpy="0.0 0.0 0.0"/>
-      <parent link="head_x"/>
-      <child link="head_y"/>
-      <axis xyz="0 1 0"/>
-      <limit lower="-0.8" upper="1.13" effort="10." velocity="0.0"/>
-      <dynamics damping="${damping}" friction="${friction}"/>
-    </joint>
-    <link name="head_y" >
-      <inertial>
-        <origin xyz="0.0 0.0 0.0" rpy="0.0 0.0 0.0"/>
-        <mass value="0.001"/>
-        <inertia ixx="1.0e-6" ixy="1.0e-8" ixz="1.0e-8" iyy="1.0e-6" iyz="1.0e-8" izz="1.0e-6"/>
-      </inertial>
-    </link>
-    <joint name="neck_yaw" type="revolute">
-      <origin xyz="0 0 0" rpy="0.0 0.0 0.0"/>
-      <parent link="head_y"/>
-      <child link="head_z"/>
-      <axis xyz="0 0 1"/>
-      <limit lower="-2.79" upper="2.79" effort="10." velocity="0.0"/>
-      <dynamics damping="${damping}" friction="${friction}"/>
-    </joint>
-    <link name="head_z">
-      <inertial>
-        <origin xyz="0.0 0.0 0.0" rpy="0.0 0.0 0.0"/>
-        <mass value="0.001"/>
-        <inertia ixx="1.0e-6" ixy="1.0e-8" ixz="1.0e-8" iyy="1.0e-6" iyz="1.0e-8" izz="1.0e-6"/>
-      </inertial>
-    </link>
+  <xacro:macro name="head" params="parent damping friction neck_config">
+  <xacro:orbita3d
+    name="neck" parent="torso"
+    length="${neck_length}" radius="${neck_radius}" mass="${neck_mass}"
+    xyz="${neck_offset_x} ${neck_offset_y} ${neck_offset_z}" rpy="0 0 ${neck_offset_yaw}"
+    damping="${damping}" friction="${friction}"
+    config_file="${neck_config}"
+  />
     <joint name="neck_fixed" type="fixed">
       <origin xyz="0 0 0" rpy="0.0 0.0 0.0"/>
-      <parent link="head_z" />
+      <parent link="neck_ball_link" />
       <child link="head" />
     </joint>
-    <!-- Fixed Orbita Arms Visuals -->
-    <!-- <joint name="neck_top" type="fixed"> -->
-    <!--   <origin xyz="0.0067 0.0 0.0478" rpy="0 0.174 0"/> -->
-    <!--   <parent link="${parent}"/> -->
-    <!--   <child link="top_neck_arm"/> -->
-    <!-- </joint> -->
-    <!-- <link name="top_neck_arm"> -->
-    <!--   <inertial> -->
-    <!--     <origin xyz="0.0 0.0 0.0" rpy="0.0 0.0 0.0"/> -->
-    <!--     <mass value="0.001"/> -->
-    <!--     <inertia ixx="1.0e-6" ixy="1.0e-8" ixz="1.0e-8" iyy="1.0e-6" iyz="1.0e-8" izz="1.0e-6"/> -->
-    <!--   </inertial> -->
-    <!--   <visual name=""> -->
-    <!--     <origin xyz="0.0 0.0 0.0" rpy="0.0 0.0 0.5236"/> -->
-    <!--     <geometry> -->
-    <!--       <mesh filename="file://$(find reachy_description)/meshes/orbita_arm.dae"/> -->
-    <!--     </geometry> -->
-    <!--   </visual> -->
-    <!--   <collision> -->
-    <!--     <origin xyz="0.0 0.0 0.0" rpy="0.0 0.0 0.0"/> -->
-    <!--     <geometry> -->
-    <!--       <cylinder length="0.0" radius="0.0" /> -->
-    <!--     </geometry> -->
-    <!--   </collision> -->
-    <!-- </link> -->
-    <!-- <joint name="neck_middle" type="fixed"> -->
-    <!--   <origin xyz="0.0067 0.0 0.0478" rpy="0 0.174 0"/> -->
-    <!--   <parent link="${parent}"/> -->
-    <!--   <child link="middle_neck_arm"/> -->
-    <!-- </joint> -->
-    <!-- <link name="middle_neck_arm"> -->
-    <!--   <inertial> -->
-    <!--     <origin xyz="0.0 0.0 0.0" rpy="0.0 0.0 0.0"/> -->
-    <!--     <mass value="0.001"/> -->
-    <!--     <inertia ixx="1.0e-6" ixy="1.0e-8" ixz="1.0e-8" iyy="1.0e-6" iyz="1.0e-8" izz="1.0e-6"/> -->
-    <!--   </inertial> -->
-    <!--   <visual name=""> -->
-    <!--     <origin xyz="0.0 0.0 0.0" rpy="0.0 0.0 2.618"/> -->
-    <!--     <geometry> -->
-    <!--       <mesh filename="file://$(find reachy_description)/meshes/orbita_arm.dae"/> -->
-    <!--     </geometry> -->
-    <!--   </visual> -->
-    <!--   <collision> -->
-    <!--     <origin xyz="0.0 0.0 0.0" rpy="0.0 0.0 0.0"/> -->
-    <!--     <geometry> -->
-    <!--       <cylinder length="0.0" radius="0.0" /> -->
-    <!--     </geometry> -->
-    <!--   </collision> -->
-    <!-- </link> -->
-    <!-- <joint name="neck_bottom" type="fixed"> -->
-    <!--   <origin xyz="0.0067 0.0 0.0478" rpy="0 0.174 0"/> -->
-    <!--   <parent link="${parent}"/> -->
-    <!--   <child link="bottom_neck_arm"/> -->
-    <!-- </joint> -->
-    <!-- <link name="bottom_neck_arm"> -->
-    <!--   <inertial> -->
-    <!--     <origin xyz="0.0 0.0 0.0" rpy="0.0 0.0 0.0"/> -->
-    <!--     <mass value="0.001"/> -->
-    <!--     <inertia ixx="1.0e-6" ixy="1.0e-8" ixz="1.0e-8" iyy="1.0e-6" iyz="1.0e-8" izz="1.0e-6"/> -->
-    <!--   </inertial> -->
-    <!--   <visual name=""> -->
-    <!--     <origin xyz="0.0 0.0 0.0" rpy="0.0 0.0 -1.57"/> -->
-    <!--     <geometry> -->
-    <!--       <mesh filename="file://$(find reachy_description)/meshes/orbita_arm.dae"/> -->
-    <!--     </geometry> -->
-    <!--   </visual> -->
-    <!--   <collision> -->
-    <!--     <origin xyz="0.0 0.0 0.0" rpy="0.0 0.0 0.0"/> -->
-    <!--     <geometry> -->
-    <!--       <cylinder length="0.0" radius="0.0" /> -->
-    <!--     </geometry> -->
-    <!--   </collision> -->
-    <!-- </link> -->
     <!-- Head Links -->
     <link name="head">
@@ -173,18 +68,18 @@
       <child link="head_base" />
     </joint>
-    <link name="head_tracker">
-      <visual name="">
-        <origin xyz="0 0 0" rpy="0.0 0.0 0.0"/>
-        <geometry>
-	  <cylinder length="0.04" radius="0.04"/>
-        </geometry>
-	<material name="camblack"/>
-      </visual>
-    </link>
-    <joint name="head_tracker_fixed" type="fixed">
-      <origin xyz="-0.030 0.0 0.111" rpy="0.0 0.0 0"/>
-      <parent link="head" />
-      <child link="head_tracker" />
-    </joint>
+    <!-- <link name="head_tracker"> -->
+    <!--   <visual name=""> -->
+    <!--     <origin xyz="0 0 0" rpy="0.0 0.0 0.0"/> -->
+    <!--     <geometry> -->
+    <!-- 	  <cylinder length="0.04" radius="0.04"/> -->
+    <!--     </geometry> -->
+    <!-- 	<material name="camblack"/> -->
+    <!--   </visual> -->
+    <!-- </link> -->
+    <!-- <joint name="head_tracker_fixed" type="fixed"> -->
+    <!--   <origin xyz="-0.030 0.0 0.111" rpy="0.0 0.0 0"/> -->
+    <!--   <parent link="head" /> -->
+    <!--   <child link="head_tracker" /> -->
+    <!-- </joint> -->
     <link name="head_tip" >
     </link>
@@ -207,73 +102,4 @@
       <child link="camera_optical_left" />
     </joint>
-    <!-- <link name="l_antenna_link"> -->
-    <!--   <inertial> -->
-    <!--     <origin xyz="-0.001 0.0 0.008" rpy="0.0 0.0 0.0"/> -->
-    <!--     <mass value="0.004"/> -->
-    <!--     <inertia ixx="1.794e-7" ixy="-1.240e-5" ixz="1.91701e-8" iyy="1.5e-7" iyz="3.169e-6" izz="1.933e-7"/> -->
-    <!--   </inertial> -->
-    <!--   <visual name=""> -->
-    <!--     <origin xyz="0.0 0.0 0.0" rpy="0.0 0.0 0.0"/> -->
-    <!--     <geometry> -->
-    <!--       <mesh filename="file://$(find reachy_description)/meshes/antenna.dae"/> -->
-    <!--     </geometry> -->
-    <!--   </visual> -->
-    <!--   <collision> -->
-    <!--     <origin xyz="0.1 0.0 0.1" rpy="0.0 0 0.0"/> -->
-    <!--     <geometry> -->
-    <!--       <cylinder length="0.0" radius="0.0" /> -->
-    <!--     </geometry> -->
-    <!--   </collision> -->
-    <!-- </link> -->
-    <!-- <joint name="l_antenna" type="revolute"> -->
-    <!--   <origin xyz="-0.052 0.057 0.086" rpy="0.166 -1.054 -1.11"/> -->
-    <!--   <parent link="head"/> -->
-    <!--   <child link="l_antenna_link"/> -->
-    <!--   <axis xyz="0 0 1"/> -->
-    <!--   <limit lower="-2.618" upper="2.618" effort="10." velocity="0.0"/> -->
-    <!-- </joint> -->
-    <!-- <link name="r_antenna_link"> -->
-    <!--   <inertial> -->
-    <!--     <origin xyz="-0.001 0.0 0.008" rpy="0.0 0.0 0.0"/> -->
-    <!--     <mass value="0.004"/> -->
-    <!--     <inertia ixx="1.794e-7" ixy="-1.240e-5" ixz="1.91701e-8" iyy="1.5e-7" iyz="3.169e-6" izz="1.933e-7"/> -->
-    <!--   </inertial> -->
-    <!--   <visual name=""> -->
-    <!--     <origin xyz="0.0 0.0 0.0" rpy="0.0 0.0 0.0"/> -->
-    <!--     <geometry> -->
-    <!--       <mesh filename="file://$(find reachy_description)/meshes/antenna.dae"/> -->
-    <!--     </geometry> -->
-    <!--   </visual> -->
-    <!--   <collision> -->
-    <!--     <origin xyz="0.0 0.0 0.0" rpy="0.0 0.0 0.0"/> -->
-    <!--     <geometry> -->
-    <!--       <cylinder length="0.0" radius="0.0" /> -->
-    <!--     </geometry> -->
-    <!--   </collision> -->
-    <!-- </link> -->
-    <!-- <joint name="r_antenna" type="revolute"> -->
-    <!--   <origin xyz="-0.052 -0.057 0.086" rpy="-0.166 -1.054 1.11"/> -->
-    <!--   <parent link="head"/> -->
-    <!--   <child link="r_antenna_link"/> -->
-    <!--   <axis xyz="0 0 1"/> -->
-    <!--   <limit lower="-2.618" upper="2.618" effort="10." velocity="0.0"/> -->
-    <!-- </joint> -->
-    <xacro:head_control
-      neck_orbita_serial_port="${neck_orbita_serial_port}"
-      neck_orbita_id="${neck_orbita_id}"
-      neck_orbita_alpha="${neck_orbita_alpha}"
-      neck_orbita_hardware_zero="${neck_orbita_hardware_zero}"
-      neck_orbita_reduction="${neck_orbita_reduction}"
-    />
-<!--   <xacro:orbita
-    name="neck" parent="${parent}"
-    length="${neck_length}" radius="${neck_radius}" mass="${neck_mass}"
-    xyz="0 0 0" rpy="0 0 0"
-    damping="${damping}" friction="${friction}"
-    orbita_serial_port="${neck_orbita_serial_port}"
-    orbita_id="${neck_orbita_id}"
-    orbita_hardware_zero="${neck_orbita_hardware_zero}"
-    orbita_reduction="${neck_orbita_reduction}"
-  /> -->
     <!-- Reachy Cameras -->
 <!--     <xacro:if value="$(arg use_gazebo)"> -->

File: reachy_description/urdf/reachy.urdf.xacro (robot description, xacro)
@@ -5,33 +5,14 @@
   <xacro:include filename="$(find reachy_description)/urdf/arm.urdf.xacro"/>
   <xacro:include filename="$(find reachy_description)/urdf/head.urdf.xacro"/>
-  <xacro:include filename="$(find reachy_description)/urdf/inertial_primitives.urdf.xacro"/>
+  <xacro:include filename="$(find pollen_generic_description)/urdf/inertial_primitives.urdf.xacro"/>
+  <!-- config  -->
+  <xacro:arg name="neck_config" default="$(find orbita3d_controller)/config/fake.yaml"/>
+  <xacro:arg name="r_shoulder_config" default="$(find orbita2d_controller)/config/fake.yaml"/>
+  <xacro:arg name="r_elbow_config" default="$(find orbita2d_controller)/config/fake.yaml"/>
+  <xacro:arg name="r_wrist_config" default="$(find orbita3d_controller)/config/fake.yaml"/>
+  <!-- config  -->
   <!-- HWI IDs -->
-    <xacro:property name="right_elbow_port_a" value="/dev/right_elbow_A"/>
-    <xacro:property name="right_elbow_port_b" value="/dev/right_elbow_B"/>
-    <xacro:property name="right_elbow_id_a" value="71"/>
-    <xacro:property name="right_elbow_id_b" value="72"/>
-    <xacro:property name="right_wrist_id" value="70"/>
-    <xacro:property name="right_wrist_port" value="/dev/right_wrist"/>
-    <xacro:arg name="right_wrist_hardware_zero" default="0.0, 0.0, 0.0"/>
-    <xacro:property name="neck_id" value="10"/>
-    <xacro:property name="neck_port" value="/dev/neck"/>
-    <xacro:arg name="neck_hardware_zero" default="0.0, 0.0, 0.0"/>
-    <!-- <xacro:property name="left_elbow_id_a" value="8"/> -->
-    <!-- <xacro:property name="left_elbow_id_b" value="9"/> -->
-    <!-- <xacro:property name="left_wrist_id" value="10"/> -->
-    <!-- <xacro:property name="left_shoulder_id_a" value="2"/> -->
-    <!-- <xacro:property name="left_shoulder_id_b" value="1"/> -->
-    <xacro:property name="right_shoulder_port_a" value="/dev/right_shoulder_A"/>
-    <xacro:property name="right_shoulder_port_b" value="/dev/right_shoulder_B"/>
-    <xacro:property name="right_shoulder_id_a" value="81"/>
-    <xacro:property name="right_shoulder_id_b" value="82"/>
     <xacro:property name="right_gripper_id" value="11"/>
     <xacro:property name="right_gripper_port" value="/dev/right_gripper"/>
-  <!-- <xacro:property name="dynamixel_multiplexer_right" value="http://127.0.0.1:50099"/> -->
-  <!--   <xacro:property name="right_gripper_grasping_finger_id" value="11"/> -->
-  <!--   <xacro:property name="right_gripper_action_finger_id" value="12"/> -->
-  <!-- <xacro:property name="dynamixel_multiplexer_left" value="http://127.0.0.1:50096"/> -->
-  <!--   <xacro:property name="left_gripper_grasping_finger_id" value="21"/> -->
-  <!--   <xacro:property name="left_gripper_action_finger_id" value="22"/> -->
   <!-- HWI IDs -->
   <!-- MODEL PARAMETERS -->
@@ -44,5 +25,5 @@
   <!-- MODEL PARAMETERS -->
     <material name="torsoblack">
-        <color rgba="0.5 0.5 0.5 1"/>
+        <color rgba="0.5 0.5 0.5 1.0"/>
     </material>
   <link name="world"/>
@@ -85,21 +66,14 @@
     parent="torso"
     damping="${damping}" friction="${friction}"
-    neck_orbita_serial_port="${neck_port}"
-    neck_orbita_id="${neck_id}"
-    neck_orbita_hardware_zero="$(arg neck_hardware_zero)"
+    neck_config="$(arg neck_config)"
   />
+<!-- <xacro:macro name="arm" params="prefix parent side damping friction orbita2d_shoulder_config orbita2d_elbow_config orbita3d_wrist_config gripper_port gripper_id"> -->
   <!-- RIGHT ARM -->
   <xacro:arm
     prefix="r" parent="torso" side="right"
     damping="${damping}" friction="${friction}"
-    shoulder_port_a="${right_shoulder_port_a}" shoulder_port_b="${right_shoulder_port_b}"
-    elbow_port_a="${right_elbow_port_a}" elbow_port_b="${right_elbow_port_b}"
-    wrist_port="${right_wrist_port}"
-    shoulder_id_a="${right_shoulder_id_a}" shoulder_id_b="${right_shoulder_id_b}"
-    elbow_id_a="${right_elbow_id_a}" elbow_id_b="${right_elbow_id_b}"
-    wrist_id="${right_wrist_id}"
-    wrist_hardware_zero="$(arg right_wrist_hardware_zero)"
-    gripper_id="${right_gripper_id}"
-    gripper_port="${right_gripper_port}"
+    orbita2d_shoulder_config="$(arg r_shoulder_config)"
+    orbita2d_elbow_config="$(arg r_elbow_config)"
+    orbita3d_wrist_config="$(arg r_wrist_config)"
     />
   <!-- <link name="r_wrist_cam_frame"/> -->

Commit message: right arm launch ok

File: reachy_description/urdf/arm.urdf.xacro (robot description, xacro)
@@ -83,10 +83,10 @@
     gripper_id="${gripper_id}"
   />
-  <link name="${p}_arm_tip"/>
-  <joint name="${p}_tip_joint" type="fixed">
-    <origin xyz="0 0 0.1" rpy="${pi} 0 0"/>
-    <parent link="${p}_gripper_palm_link"/>
-    <child link="${p}_arm_tip"/>
-  </joint>
+  <!-- <link name="${p}_arm_tip"/> -->
+  <!-- <joint name="${p}_tip_joint" type="fixed"> -->
+  <!--   <origin xyz="0 0 0.1" rpy="${pi} 0 0"/> -->
+  <!--   <parent link="${p}_gripper_palm_link"/> -->
+  <!--   <child link="${p}_arm_tip"/> -->
+  <!-- </joint> -->
 </xacro:macro>
 </robot>

File: reachy_description/urdf/reachy.urdf.xacro (robot description, xacro)
@@ -15,6 +15,6 @@
   <!-- config  -->
   <!-- HWI IDs -->
-    <xacro:property name="right_gripper_id" value="11"/>
-    <xacro:property name="right_gripper_port" value="/dev/right_gripper"/>
+    <!-- <xacro:property name="left_gripper_id" value="12"/> -->
+    <!-- <xacro:property name="left_gripper_port" value="/dev/left_gripper"/> -->
   <!-- HWI IDs -->
   <!-- MODEL PARAMETERS -->
