Commit message: starting the torture...

File: reachy_description/urdf/arm.urdf.xacro (robot description, xacro)
@@ -83,10 +83,10 @@
     gripper_id="${gripper_id}"
   />
-  <!-- <link name="${p}_arm_tip"/> -->
-  <!-- <joint name="${p}_tip_joint" type="fixed"> -->
-  <!--   <origin xyz="0 0 0.1" rpy="${pi} 0 0"/> -->
-  <!--   <parent link="${p}_gripper_palm_link"/> -->
-  <!--   <child link="${p}_arm_tip"/> -->
-  <!-- </joint> -->
+  <link name="${p}_arm_tip"/>
+  <joint name="${p}_tip_joint" type="fixed">
+    <origin xyz="0 0 0.1" rpy="${pi} 0 0"/>
+    <parent link="${p}_gripper_palm_link"/>
+    <child link="${p}_arm_tip"/>
+  </joint>
 </xacro:macro>
 </robot>

Commit message: Fix shoulder roll limits.

File: reachy_description/urdf/arm.urdf.xacro (robot description, xacro)
@@ -58,5 +58,5 @@
     <xacro:if value="${side == 'left'}">
       <xacro:property name="reflect" value="-1" />
-      <xacro:property name="min_shoulder_roll" value="-0.0" />
+      <xacro:property name="min_shoulder_roll" value="-0.51" />
       <xacro:property name="max_shoulder_roll" value="${pi}" />
       <xacro:property name="shoulder_axis1_inverted" value="0" />
@@ -68,5 +68,5 @@
       <xacro:property name="reflect" value="1" />
       <xacro:property name="min_shoulder_roll" value="-${pi}" />
-      <xacro:property name="max_shoulder_roll" value="0.0" />
+      <xacro:property name="max_shoulder_roll" value="0.51" />
       <xacro:property name="shoulder_axis1_inverted" value="1" />
       <xacro:property name="shoulder_axis2_inverted" value="0" />
