Commit message: add head and gripper

File: reachy_description/ros2_control/head.ros2_control.xacro (robot description, xacro)
@@ -1,5 +1,5 @@
 <?xml version="1.0" ?>
 <robot xmlns:xacro="http://www.ros.org/wiki/xacro">
-    <xacro:macro name="head_control" params="neck_orbita_serial_port neck_orbita_id neck_orbita_alpha neck_orbita_hardware_zero neck_orbita_reduction head_serial_port head_xl320_ids head_xl320_offsets head_xl320_is_direct head_xl320_reductions head_fan_id">
+    <xacro:macro name="head_control" params="neck_orbita_serial_port neck_orbita_id neck_orbita_alpha neck_orbita_hardware_zero neck_orbita_reduction">
         <xacro:include filename="$(find reachy_description)/ros2_control/joint.ros2_control.xacro"/>
         <ros2_control name="head" type="system">
@@ -28,41 +28,41 @@
                  <xacro:position_joint_control name="neck_yaw"/>
         </ros2_control>
-        <ros2_control name="antennas" type="system">
-            <hardware>
-                <xacro:unless value="$(arg use_fake_hardware)">
-                    <plugin>head_system_hwi/HeadSystem</plugin>
-                    <param name="serial_port">${head_serial_port}</param>
-                    <param name="xl320_ids">${head_xl320_ids}</param>
-                    <param name="offsets">${head_xl320_offsets}</param>
-                    <param name="is_direct">${head_xl320_is_direct}</param>
-                    <param name="reductions">${head_xl320_reductions}</param>
-                    <param name="fan_id">${head_fan_id}</param>
-                </xacro:unless>
-                <xacro:if value="$(arg use_fake_hardware)">
-                    <!-- Use gazebo as hardware simulation. -->
-                    <xacro:if value="$(arg use_gazebo)">
-                        <plugin>gazebo_ros2_control/GazeboSystem</plugin>
-                    </xacro:if>
-                    <!-- Use fake components. -->
-                    <xacro:unless value="$(arg use_gazebo)">
-                        <plugin>fake_components/GenericSystem</plugin>
-                    </xacro:unless>
-                </xacro:if>
-            </hardware>
-            <xacro:position_joint_control name="l_antenna"/>
-            <xacro:position_joint_control name="r_antenna"/>
-            <joint name="l_antenna_fan">
-                <state_interface name="state">
-                    <param name="initial_value">0.0</param>
-                </state_interface>
-                <command_interface name="state"/>
-            </joint>
-            <joint name="r_antenna_fan">
-                <state_interface name="state">
-                    <param name="initial_value">0.0</param>
-                </state_interface>
-                <command_interface name="state"/>
-            </joint>
-        </ros2_control>
+        <!-- <ros2_control name="antennas" type="system"> -->
+        <!--     <hardware> -->
+        <!--         <xacro:unless value="$(arg use_fake_hardware)"> -->
+        <!--             <plugin>head_system_hwi/HeadSystem</plugin> -->
+        <!--             <param name="serial_port">${head_serial_port}</param> -->
+        <!--             <param name="xl320_ids">${head_xl320_ids}</param> -->
+        <!--             <param name="offsets">${head_xl320_offsets}</param> -->
+        <!--             <param name="is_direct">${head_xl320_is_direct}</param> -->
+        <!--             <param name="reductions">${head_xl320_reductions}</param> -->
+        <!--             <param name="fan_id">${head_fan_id}</param> -->
+        <!--         </xacro:unless> -->
+        <!--         <xacro:if value="$(arg use_fake_hardware)"> -->
+        <!--             <!-\- Use gazebo as hardware simulation. -\-> -->
+        <!--             <xacro:if value="$(arg use_gazebo)"> -->
+        <!--                 <plugin>gazebo_ros2_control/GazeboSystem</plugin> -->
+        <!--             </xacro:if> -->
+        <!--             <!-\- Use fake components. -\-> -->
+        <!--             <xacro:unless value="$(arg use_gazebo)"> -->
+        <!--                 <plugin>fake_components/GenericSystem</plugin> -->
+        <!--             </xacro:unless> -->
+        <!--         </xacro:if> -->
+        <!--     </hardware> -->
+        <!--     <xacro:position_joint_control name="l_antenna"/> -->
+        <!--     <xacro:position_joint_control name="r_antenna"/> -->
+        <!--     <joint name="l_antenna_fan"> -->
+        <!--         <state_interface name="state"> -->
+        <!--             <param name="initial_value">0.0</param> -->
+        <!--         </state_interface> -->
+        <!--         <command_interface name="state"/> -->
+        <!--     </joint> -->
+        <!--     <joint name="r_antenna_fan"> -->
+        <!--         <state_interface name="state"> -->
+        <!--             <param name="initial_value">0.0</param> -->
+        <!--         </state_interface> -->
+        <!--         <command_interface name="state"/> -->
+        <!--     </joint> -->
+        <!-- </ros2_control> -->
     </xacro:macro>
 </robot>

File: reachy_description/urdf/arm.urdf.xacro (robot description, xacro)
@@ -4,4 +4,5 @@
   <xacro:include filename="$(find reachy_description)/urdf/orbita.urdf.xacro"/>
   <xacro:include filename="$(find reachy_description)/urdf/orbita2dof.urdf.xacro"/>
+  <xacro:include filename="$(find reachy_description)/urdf/smartgripper.urdf.xacro"/>
   <!-- ARM PARAMETERS -->
   <!-- TODO: USE REAL VALUES -->
@@ -76,11 +77,10 @@
     orbita_reduction="${wrist_reduction}"
   />
-  <!-- <xacro:gripper -->
-  <!--   prefix="${p}" parent="${p}_wrist_ball_link" side="${side}" -->
-  <!--   damping="${damping}" friction="${friction}" -->
-  <!--   grpc_multiplexer_url="${grpc_dynamixel_multiplexer_url}" -->
-  <!--   gripper_grasping_finger_id="${gripper_grasping_finger_id}" -->
-  <!--   gripper_action_finger_id="${gripper_action_finger_id}" -->
-  <!-- /> -->
+  <xacro:smartgripper
+    prefix="${p}" parent="${p}_wrist_ball_link" side="${side}"
+    damping="${damping}" friction="${friction}"
+    gripper_port="${gripper_port}"
+    gripper_id="${gripper_id}"
+  />
   <link name="${p}_arm_tip"/>
   <joint name="${p}_tip_joint" type="fixed">

File: reachy_description/urdf/head.urdf.xacro (robot description, xacro)
@@ -4,8 +4,10 @@
   <xacro:property name="camera_link" value="0.05" /> <!-- Size of square 'camera' box -->
   <xacro:property name="camera_convergence" value="0.0" /> <!-- convergence angle (rad) of the cameras. 0=parallel-->
-  <xacro:macro name="head" params="parent damping friction neck_orbita_serial_port neck_orbita_id neck_orbita_alpha neck_orbita_hardware_zero neck_orbita_reduction head_serial_port head_xl320_ids head_xl320_offsets head_xl320_is_direct head_xl320_reductions head_fan_id">
+  <xacro:property name="neck_orbita_reduction" value="4.0"/>
+  <xacro:property name="neck_orbita_alpha" value="0.9424777960769379"/>
+  <xacro:macro name="head" params="parent damping friction neck_orbita_serial_port neck_orbita_id neck_orbita_hardware_zero">
     <xacro:include filename="$(find reachy_description)/ros2_control/head.ros2_control.xacro"/>
     <joint name="neck_roll" type="revolute">
-      <origin xyz="0.015 0.0 0.095" rpy="-0.15105105 0.08669986 -1.05356462"/>
+      <origin xyz="-0.032893 0.0 0.110675" rpy="-0.15105105 0.08669986 -1.05356462"/>
       <parent link="${parent}"/>
       <child link="head_x"/>
@@ -57,76 +59,76 @@
     </joint>
     <!-- Fixed Orbita Arms Visuals -->
-    <joint name="neck_top" type="fixed">
-      <origin xyz="0.0067 0.0 0.0478" rpy="0 0.174 0"/>
-      <parent link="${parent}"/>
-      <child link="top_neck_arm"/>
-    </joint>
-    <link name="top_neck_arm">
-      <inertial>
-        <origin xyz="0.0 0.0 0.0" rpy="0.0 0.0 0.0"/>
-        <mass value="0.001"/>
-        <inertia ixx="1.0e-6" ixy="1.0e-8" ixz="1.0e-8" iyy="1.0e-6" iyz="1.0e-8" izz="1.0e-6"/>
-      </inertial>
-      <visual name="">
-        <origin xyz="0.0 0.0 0.0" rpy="0.0 0.0 0.5236"/>
-        <geometry>
-          <mesh filename="file://$(find reachy_description)/meshes/orbita_arm.dae"/>
-        </geometry>
-      </visual>
-      <collision>
-        <origin xyz="0.0 0.0 0.0" rpy="0.0 0.0 0.0"/>
-        <geometry>
-          <cylinder length="0.0" radius="0.0" />
-        </geometry>
-      </collision>
-    </link>
-    <joint name="neck_middle" type="fixed">
-      <origin xyz="0.0067 0.0 0.0478" rpy="0 0.174 0"/>
-      <parent link="${parent}"/>
-      <child link="middle_neck_arm"/>
-    </joint>
-    <link name="middle_neck_arm">
-      <inertial>
-        <origin xyz="0.0 0.0 0.0" rpy="0.0 0.0 0.0"/>
-        <mass value="0.001"/>
-        <inertia ixx="1.0e-6" ixy="1.0e-8" ixz="1.0e-8" iyy="1.0e-6" iyz="1.0e-8" izz="1.0e-6"/>
-      </inertial>
-      <visual name="">
-        <origin xyz="0.0 0.0 0.0" rpy="0.0 0.0 2.618"/>
-        <geometry>
-          <mesh filename="file://$(find reachy_description)/meshes/orbita_arm.dae"/>
-        </geometry>
-      </visual>
-      <collision>
-        <origin xyz="0.0 0.0 0.0" rpy="0.0 0.0 0.0"/>
-        <geometry>
-          <cylinder length="0.0" radius="0.0" />
-        </geometry>
-      </collision>
-    </link>
-    <joint name="neck_bottom" type="fixed">
-      <origin xyz="0.0067 0.0 0.0478" rpy="0 0.174 0"/>
-      <parent link="${parent}"/>
-      <child link="bottom_neck_arm"/>
-    </joint>
-    <link name="bottom_neck_arm">
-      <inertial>
-        <origin xyz="0.0 0.0 0.0" rpy="0.0 0.0 0.0"/>
-        <mass value="0.001"/>
-        <inertia ixx="1.0e-6" ixy="1.0e-8" ixz="1.0e-8" iyy="1.0e-6" iyz="1.0e-8" izz="1.0e-6"/>
-      </inertial>
-      <visual name="">
-        <origin xyz="0.0 0.0 0.0" rpy="0.0 0.0 -1.57"/>
-        <geometry>
-          <mesh filename="file://$(find reachy_description)/meshes/orbita_arm.dae"/>
-        </geometry>
-      </visual>
-      <collision>
-        <origin xyz="0.0 0.0 0.0" rpy="0.0 0.0 0.0"/>
-        <geometry>
-          <cylinder length="0.0" radius="0.0" />
-        </geometry>
-      </collision>
-    </link>
+    <!-- <joint name="neck_top" type="fixed"> -->
+    <!--   <origin xyz="0.0067 0.0 0.0478" rpy="0 0.174 0"/> -->
+    <!--   <parent link="${parent}"/> -->
+    <!--   <child link="top_neck_arm"/> -->
+    <!-- </joint> -->
+    <!-- <link name="top_neck_arm"> -->
+    <!--   <inertial> -->
+    <!--     <origin xyz="0.0 0.0 0.0" rpy="0.0 0.0 0.0"/> -->
+    <!--     <mass value="0.001"/> -->
+    <!--     <inertia ixx="1.0e-6" ixy="1.0e-8" ixz="1.0e-8" iyy="1.0e-6" iyz="1.0e-8" izz="1.0e-6"/> -->
+    <!--   </inertial> -->
+    <!--   <visual name=""> -->
+    <!--     <origin xyz="0.0 0.0 0.0" rpy="0.0 0.0 0.5236"/> -->
+    <!--     <geometry> -->
+    <!--       <mesh filename="file://$(find reachy_description)/meshes/orbita_arm.dae"/> -->
+    <!--     </geometry> -->
+    <!--   </visual> -->
+    <!--   <collision> -->
+    <!--     <origin xyz="0.0 0.0 0.0" rpy="0.0 0.0 0.0"/> -->
+    <!--     <geometry> -->
+    <!--       <cylinder length="0.0" radius="0.0" /> -->
+    <!--     </geometry> -->
+    <!--   </collision> -->
+    <!-- </link> -->
+    <!-- <joint name="neck_middle" type="fixed"> -->
+    <!--   <origin xyz="0.0067 0.0 0.0478" rpy="0 0.174 0"/> -->
+    <!--   <parent link="${parent}"/> -->
+    <!--   <child link="middle_neck_arm"/> -->
+    <!-- </joint> -->
+    <!-- <link name="middle_neck_arm"> -->
+    <!--   <inertial> -->
+    <!--     <origin xyz="0.0 0.0 0.0" rpy="0.0 0.0 0.0"/> -->
+    <!--     <mass value="0.001"/> -->
+    <!--     <inertia ixx="1.0e-6" ixy="1.0e-8" ixz="1.0e-8" iyy="1.0e-6" iyz="1.0e-8" izz="1.0e-6"/> -->
+    <!--   </inertial> -->
+    <!--   <visual name=""> -->
+    <!--     <origin xyz="0.0 0.0 0.0" rpy="0.0 0.0 2.618"/> -->
+    <!--     <geometry> -->
+    <!--       <mesh filename="file://$(find reachy_description)/meshes/orbita_arm.dae"/> -->
+    <!--     </geometry> -->
+    <!--   </visual> -->
+    <!--   <collision> -->
+    <!--     <origin xyz="0.0 0.0 0.0" rpy="0.0 0.0 0.0"/> -->
+    <!--     <geometry> -->
+    <!--       <cylinder length="0.0" radius="0.0" /> -->
+    <!--     </geometry> -->
+    <!--   </collision> -->
+    <!-- </link> -->
+    <!-- <joint name="neck_bottom" type="fixed"> -->
+    <!--   <origin xyz="0.0067 0.0 0.0478" rpy="0 0.174 0"/> -->
+    <!--   <parent link="${parent}"/> -->
+    <!--   <child link="bottom_neck_arm"/> -->
+    <!-- </joint> -->
+    <!-- <link name="bottom_neck_arm"> -->
+    <!--   <inertial> -->
+    <!--     <origin xyz="0.0 0.0 0.0" rpy="0.0 0.0 0.0"/> -->
+    <!--     <mass value="0.001"/> -->
+    <!--     <inertia ixx="1.0e-6" ixy="1.0e-8" ixz="1.0e-8" iyy="1.0e-6" iyz="1.0e-8" izz="1.0e-6"/> -->
+    <!--   </inertial> -->
+    <!--   <visual name=""> -->
+    <!--     <origin xyz="0.0 0.0 0.0" rpy="0.0 0.0 -1.57"/> -->
+    <!--     <geometry> -->
+    <!--       <mesh filename="file://$(find reachy_description)/meshes/orbita_arm.dae"/> -->
+    <!--     </geometry> -->
+    <!--   </visual> -->
+    <!--   <collision> -->
+    <!--     <origin xyz="0.0 0.0 0.0" rpy="0.0 0.0 0.0"/> -->
+    <!--     <geometry> -->
+    <!--       <cylinder length="0.0" radius="0.0" /> -->
+    <!--     </geometry> -->
+    <!--   </collision> -->
+    <!-- </link> -->
     <!-- Head Links -->
     <link name="head">
@@ -159,56 +161,56 @@
       <child link="head_tip" />
     </joint>
-    <link name="l_antenna_link">
-      <inertial>
-        <origin xyz="-0.001 0.0 0.008" rpy="0.0 0.0 0.0"/>
-        <mass value="0.004"/>
-        <inertia ixx="1.794e-7" ixy="-1.240e-5" ixz="1.91701e-8" iyy="1.5e-7" iyz="3.169e-6" izz="1.933e-7"/>
-      </inertial>
-      <visual name="">
-        <origin xyz="0.0 0.0 0.0" rpy="0.0 0.0 0.0"/>
-        <geometry>
-          <mesh filename="file://$(find reachy_description)/meshes/antenna.dae"/>
-        </geometry>
-      </visual>
-      <collision>
-        <origin xyz="0.1 0.0 0.1" rpy="0.0 0 0.0"/>
-        <geometry>
-          <cylinder length="0.0" radius="0.0" />
-        </geometry>
-      </collision>
-    </link>
-    <joint name="l_antenna" type="revolute">
-      <origin xyz="-0.052 0.057 0.086" rpy="0.166 -1.054 -1.11"/>
-      <parent link="head"/>
-      <child link="l_antenna_link"/>
-      <axis xyz="0 0 1"/>
-      <limit lower="-2.618" upper="2.618" effort="10." velocity="0.0"/>
-    </joint>
-    <link name="r_antenna_link">
-      <inertial>
-        <origin xyz="-0.001 0.0 0.008" rpy="0.0 0.0 0.0"/>
-        <mass value="0.004"/>
-        <inertia ixx="1.794e-7" ixy="-1.240e-5" ixz="1.91701e-8" iyy="1.5e-7" iyz="3.169e-6" izz="1.933e-7"/>
-      </inertial>
-      <visual name="">
-        <origin xyz="0.0 0.0 0.0" rpy="0.0 0.0 0.0"/>
-        <geometry>
-          <mesh filename="file://$(find reachy_description)/meshes/antenna.dae"/>
-        </geometry>
-      </visual>
-      <collision>
-        <origin xyz="0.0 0.0 0.0" rpy="0.0 0.0 0.0"/>
-        <geometry>
-          <cylinder length="0.0" radius="0.0" />
-        </geometry>
-      </collision>
-    </link>
-    <joint name="r_antenna" type="revolute">
-      <origin xyz="-0.052 -0.057 0.086" rpy="-0.166 -1.054 1.11"/>
-      <parent link="head"/>
-      <child link="r_antenna_link"/>
-      <axis xyz="0 0 1"/>
-      <limit lower="-2.618" upper="2.618" effort="10." velocity="0.0"/>
-    </joint>
+    <!-- <link name="l_antenna_link"> -->
+    <!--   <inertial> -->
+    <!--     <origin xyz="-0.001 0.0 0.008" rpy="0.0 0.0 0.0"/> -->
+    <!--     <mass value="0.004"/> -->
+    <!--     <inertia ixx="1.794e-7" ixy="-1.240e-5" ixz="1.91701e-8" iyy="1.5e-7" iyz="3.169e-6" izz="1.933e-7"/> -->
+    <!--   </inertial> -->
+    <!--   <visual name=""> -->
+    <!--     <origin xyz="0.0 0.0 0.0" rpy="0.0 0.0 0.0"/> -->
+    <!--     <geometry> -->
+    <!--       <mesh filename="file://$(find reachy_description)/meshes/antenna.dae"/> -->
+    <!--     </geometry> -->
+    <!--   </visual> -->
+    <!--   <collision> -->
+    <!--     <origin xyz="0.1 0.0 0.1" rpy="0.0 0 0.0"/> -->
+    <!--     <geometry> -->
+    <!--       <cylinder length="0.0" radius="0.0" /> -->
+    <!--     </geometry> -->
+    <!--   </collision> -->
+    <!-- </link> -->
+    <!-- <joint name="l_antenna" type="revolute"> -->
+    <!--   <origin xyz="-0.052 0.057 0.086" rpy="0.166 -1.054 -1.11"/> -->
+    <!--   <parent link="head"/> -->
+    <!--   <child link="l_antenna_link"/> -->
+    <!--   <axis xyz="0 0 1"/> -->
+    <!--   <limit lower="-2.618" upper="2.618" effort="10." velocity="0.0"/> -->
+    <!-- </joint> -->
+    <!-- <link name="r_antenna_link"> -->
+    <!--   <inertial> -->
+    <!--     <origin xyz="-0.001 0.0 0.008" rpy="0.0 0.0 0.0"/> -->
+    <!--     <mass value="0.004"/> -->
+    <!--     <inertia ixx="1.794e-7" ixy="-1.240e-5" ixz="1.91701e-8" iyy="1.5e-7" iyz="3.169e-6" izz="1.933e-7"/> -->
+    <!--   </inertial> -->
+    <!--   <visual name=""> -->
+    <!--     <origin xyz="0.0 0.0 0.0" rpy="0.0 0.0 0.0"/> -->
+    <!--     <geometry> -->
+    <!--       <mesh filename="file://$(find reachy_description)/meshes/antenna.dae"/> -->
+    <!--     </geometry> -->
+    <!--   </visual> -->
+    <!--   <collision> -->
+    <!--     <origin xyz="0.0 0.0 0.0" rpy="0.0 0.0 0.0"/> -->
+    <!--     <geometry> -->
+    <!--       <cylinder length="0.0" radius="0.0" /> -->
+    <!--     </geometry> -->
+    <!--   </collision> -->
+    <!-- </link> -->
+    <!-- <joint name="r_antenna" type="revolute"> -->
+    <!--   <origin xyz="-0.052 -0.057 0.086" rpy="-0.166 -1.054 1.11"/> -->
+    <!--   <parent link="head"/> -->
+    <!--   <child link="r_antenna_link"/> -->
+    <!--   <axis xyz="0 0 1"/> -->
+    <!--   <limit lower="-2.618" upper="2.618" effort="10." velocity="0.0"/> -->
+    <!-- </joint> -->
     <xacro:head_control
       neck_orbita_serial_port="${neck_orbita_serial_port}"
@@ -217,10 +219,4 @@
       neck_orbita_hardware_zero="${neck_orbita_hardware_zero}"
       neck_orbita_reduction="${neck_orbita_reduction}"
-      head_serial_port="${head_serial_port}"
-      head_xl320_ids="${head_xl320_ids}"
-      head_xl320_offsets="${head_xl320_offsets}"
-      head_xl320_is_direct="${head_xl320_is_direct}"
-      head_xl320_reductions="${head_xl320_reductions}"
-      head_fan_id="${head_fan_id}"
     />
     <!-- Cameras -->

File: reachy_description/urdf/reachy.urdf.xacro (robot description, xacro)
@@ -4,5 +4,5 @@
   <xacro:arg name="use_gazebo" default="false"/>
   <xacro:include filename="$(find reachy_description)/urdf/arm.urdf.xacro"/>
-  <!-- <xacro:include filename="$(find reachy_description)/urdf/head.urdf.xacro"/> -->
+  <xacro:include filename="$(find reachy_description)/urdf/head.urdf.xacro"/>
   <!-- <xacro:include filename="$(find reachy_description)/urdf/gripper.urdf.xacro"/> -->
   <xacro:include filename="$(find reachy_description)/urdf/inertial_primitives.urdf.xacro"/>
@@ -15,4 +15,7 @@
     <xacro:property name="right_wrist_port" value="/dev/right_wrist"/>
     <xacro:arg name="right_wrist_hardware_zero" default="0.0, 0.0, 0.0"/>
+    <xacro:property name="neck_id" value="2"/>
+    <xacro:property name="neck_port" value="/dev/neck"/>
+    <xacro:arg name="neck_hardware_zero" default="0.0, 0.0, 0.0"/>
     <!-- <xacro:property name="left_elbow_id_a" value="8"/> -->
     <!-- <xacro:property name="left_elbow_id_b" value="9"/> -->
@@ -59,7 +62,7 @@
     <xacro:if value="${base_visual}">
       <visual>
-        <origin xyz="0 0 -0.1" rpy="0 0.0 0"/>
+        <origin xyz="-0.05 0 -0.05" rpy="0 0.0 0"/>
         <geometry>
-          <box size="0.11 0.2 0.32"/>
+          <box size="0.1 0.2 0.22"/>
         </geometry>
         <!-- <origin xyz="0 0 -0.5" rpy="0 0 0"/> -->
@@ -77,10 +80,11 @@
   </gazebo>
   <!-- TORSO -->
-  <!-- <xacro:head -->
-  <!--   parent="torso" -->
-  <!--   damping="${damping}" friction="${friction}" -->
-  <!--   grpc_multiplexer_url="${ethercat_multiplexer}" -->
-  <!--   neck_id_top="${neck_id_top}" neck_id_middle="${neck_id_middle}" neck_id_bottom="${neck_id_bottom}" -->
-  <!-- /> -->
+  <xacro:head
+    parent="torso"
+    damping="${damping}" friction="${friction}"
+    neck_orbita_serial_port="${neck_port}"
+    neck_orbita_id="${neck_id}"
+    neck_orbita_hardware_zero="$(arg neck_hardware_zero)"
+  />
   <!-- RIGHT ARM -->
   <xacro:arm
