Commit message: add head, torque ok

File: reachy_description/ros2_control/head.ros2_control.xacro (robot description, xacro)
@@ -3,5 +3,5 @@
     <xacro:macro name="head_control" params="neck_orbita_serial_port neck_orbita_id neck_orbita_alpha neck_orbita_hardware_zero neck_orbita_reduction">
         <xacro:include filename="$(find reachy_description)/ros2_control/joint.ros2_control.xacro"/>
-        <ros2_control name="head" type="system">
+        <ros2_control name="neck" type="system">
             <hardware>
                 <xacro:unless value="$(arg use_fake_hardware)">

File: reachy_description/ros2_control/orbita.ros2_control.xacro (robot description, xacro)
@@ -3,5 +3,5 @@
     <xacro:macro name="orbita_control" params="name orbita_serial_port orbita_id orbita_alpha orbita_hardware_zero orbita_reduction">
         <xacro:include filename="$(find reachy_description)/ros2_control/joint.ros2_control.xacro"/>
-        <ros2_control name="orbita" type="system">
+        <ros2_control name="${name}" type="system">
             <hardware>
                 <xacro:unless value="$(arg use_fake_hardware)">

File: reachy_description/ros2_control/orbita2dof.ros2_control.xacro (robot description, xacro)
@@ -2,18 +2,19 @@
 <robot xmlns:xacro="http://www.ros.org/wiki/xacro">
   <xacro:include filename="$(find reachy_description)/ros2_control/joint.ros2_control.xacro"/>
-  <xacro:macro name="orbita2dof_control" params="name joint1 joint2 port_a port_b id_a id_b offset_a offset_b ratio_a ratio_b">
+  <xacro:macro name="orbita2dof_control" params="name joint1 joint2 port_a port_b id_a id_b offset_a offset_b ratio_a ratio_b lower_limit_a upper_limit_a lower_limit_b upper_limit_b axis1_inverted axis2_inverted">
     <ros2_control name="${name}" type="system">
       <hardware>
         <!-- Use real hardware. -->
         <xacro:unless value="$(arg use_fake_hardware)">
-          <plugin>orbita2d_hardware_interface/Orbita2dofSystem</plugin>
-          <param name="port_a">${port_a}</param>
-          <param name="port_b">${port_b}</param>
-          <param name="id_a">${id_a}</param>
-          <param name="id_b">${id_b}</param>
-          <param name="offset_a">${offset_a}</param>
-          <param name="offset_b">${offset_b}</param>
-          <param name="ratio_a">${ratio_a}</param>
-          <param name="ratio_b">${ratio_b}</param>
+          <plugin>orbita2d_serial_system_hwi/Orbita2dSerialSystem</plugin>
+          <param name="serial_port_1">${port_a}</param>
+          <param name="serial_port_2">${port_b}</param>
+          <param name="id_1">${id_a}</param>
+          <param name="id_2">${id_b}</param>
+          <param name="offsets">${offset_a},${offset_b}</param>
+          <param name="ratio">${ratio_a},${ratio_b}</param>
+          <param name="limits">${lower_limit_a},${upper_limit_a},${lower_limit_b},${upper_limit_b}</param>
+          <param name="axis1_inverted">${axis1_inverted}</param>
+          <param name="axis2_inverted">${axis2_inverted}</param>
         </xacro:unless>
         <xacro:if value="$(arg use_fake_hardware)">
@@ -30,8 +31,4 @@
       <xacro:position_joint_control name="${name}_${joint1}"/>
       <xacro:position_joint_control name="${name}_${joint2}"/>
-      <gpio name="${name}">
-        <state_interface name="torque" data_type="bool"/>
-        <command_interface name="torque" data_type="bool"/>
-      </gpio>
     </ros2_control>
   </xacro:macro>

File: reachy_description/ros2_control/smartgripper.ros2_control.xacro (robot description, xacro)
@@ -7,9 +7,10 @@
         <!-- Use real hardware. -->
         <xacro:unless value="$(arg use_fake_hardware)">
-          <plugin>smart_gripper_system_hwi/GripperSystem</plugin>
+          <plugin>fake_components/GenericSystem</plugin>
+          <!-- <plugin>smart_gripper_system_hwi/GripperSystem</plugin>
           <param name="gripper_port">${gripper_port}</param>
           <param name="gripper_id">${gripper_id}</param>
           <param name="min_grasping_finger">${min_grasping_finger}</param>
-          <param name="max_grasping_finger">${max_grasping_finger}</param>
+          <param name="max_grasping_finger">${max_grasping_finger}</param> -->
         </xacro:unless>
         <xacro:if value="$(arg use_fake_hardware)">
@@ -25,8 +26,4 @@
       </hardware>
       <xacro:position_joint_control name="${name}_finger"/>
-      <gpio name="${name}">
-        <state_interface name="torque" data_type="bool"/>
-        <command_interface name="torque" data_type="bool"/>
-      </gpio>
     </ros2_control>
   </xacro:macro>

File: reachy_description/urdf/arm.urdf.xacro (robot description, xacro)
@@ -14,11 +14,11 @@
   <xacro:property name="arm_radius" value="0.03"/>
   <xacro:property name="arm_mass" value="0.5"/>
-  <xacro:property name="shoulder_ratio_a" value="-1.5"/>
-  <xacro:property name="shoulder_ratio_b" value="-1.5"/>
+  <xacro:property name="shoulder_ratio_a" value="47.519"/>
+  <xacro:property name="shoulder_ratio_b" value="47.519"/>
   <xacro:property name="forearm_length" value="0.28"/>
   <xacro:property name="forearm_radius" value="0.025"/>
   <xacro:property name="forearm_mass" value="0.45"/>
-  <xacro:property name="elbow_ratio_a" value="1.778"/>
-  <xacro:property name="elbow_ratio_b" value="1.778"/>
+  <xacro:property name="elbow_ratio_a" value="45.018"/>
+  <xacro:property name="elbow_ratio_b" value="45.018"/>
   <xacro:property name="wrist_length" value="0.01"/>
   <xacro:property name="wrist_radius" value="0.02"/>
@@ -30,5 +30,8 @@
     <xacro:property name="min_shoulder_roll" value="-0.0"/>
     <xacro:property name="max_shoulder_roll" value="${pi/2}"/>
-    <xacro:property name="pitch_inverted" value="1.0"/>
+    <xacro:property name="shoulder_axis1_inverted" value="0"/>
+    <xacro:property name="shoulder_axis2_inverted" value="0"/>
+    <xacro:property name="elbow_axis1_inverted" value="0"/>
+    <xacro:property name="elbow_axis2_inverted" value="0"/>
   </xacro:if>
   <xacro:if value="${side == 'right'}">
@@ -36,9 +39,12 @@
     <xacro:property name="min_shoulder_roll" value="-${pi/2}"/>
     <xacro:property name="max_shoulder_roll" value="0.0"/>
-    <xacro:property name="pitch_inverted" value="0.0"/>
+    <xacro:property name="shoulder_axis1_inverted" value="1"/>
+    <xacro:property name="shoulder_axis2_inverted" value="0"/>
+    <xacro:property name="elbow_axis1_inverted" value="1"/>
+    <xacro:property name="elbow_axis2_inverted" value="0"/>
   </xacro:if>
   <xacro:property name="p" value="${prefix}"/>
   <xacro:orbita2dof
-    name="${p}_arm" parent="${parent}"
+    name="${p}_shoulder" parent="${parent}"
     length="${arm_length}" radius="${arm_radius}" mass="${arm_mass}"
     xyz="${arm_offset_x} ${arm_offset_y*reflect} ${arm_offset_z}" rpy="0 0 ${arm_offset_yaw*reflect}"
@@ -51,8 +57,9 @@
     offset_a="0.0" offset_b="0.0"
     ratio_a="${shoulder_ratio_a}" ratio_b="${shoulder_ratio_b}"
-    pitch_inverted="${pitch_inverted}"
+    axis1_inverted="${shoulder_axis1_inverted}"
+    axis2_inverted="${shoulder_axis2_inverted}"
   />
-  <xacro:orbita2dof
-    name="${p}_forearm" parent="${p}_arm_ball_link"
+   <xacro:orbita2dof
+    name="${p}_elbow" parent="${p}_shoulder_ball_link"
     length="${forearm_length}" radius="${forearm_radius}" mass="${forearm_mass}"
     xyz="0 0 -${arm_length}" rpy="0 0 0"
@@ -65,8 +72,9 @@
     offset_a="0.0" offset_b="0.0"
     ratio_a="${elbow_ratio_a}" ratio_b="${elbow_ratio_b}"
-    pitch_inverted="0.0"
+    axis1_inverted="${elbow_axis1_inverted}"
+    axis2_inverted="${elbow_axis2_inverted}"
   />
   <xacro:orbita
-    name="${p}_wrist" parent="${p}_forearm_ball_link"
+    name="${p}_wrist" parent="${p}_elbow_ball_link"
     length="${wrist_length}" radius="${wrist_radius}" mass="${wrist_mass}"
     xyz="0 0 -${forearm_length}" rpy="${pi} 0 0"
@@ -77,5 +85,5 @@
     orbita_reduction="${wrist_reduction}"
   />
-  <xacro:smartgripper
+<!--   <xacro:smartgripper
     prefix="${p}" parent="${p}_wrist_ball_link" side="${side}"
     damping="${damping}" friction="${friction}"
@@ -88,5 +96,5 @@
     <parent link="${p}_gripper_palm_link"/>
     <child link="${p}_arm_tip"/>
-  </joint>
+  </joint> -->
 </xacro:macro>
 </robot>

File: reachy_description/urdf/head.urdf.xacro (robot description, xacro)
@@ -220,4 +220,14 @@
       neck_orbita_reduction="${neck_orbita_reduction}"
     />
+<!--   <xacro:orbita
+    name="neck" parent="${parent}"
+    length="${neck_length}" radius="${neck_radius}" mass="${neck_mass}"
+    xyz="0 0 0" rpy="0 0 0"
+    damping="${damping}" friction="${friction}"
+    orbita_serial_port="${neck_orbita_serial_port}"
+    orbita_id="${neck_orbita_id}"
+    orbita_hardware_zero="${neck_orbita_hardware_zero}"
+    orbita_reduction="${neck_orbita_reduction}"
+  /> -->
     <!-- Cameras -->
     <xacro:if value="$(arg use_gazebo)">

File: reachy_description/urdf/orbita2dof.urdf.xacro (robot description, xacro)
@@ -14,5 +14,5 @@
     </xacro:if>
   </xacro:macro>
-  <xacro:macro name="orbita2dof" params="name parent length radius mass xyz rpy damping friction joint1 joint2 joint1_min_angle joint1_max_angle joint2_min_angle joint2_max_angle port_a port_b id_a id_b offset_a offset_b ratio_a ratio_b pitch_inverted">
+  <xacro:macro name="orbita2dof" params="name parent length radius mass xyz rpy damping friction joint1 joint2 joint1_min_angle joint1_max_angle joint2_min_angle joint2_max_angle port_a port_b id_a id_b offset_a offset_b ratio_a ratio_b axis1_inverted axis2_inverted">
     <!--
       Orbita 2 dof
@@ -87,5 +87,18 @@
       name="${name}"
       joint1="${joint1}" joint2="${joint2}"
-      port_a="${port_a}" port_b="${port_b}" id_a="${id_a}" id_b="${id_b}" offset_a="${offset_a}" offset_b="${offset_b}" ratio_a="${ratio_a}" ratio_b="${ratio_b}"
+      port_a="${port_a}"
+      id_a="${id_a}"
+      port_b="${port_b}"
+      id_b="${id_b}"
+      offset_a="${offset_a}"
+      offset_b="${offset_b}"
+      ratio_a="${ratio_a}"
+      ratio_b="${ratio_b}"
+      lower_limit_a="${joint1_min_angle}"
+      upper_limit_a="${joint1_max_angle}"
+      lower_limit_b="${joint2_min_angle}"
+      upper_limit_b="${joint2_max_angle}"
+      axis1_inverted="${axis1_inverted}"
+      axis2_inverted="${axis2_inverted}"
     />
   </xacro:macro>

File: reachy_description/urdf/reachy.urdf.xacro (robot description, xacro)
@@ -9,10 +9,10 @@
     <xacro:property name="right_elbow_port_a" value="/dev/right_elbow_A"/>
     <xacro:property name="right_elbow_port_b" value="/dev/right_elbow_B"/>
-    <xacro:property name="right_elbow_id_a" value="1"/>
-    <xacro:property name="right_elbow_id_b" value="0"/>
-    <xacro:property name="right_wrist_id" value="2"/>
+    <xacro:property name="right_elbow_id_a" value="71"/>
+    <xacro:property name="right_elbow_id_b" value="72"/>
+    <xacro:property name="right_wrist_id" value="70"/>
     <xacro:property name="right_wrist_port" value="/dev/right_wrist"/>
     <xacro:arg name="right_wrist_hardware_zero" default="0.0, 0.0, 0.0"/>
-    <xacro:property name="neck_id" value="2"/>
+    <xacro:property name="neck_id" value="10"/>
     <xacro:property name="neck_port" value="/dev/neck"/>
     <xacro:arg name="neck_hardware_zero" default="0.0, 0.0, 0.0"/>
@@ -24,7 +24,7 @@
     <xacro:property name="right_shoulder_port_a" value="/dev/right_shoulder_A"/>
     <xacro:property name="right_shoulder_port_b" value="/dev/right_shoulder_B"/>
-    <xacro:property name="right_shoulder_id_a" value="6"/>
-    <xacro:property name="right_shoulder_id_b" value="5"/>
-    <xacro:property name="right_gripper_id" value="11"/>
+    <xacro:property name="right_shoulder_id_a" value="81"/>
+    <xacro:property name="right_shoulder_id_b" value="82"/>
+    <xacro:property name="right_gripper_id" value="41"/>
     <xacro:property name="right_gripper_port" value="/dev/right_gripper"/>
   <!-- <xacro:property name="dynamixel_multiplexer_right" value="http://127.0.0.1:50099"/> -->
