Commit message: Add smart gripper hwi.

File: reachy_description/ros2_control/smartgripper.ros2_control.xacro (robot description, xacro)
@@ -7,10 +7,9 @@
         <!-- Use real hardware. -->
         <xacro:unless value="$(arg use_fake_hardware)">
-          <plugin>fake_components/GenericSystem</plugin>
-          <!-- <plugin>smart_gripper_system_hwi/GripperSystem</plugin>
+          <plugin>smart_gripper_dynamixel_system_hwi/SmartGripperDynamixelSystem</plugin>
           <param name="gripper_port">${gripper_port}</param>
           <param name="gripper_id">${gripper_id}</param>
           <param name="min_grasping_finger">${min_grasping_finger}</param>
-          <param name="max_grasping_finger">${max_grasping_finger}</param> -->
+          <param name="max_grasping_finger">${max_grasping_finger}</param>
         </xacro:unless>
         <xacro:if value="$(arg use_fake_hardware)">

File: reachy_description/urdf/arm.urdf.xacro (robot description, xacro)
@@ -85,5 +85,5 @@
     orbita_reduction="${wrist_reduction}"
   />
-<!--   <xacro:smartgripper
+  <xacro:smartgripper
     prefix="${p}" parent="${p}_wrist_ball_link" side="${side}"
     damping="${damping}" friction="${friction}"
@@ -96,5 +96,5 @@
     <parent link="${p}_gripper_palm_link"/>
     <child link="${p}_arm_tip"/>
-  </joint> -->
+  </joint>
 </xacro:macro>
 </robot>

File: reachy_description/urdf/reachy.urdf.xacro (robot description, xacro)
@@ -26,5 +26,5 @@
     <xacro:property name="right_shoulder_id_a" value="81"/>
     <xacro:property name="right_shoulder_id_b" value="82"/>
-    <xacro:property name="right_gripper_id" value="41"/>
+    <xacro:property name="right_gripper_id" value="11"/>
     <xacro:property name="right_gripper_port" value="/dev/right_gripper"/>
   <!-- <xacro:property name="dynamixel_multiplexer_right" value="http://127.0.0.1:50099"/> -->

Commit message: add back smartgripper

File: reachy_description/ros2_control/smartgripper.ros2_control.xacro (robot description, xacro)
@@ -2,5 +2,5 @@
 <robot xmlns:xacro="http://www.ros.org/wiki/xacro">
   <xacro:macro name="smart_gripper_control" params="name gripper_port gripper_id min_grasping_finger max_grasping_finger">
-    <xacro:include filename="$(find reachy_description)/ros2_control/joint.ros2_control.xacro"/>
+  <xacro:include filename="$(find pollen_generic_description)/ros2_control/joint.ros2_control.xacro"/>
     <ros2_control name="${name}" type="system">
       <hardware>

File: reachy_description/urdf/arm.urdf.xacro (robot description, xacro)
@@ -1,8 +1,8 @@
 <?xml version="1.0" ?>
 <robot xmlns:xacro="http://www.ros.org/wiki/xacro">
-<xacro:macro name="arm" params="prefix parent side damping friction orbita2d_shoulder_config orbita2d_elbow_config orbita3d_wrist_config">
+<xacro:macro name="arm" params="prefix parent side damping friction orbita2d_shoulder_config orbita2d_elbow_config orbita3d_wrist_config gripper_port gripper_id">
   <xacro:include filename="$(find orbita3d_description)/urdf/orbita3d.urdf.xacro"/>
   <xacro:include filename="$(find orbita2d_description)/urdf/orbita2d.urdf.xacro"/>
-  <!-- <xacro:include filename="$(find reachy_description)/urdf/smartgripper.urdf.xacro"/> -->
+  <xacro:include filename="$(find reachy_description)/urdf/smartgripper.urdf.xacro"/>
   <!-- <!-\- Orbita2d config -\-> -->
   <!-- <xacro:arg name="orbita2d_shoulder_config" default="$(find orbita2d_description)/config/fake.yaml"/> -->
@@ -77,16 +77,16 @@
     config_file="${orbita3d_wrist_config}"
   />
-  <!-- <xacro:smartgripper -->
-  <!--   prefix="${p}" parent="${p}_wrist_ball_link" side="${side}" -->
-  <!--   damping="${damping}" friction="${friction}" -->
-  <!--   gripper_port="${gripper_port}" -->
-  <!--   gripper_id="${gripper_id}" -->
-  <!-- /> -->
-  <!-- <link name="${p}_arm_tip"/> -->
-  <!-- <joint name="${p}_tip_joint" type="fixed"> -->
-  <!--   <origin xyz="0 0 0.1" rpy="${pi} 0 0"/> -->
-  <!--   <parent link="${p}_gripper_palm_link"/> -->
-  <!--   <child link="${p}_arm_tip"/> -->
-  <!-- </joint> -->
+  <xacro:smartgripper
+    prefix="${p}" parent="${p}_wrist_ball_link" side="${side}"
+    damping="${damping}" friction="${friction}"
+    gripper_port="${gripper_port}"
+    gripper_id="${gripper_id}"
+  />
+  <link name="${p}_arm_tip"/>
+  <joint name="${p}_tip_joint" type="fixed">
+    <origin xyz="0 0 0.1" rpy="${pi} 0 0"/>
+    <parent link="${p}_gripper_palm_link"/>
+    <child link="${p}_arm_tip"/>
+  </joint>
 </xacro:macro>
 </robot>

File: reachy_description/urdf/reachy.urdf.xacro (robot description, xacro)
@@ -11,4 +11,6 @@
   <xacro:arg name="r_elbow_config" default="$(find orbita2d_controller)/config/fake.yaml"/>
   <xacro:arg name="r_wrist_config" default="$(find orbita3d_controller)/config/fake.yaml"/>
+  <xacro:property name="right_gripper_id" value="11"/>
+  <xacro:property name="right_gripper_port" value="/dev/right_gripper"/>
   <!-- config  -->
   <!-- HWI IDs -->
@@ -76,4 +78,6 @@
     orbita2d_elbow_config="$(arg r_elbow_config)"
     orbita3d_wrist_config="$(arg r_wrist_config)"
+    gripper_id="${right_gripper_id}"
+    gripper_port="${right_gripper_port}"
     />
   <!-- <link name="r_wrist_cam_frame"/> -->
