Commit message: Update URDF and ros conrtol files.

File: reachy_description/ros2_control/dynamixel_gripper.ros2_control.xacro (robot description, xacro)
@@ -1,5 +1,5 @@
 <?xml version="1.0" ?>
 <robot xmlns:xacro="http://www.ros.org/wiki/xacro">
-  <xacro:macro name="smart_gripper_control" params="name gripper_port gripper_id min_grasping_finger max_grasping_finger">
+  <xacro:macro name="dynamixel_gripper_control" params="name gripper_port gripper_id min_grasping_finger max_grasping_finger">
   <xacro:include filename="$(find pollen_generic_description)/ros2_control/joint.ros2_control.xacro"/>
     <ros2_control name="${name}" type="system">
@@ -7,5 +7,5 @@
         <!-- Use real hardware. -->
         <xacro:unless value="$(arg use_fake_hardware)">
-          <plugin>smart_gripper_dynamixel_system_hwi/SmartGripperDynamixelSystem</plugin>
+          <plugin>gripper_dynamixel_system_hwi/GripperDynamixelSystem</plugin>
           <param name="gripper_port">${gripper_port}</param>
           <param name="gripper_id">${gripper_id}</param>

File: reachy_description/urdf/arm.urdf.xacro (robot description, xacro)
@@ -4,5 +4,5 @@
   <xacro:include filename="$(find orbita3d_description)/urdf/orbita3d.urdf.xacro"/>
   <xacro:include filename="$(find orbita2d_description)/urdf/orbita2d.urdf.xacro"/>
-  <xacro:include filename="$(find reachy_description)/urdf/smartgripper.urdf.xacro"/>
+  <xacro:include filename="$(find reachy_description)/urdf/dynamixel_gripper.urdf.xacro"/>
   <!-- <!-\- Orbita2d config -\-> -->
   <!-- <xacro:arg name="orbita2d_shoulder_config" default="$(find orbita2d_description)/config/fake.yaml"/> -->
@@ -77,5 +77,5 @@
     config_file="${orbita3d_wrist_config}"
   />
-  <xacro:smartgripper
+  <xacro:dynamixel_gripper
     prefix="${p}" parent="${p}_wrist_ball_link" side="${side}"
     damping="${damping}" friction="${friction}"

File: reachy_description/urdf/dynamixel_gripper.urdf.xacro (robot description, xacro)
@@ -1,6 +1,6 @@
 <?xml version="1.0" ?>
 <robot xmlns:xacro="http://www.ros.org/wiki/xacro">
-<xacro:macro name="smartgripper" params="prefix parent side damping friction gripper_port gripper_id">
-  <xacro:include filename="$(find reachy_description)/ros2_control/smartgripper.ros2_control.xacro"/>
+<xacro:macro name="dynamixel_gripper" params="prefix parent side damping friction gripper_port gripper_id">
+  <xacro:include filename="$(find reachy_description)/ros2_control/dynamixel_gripper.ros2_control.xacro"/>
   <xacro:include filename="$(find pollen_generic_description)/urdf/materials.urdf.xacro"/>
   <xacro:property name="gripper_length" value="0.12"/>
@@ -97,5 +97,5 @@
     <mimic joint="${p}_finger" multiplier="-1" offset="0" />
   </joint>
-  <xacro:smart_gripper_control
+  <xacro:dynamixel_gripper_control
     name="${p}"
     gripper_port="${gripper_port}"
