Commit message: pretty substantial rework of the urdf...

File: reachy_controllers/dynamixel_control/dynamixel_description/ros2_control/dynamixel_gripper.ros2_control.xacro (robot description, xacro)
@@ -4,5 +4,5 @@
   <xacro:include filename="$(find dynamixel_description)/ros2_control/dynamixel_axis_control.ros2_control.xacro"/>
   <xacro:include filename="$(find dynamixel_description)/ros2_control/dynamixel_raw_motor_control.ros2_control.xacro"/>
-  <xacro:macro name="dynamixel_gripper_control" params="joint1 joint2 config_file ">
+  <xacro:macro name="dynamixel_gripper_control" params="name joint1 joint2 config_file ">
     <ros2_control name="${name}" type="system">
       <hardware>

File: reachy_description/urdf/reachy.urdf.xacro (robot description, xacro)
@@ -5,5 +5,7 @@
   <xacro:arg name="use_moveit_gazebo" default="false" />
   <xacro:include filename="$(find reachy_description)/urdf/head.urdf.xacro" />
-  <xacro:include filename="$(find arm_description)/urdf/arm.urdf.xacro" />
+  <xacro:include filename="$(find reachy_description)/urdf/arm.urdf.xacro" />
+  <xacro:include filename="$(find dynamixel_description)/urdf/dynamixel_gripper.urdf.xacro" />
+  <xacro:include filename="$(find dynamixel_description)/ros2_control/dynamixel_gripper.ros2_control.xacro" />
   <xacro:include filename="$(find pollen_generic_description)/urdf/inertial_primitives.urdf.xacro" />
   <xacro:include filename="$(find pollen_generic_description)/urdf/materials.urdf.xacro" />
@@ -32,8 +34,14 @@
   <!-- config  -->
   <xacro:arg name="antenna_config" default="$(find dynamixel_description)/config/two_fake.yaml"/>
-  <!-- <xacro:arg name="antenna_config" default="$(find dynamixel_description)/config/antennas.yaml"/> -->
   <xacro:arg name="neck_config" default="$(find orbita3d_description)/config/fake_neck.yaml" />
-  <xacro:arg name="right_arm_config" default="$(find arm_description)/config/fake_r_arm.yaml" />
-  <xacro:arg name="left_arm_config" default="$(find arm_description)/config/fake_l_arm.yaml" />
+  <xacro:arg name="right_shoulder_config" default="$(find orbita2d_description)/config/fake.yaml" />
+  <xacro:arg name="right_elbow_config" default="$(find orbita2d_description)/config/fake.yaml" />
+  <xacro:arg name="right_wrist_config" default="$(find orbita3d_description)/config/fake.yaml" />
+  <xacro:arg name="left_shoulder_config" default="$(find orbita2d_description)/config/fake.yaml" />
+  <xacro:arg name="left_elbow_config" default="$(find orbita2d_description)/config/fake.yaml" />
+  <xacro:arg name="left_wrist_config" default="$(find orbita3d_description)/config/fake.yaml" />
+  <!-- <xacro:arg name="right_arm_config" default="$(find arm_description)/config/fake_r_arm.yaml" /> -->
+  <!-- <xacro:arg name="left_arm_config" default="$(find arm_description)/config/fake_l_arm.yaml" /> -->
+  <xacro:arg name="grippers_config" default="$(find dynamixel_description)/config/two_fake.yaml"/>
   <xacro:arg name="robot_model" default="none" />
   <!-- config  -->
@@ -196,14 +204,92 @@
     prefix="r" parent="torso" side="right"
     damping="${damping}" friction="${friction}"
-    config_file="$(arg right_arm_config)"
+    shoulder_config_file="$(arg right_shoulder_config)"
+    elbow_config_file="$(arg right_elbow_config)"
+    wrist_config_file="$(arg right_wrist_config)"
     robot_model="$(arg robot_model)"
   />
+    <xacro:dynamixel_gripper
+      prefix="r_hand" parent="r_wrist_out_link" side="right"
+      damping="${damping}" friction="${friction}"
+    />
+    <link name="r_arm_tip">
+      <inertial>
+        <origin xyz="0.0 0.0 0.0" rpy="0.0 0.0 0.0" />
+        <mass value="0.001" />
+        <inertia ixx="1.0e-6" ixy="1.0e-8" ixz="1.0e-8" iyy="1.0e-6" iyz="1.0e-8" izz="1.0e-6" />
+      </inertial>
+    </link>
+    <joint name="r_tip_joint" type="fixed">
+      <!-- Rotated to be aligned with trunk in resting pos (elbows at -90°) -->
+      <!-- <origin xyz="-0.012 0 0.14432" rpy="${pi} ${-pi/2} 0" /> -->
+      <!-- <origin xyz="-0.012 0 0.14432" rpy="${pi} 0 0" /> -->
+      <!-- Aligned with trunk in zero position -->
+      <!-- <origin xyz="-0.012 0 0.14432" rpy="${pi} 0 0" /> -->
+      <!-- Hard coded in symbolic ik... -->
+      <origin xyz="0.0 0 0.10" rpy="${pi} 0 0" />
+      <parent link="r_hand_palm_link" />
+      <child link="r_arm_tip" />
+    </joint>
+    <link name="r_arm_tip_bottom">
+      <inertial>
+        <origin xyz="0.0 0.0 0.0" rpy="0.0 0.0 0.0" />
+        <mass value="0.001" />
+        <inertia ixx="1.0e-6" ixy="1.0e-8" ixz="1.0e-8" iyy="1.0e-6" iyz="1.0e-8" izz="1.0e-6" />
+      </inertial>
+    </link>
+    <joint name="r_tip_joint_bottom" type="fixed">
+      <!-- <origin xyz="-0.028 0 0.14432" rpy="${pi} ${-pi/2} 0" /> -->
+      <origin xyz="-0.028 0 0.14432" rpy="${pi} 0 0" />
+      <parent link="r_hand_palm_link" />
+      <child link="r_arm_tip_bottom" />
+    </joint>
   <!-- LEFT ARM -->
   <xacro:arm
     prefix="l" parent="torso" side="left"
     damping="${damping}" friction="${friction}"
-    config_file="$(arg left_arm_config)"
+    shoulder_config_file="$(arg left_shoulder_config)"
+    elbow_config_file="$(arg left_elbow_config)"
+    wrist_config_file="$(arg left_wrist_config)"
     robot_model="$(arg robot_model)"
   />
+    <xacro:dynamixel_gripper
+      prefix="l_hand" parent="l_wrist_out_link" side="right"
+      damping="${damping}" friction="${friction}"
+    />
+    <link name="l_arm_tip">
+      <inertial>
+        <origin xyz="0.0 0.0 0.0" rpy="0.0 0.0 0.0" />
+        <mass value="0.001" />
+        <inertia ixx="1.0e-6" ixy="1.0e-8" ixz="1.0e-8" iyy="1.0e-6" iyz="1.0e-8" izz="1.0e-6" />
+      </inertial>
+    </link>
+    <joint name="l_tip_joint" type="fixed">
+      <!-- Rotated to be aligned with trunk in resting pos (elbows at -90°) -->
+      <!-- <origin xyz="-0.012 0 0.14432" rpy="${pi} ${-pi/2} 0" /> -->
+      <!-- <origin xyz="-0.012 0 0.14432" rpy="${pi} 0 0" /> -->
+      <!-- Aligned with trunk in zero position -->
+      <!-- <origin xyz="-0.012 0 0.14432" rpy="${pi} 0 0" /> -->
+      <!-- Hard coded in symbolic ik... -->
+      <origin xyz="0.0 0 0.10" rpy="${pi} 0 0" />
+      <parent link="l_hand_palm_link" />
+      <child link="l_arm_tip" />
+    </joint>
+    <link name="l_arm_tip_bottom">
+      <inertial>
+        <origin xyz="0.0 0.0 0.0" rpy="0.0 0.0 0.0" />
+        <mass value="0.001" />
+        <inertia ixx="1.0e-6" ixy="1.0e-8" ixz="1.0e-8" iyy="1.0e-6" iyz="1.0e-8" izz="1.0e-6" />
+      </inertial>
+    </link>
+    <joint name="l_tip_joint_bottom" type="fixed">
+      <!-- <origin xyz="-0.028 0 0.14432" rpy="${pi} ${-pi/2} 0" /> -->
+      <origin xyz="-0.028 0 0.14432" rpy="${pi} 0 0" />
+      <parent link="l_hand_palm_link" />
+      <child link="l_arm_tip_bottom" />
+    </joint>
+  <xacro:dynamixel_gripper_control
+    name="gripper" joint1="l_hand" joint2="r_hand"
+    config_file="$(arg grippers_config)"
+    />
   <link name="depth_cam_l_optical">
     <inertial>

Commit message: wip with mimic plugin

File: reachy_controllers/dynamixel_control/dynamixel_description/ros2_control/dynamixel_gripper.ros2_control.xacro (robot description, xacro)
@@ -26,4 +26,5 @@
         </xacro:if>
       </hardware>
+      <!-- <xacro:unless value="$(arg use_gazebo)"> -->
       <xacro:dynamixel_actuator_control name="${joint1}"/>
       <xacro:dynamixel_actuator_control name="${joint2}"/>
@@ -32,5 +33,38 @@
       <xacro:dynamixel_raw_motor_control name="${joint1}_raw_motor_1"/>
       <xacro:dynamixel_raw_motor_control name="${joint2}_raw_motor_1"/>
+      <!-- </xacro:unless> -->
     </ros2_control>
+    <xacro:if value="$(arg use_gazebo)">
+        <!-- <xacro:mimic_joint_plugin_gazebo name_prefix="${joint1}_finger_proximal" following_joint="${joint1}_finger_proximal" mimic_joint="${joint1}_finger" multiplier="-0.4689" offset="0.554" has_pid="true"/> -->
+        <!-- <!-\- <xacro:mimic_joint_plugin_gazebo name_prefix="${joint1}_finger_proximal_mimic" following_joint="${joint1}_finger_proximal_mimic" mimic_joint="${joint1}_finger_proximal" multiplier="1" offset="0.0"/> -\-> -->
+        <!-- <xacro:mimic_joint_plugin_gazebo name_prefix="${joint1}_finger_proximal_mimic" following_joint="${joint1}_finger_proximal_mimic" mimic_joint="${joint1}_finger" multiplier="-0.4689" offset="0.554" has_pid="true"/> -->
+        <!-- <xacro:mimic_joint_plugin_gazebo name_prefix="${joint1}_finger_distal" following_joint="${joint1}_finger_distal" mimic_joint="${joint1}_finger" multiplier="0.4689" offset="0.0" has_pid="true"/> -->
+        <!-- <xacro:mimic_joint_plugin_gazebo name_prefix="${joint1}_finger_distal_mimic" following_joint="${joint1}_finger_distal" mimic_joint="${joint1}_finger" multiplier="0.4689" offset="0.0" has_pid="true"/> -->
+        <!-- <xacro:mimic_joint_plugin_gazebo name_prefix="${joint2}_finger_proximal" following_joint="${joint2}_finger_proximal" mimic_joint="${joint2}_finger" multiplier="-0.4689" offset="0.554" has_pid="true"/> -->
+        <!-- <!-\- <xacro:mimic_joint_plugin_gazebo name_prefix="${joint2}_finger_proximal_mimic" following_joint="${joint2}_finger_proximal_mimic" mimic_joint="${joint2}_finger_proximal" multiplier="1" offset="0.0"/> -\-> -->
+        <!-- <xacro:mimic_joint_plugin_gazebo name_prefix="${joint2}_finger_proximal_mimic" following_joint="${joint2}_finger_proximal_mimic" mimic_joint="${joint2}_finger" multiplier="-0.4689" offset="0.554" has_pid="true"/> -->
+        <!-- <xacro:mimic_joint_plugin_gazebo name_prefix="${joint2}_finger_distal" following_joint="${joint2}_finger_distal" mimic_joint="${joint2}_finger" multiplier="0.4689" offset="0.0" has_pid="true"/> -->
+        <!-- <xacro:mimic_joint_plugin_gazebo name_prefix="${joint2}_finger_distal_mimic" following_joint="${joint2}_finger_distal" mimic_joint="${joint2}_finger" multiplier="0.4689" offset="0.0" has_pid="true"/> -->
+        <!-- <xacro:mimic_joint_plugin_gazebo name_prefix="${joint1}_finger_proximal" following_joint="${joint1}_finger" mimic_joint="${joint1}_finger_proximal" multiplier="-0.4689" offset="0.554" has_pid="true"/> -->
+        <!-- <!-\- <xacro:mimic_joint_plugin_gazebo name_prefix="${joint1}_finger_proximal_mimic" following_joint="${joint1}_finger_proximal_mimic" mimic_joint="${joint1}_finger_proximal" multiplier="1" offset="0.0"/> -\-> -->
+        <!-- <xacro:mimic_joint_plugin_gazebo name_prefix="${joint1}_finger_proximal_mimic" following_joint="${joint1}_finger" mimic_joint="${joint1}_finger_proximal_mimic" multiplier="-0.4689" offset="0.554" has_pid="true"/> -->
+        <!-- <xacro:mimic_joint_plugin_gazebo name_prefix="${joint1}_finger_distal" following_joint="${joint1}_finger" mimic_joint="${joint1}_finger_distal" multiplier="0.4689" offset="0.0" has_pid="true"/> -->
+        <!-- <xacro:mimic_joint_plugin_gazebo name_prefix="${joint1}_finger_distal_mimic" following_joint="${joint1}_finger" mimic_joint="${joint1}_finger_distal" multiplier="0.4689" offset="0.0" has_pid="true"/> -->
+        <!-- <xacro:mimic_joint_plugin_gazebo name_prefix="${joint2}_finger_proximal" following_joint="${joint2}_finger" mimic_joint="${joint2}_finger_proximal" multiplier="-0.4689" offset="0.554" has_pid="true"/> -->
+        <!-- <!-\- <xacro:mimic_joint_plugin_gazebo name_prefix="${joint2}_finger_proximal_mimic" following_joint="${joint2}_finger_proximal_mimic" mimic_joint="${joint2}_finger_proximal" multiplier="1" offset="0.0"/> -\-> -->
+        <!-- <xacro:mimic_joint_plugin_gazebo name_prefix="${joint2}_finger_proximal_mimic" following_joint="${joint2}_finger" mimic_joint="${joint2}_finger_proximal_mimic" multiplier="-0.4689" offset="0.554" has_pid="true"/> -->
+        <!-- <xacro:mimic_joint_plugin_gazebo name_prefix="${joint2}_finger_distal" following_joint="${joint2}_finger" mimic_joint="${joint2}_finger_distal" multiplier="0.4689" offset="0.0" has_pid="true"/> -->
+        <!-- <xacro:mimic_joint_plugin_gazebo name_prefix="${joint2}_finger_distal_mimic" following_joint="${joint2}_finger" mimic_joint="${joint2}_finger_distal" multiplier="0.4689" offset="0.0" has_pid="true"/> -->
+        <xacro:mimic_joint_plugin_gazebo name_prefix="${joint1}_finger_proximal" following_joint="${joint1}_finger" mimic_joint="${joint1}_finger_proximal" multiplier="-0.4689" offset="0.554"/>
+        <!-- <xacro:mimic_joint_plugin_gazebo name_prefix="${joint1}_finger_proximal_mimic" following_joint="${joint1}_finger_proximal_mimic" mimic_joint="${joint1}_finger_proximal" multiplier="1" offset="0.0"/> -->
+        <xacro:mimic_joint_plugin_gazebo name_prefix="${joint1}_finger_proximal_mimic" following_joint="${joint1}_finger" mimic_joint="${joint1}_finger_proximal_mimic" multiplier="-0.4689" offset="0.554" />
+        <xacro:mimic_joint_plugin_gazebo name_prefix="${joint1}_finger_distal" following_joint="${joint1}_finger" mimic_joint="${joint1}_finger_distal" multiplier="0.4689" offset="-0.554" />
+        <xacro:mimic_joint_plugin_gazebo name_prefix="${joint1}_finger_distal_mimic" following_joint="${joint1}_finger" mimic_joint="${joint1}_finger_distal_mimic" multiplier="0.4689" offset="-0.554" />
+        <xacro:mimic_joint_plugin_gazebo name_prefix="${joint2}_finger_proximal" following_joint="${joint2}_finger" mimic_joint="${joint2}_finger_proximal" multiplier="-0.4689" offset="0.554"/>
+        <!-- <xacro:mimic_joint_plugin_gazebo name_prefix="${joint2}_finger_proximal_mimic" following_joint="${joint2}_finger_proximal_mimic" mimic_joint="${joint2}_finger_proximal" multiplier="1" offset="0.0"/> -->
+        <xacro:mimic_joint_plugin_gazebo name_prefix="${joint2}_finger_proximal_mimic" following_joint="${joint2}_finger" mimic_joint="${joint2}_finger_proximal_mimic" multiplier="-0.4689" offset="0.554" />
+        <xacro:mimic_joint_plugin_gazebo name_prefix="${joint2}_finger_distal" following_joint="${joint2}_finger" mimic_joint="${joint2}_finger_distal" multiplier="0.4689" offset="-0.554" />
+        <xacro:mimic_joint_plugin_gazebo name_prefix="${joint2}_finger_distal_mimic" following_joint="${joint2}_finger" mimic_joint="${joint2}_finger_distal_mimic" multiplier="0.4689" offset="-0.554" />
+    </xacro:if>
   </xacro:macro>
 </robot>

File: reachy_controllers/dynamixel_control/dynamixel_description/ros2_control/dynamixel_gripper_axis_control.ros2_control.xacro (robot description, xacro)
@@ -1,4 +1,5 @@
 <?xml version="1.0" ?>
 <robot xmlns:xacro="http://www.ros.org/wiki/xacro">
+  <xacro:include filename="$(find reachy_description)/urdf/gz_mimic.urdf.xacro" />
   <xacro:macro name="dynamixel_gripper_axis_control" params="name fake gazebo" >
     <joint name="${name}">
@@ -17,40 +18,71 @@
       <!-- Use gazebo as hardware simulation, then handle the mimic joints. -->
       <xacro:if value="${gazebo}">
-	<joint name="${name}_proximal">
-	  <param name="mimic">${name}_finger</param>
-	  <param name="multiplier">-0.4689</param>
-	  <!-- offset = 0.554 WHY DIDN'T YOU IMPLEMENT THAT?!! -->
-        <!-- <param name="initial_value">0.554</param> -->
-	  <command_interface name="position"/>
-	  <state_interface name="position"/>
-	  <state_interface name="velocity"/>
-	  <state_interface name="effort"/>
-	</joint>
-	<joint name="${name}_proximal_mimic" >
-	  <param name="mimic">${name}_finger_proximal</param>
-	  <param name="multiplier">1</param>
-	  <command_interface name="position"/>
-	  <state_interface name="position"/>
-	  <state_interface name="velocity"/>
-	  <state_interface name="effort"/>
-	</joint>
-	<joint name="${name}_distal" >
-	  <param name="mimic">${name}_finger</param>
-	  <param name="multiplier">0.4689</param>
-	  <!-- offset = -0.554 WHY DIDN'T YOU IMPLEMENT THAT?!! -->
-	  <command_interface name="position"/>
-	  <state_interface name="position"/>
-	  <state_interface name="velocity"/>
-	  <state_interface name="effort"/>
-	</joint>
-	<joint name="${name}_distal_mimic">
-	  <param name="mimic">${name}_finger</param>
-	  <param name="multiplier">0.4689</param>
-	  <!-- offset = -0.554 WHY DIDN'T YOU IMPLEMENT THAT?!! -->
-	  <command_interface name="position"/>
-	  <state_interface name="position"/>
-	  <state_interface name="velocity"/>
-	  <state_interface name="effort"/>
-	</joint>
+        <!-- <xacro:mimic_joint_plugin_gazebo name_prefix="${name}_proximal" following_joint="${name}_proximal" mimic_joint="${name}_finger" multiplier="-0.4689" offset="0.554"/> -->
+        <!-- <joint name="${name}_proximal"> -->
+        <!--   <param name="mimic">${name}_finger</param> -->
+        <!--   <param name="multiplier">-0.4689</param> -->
+        <!--   <!-\- offset = 0.554 WHY DIDN'T YOU IMPLEMENT THAT?!! -\-> -->
+        <!-- <!-\- <param name="initial_value">0.554</param> -\-> -->
+        <!--   <command_interface name="position"/> -->
+        <!--   <state_interface name="position"/> -->
+        <!--   <state_interface name="velocity"/> -->
+        <!--   <state_interface name="effort"/> -->
+        <!-- </joint> -->
+        <!-- <!-\- <xacro:mimic_joint_plugin_gazebo name_prefix="${name}_proximal_mimic" following_joint="${name}_proximal_mimic" mimic_joint="${name}_finger_proximal" multiplier="1" offset="0.0"/> -\-> -->
+        <!-- <joint name="${name}_proximal_mimic" > -->
+        <!--   <param name="mimic">${name}_finger_proximal</param> -->
+        <!--   <param name="multiplier">1</param> -->
+        <!--   <command_interface name="position"/> -->
+        <!--   <state_interface name="position"/> -->
+        <!--   <state_interface name="velocity"/> -->
+        <!--   <state_interface name="effort"/> -->
+        <!-- </joint> -->
+        <!-- <!-\- <xacro:mimic_joint_plugin_gazebo name_prefix="${name}_distal" following_joint="${name}_distal" mimic_joint="${name}_finger" multiplier="0.4689" offset="0.0"/> -\-> -->
+        <!-- <joint name="${name}_distal" > -->
+        <!--   <param name="mimic">${name}_finger</param> -->
+        <!--   <param name="multiplier">0.4689</param> -->
+        <!--   <!-\- offset = -0.554 WHY DIDN'T YOU IMPLEMENT THAT?!! -\-> -->
+        <!--   <command_interface name="position"/> -->
+        <!--   <state_interface name="position"/> -->
+        <!--   <state_interface name="velocity"/> -->
+        <!--   <state_interface name="effort"/> -->
+        <!-- </joint> -->
+        <!-- <!-\- <xacro:mimic_joint_plugin_gazebo name_prefix="${name}_distal_mimic" following_joint="${name}_distal" mimic_joint="${name}_finger" multiplier="0.4689" offset="0.0"/> -\-> -->
+        <!-- <joint name="${name}_distal_mimic"> -->
+        <!--   <param name="mimic">${name}_finger</param> -->
+        <!--   <param name="multiplier">0.4689</param> -->
+        <!--   <!-\- offset = -0.554 WHY DIDN'T YOU IMPLEMENT THAT?!! -\-> -->
+        <!--   <command_interface name="position"/> -->
+        <!--   <state_interface name="position"/> -->
+        <!--   <state_interface name="velocity"/> -->
+        <!--   <state_interface name="effort"/> -->
+        <!-- </joint> -->
+        <joint name="${name}_proximal">
+          <command_interface name="position"/>
+          <state_interface name="position"/>
+          <state_interface name="velocity"/>
+          <state_interface name="effort"/>
+        </joint>
+        <!-- <xacro:mimic_joint_plugin_gazebo name_prefix="${name}_proximal_mimic" following_joint="${name}_proximal_mimic" mimic_joint="${name}_finger_proximal" multiplier="1" offset="0.0"/> -->
+        <joint name="${name}_proximal_mimic" >
+          <command_interface name="position"/>
+          <state_interface name="position"/>
+          <state_interface name="velocity"/>
+          <state_interface name="effort"/>
+        </joint>
+        <!-- <xacro:mimic_joint_plugin_gazebo name_prefix="${name}_distal" following_joint="${name}_distal" mimic_joint="${name}_finger" multiplier="0.4689" offset="0.0"/> -->
+        <joint name="${name}_distal" >
+          <command_interface name="position"/>
+          <state_interface name="position"/>
+          <state_interface name="velocity"/>
+          <state_interface name="effort"/>
+        </joint>
+        <!-- <xacro:mimic_joint_plugin_gazebo name_prefix="${name}_distal_mimic" following_joint="${name}_distal" mimic_joint="${name}_finger" multiplier="0.4689" offset="0.0"/> -->
+        <joint name="${name}_distal_mimic">
+          <command_interface name="position"/>
+          <state_interface name="position"/>
+          <state_interface name="velocity"/>
+          <state_interface name="effort"/>
+        </joint>
       </xacro:if>
     </xacro:if>

File: reachy_controllers/dynamixel_control/dynamixel_description/urdf/dynamixel_gripper.urdf.xacro (robot description, xacro)
@@ -3,4 +3,5 @@
 <xacro:macro name="dynamixel_gripper" params="prefix parent side damping friction ">
   <xacro:include filename="$(find pollen_generic_description)/urdf/materials.urdf.xacro"/>
+  <xacro:include filename="$(find pollen_generic_description)/urdf/inertial_primitives.urdf.xacro"/>
   <xacro:property name="gripper_length" value="0.12"/>
   <xacro:property name="gripper_radius" value="0.03"/>
@@ -78,9 +79,11 @@
   </joint>
   <link name="${p}_virtual_gripper_link">
-      <inertial>
-        <origin xyz="0.0 0.0 0.0" rpy="0.0 0.0 0.0"/>
-        <mass value="0.01"/>
-        <inertia ixx="1.0e-6" ixy="1.0e-8" ixz="1.0e-8" iyy="1.0e-6" iyz="1.0e-8" izz="1.0e-6"/>
-      </inertial>
+      <!-- <inertial> -->
+      <!--   <origin xyz="0.0 0.0 0.0" rpy="0.0 0.0 0.0"/> -->
+      <!--   <mass value="0.01"/> -->
+      <!--   <inertia ixx="1.0e-6" ixy="1.0e-8" ixz="1.0e-8" iyy="1.0e-6" iyz="1.0e-8" izz="1.0e-6"/> -->
+      <!-- </inertial> -->
+      <xacro:inertial_cuboid mass="${0.01}" xyz="0 0 0"  rpy="0 0 0" x_length="0.01" y_length="0.01" z_length="0.01">
+      </xacro:inertial_cuboid>
   </link>
   <joint name="${p}_finger" type="revolute">
@@ -225,4 +228,34 @@
   <!--   <selfCollide>false</selfCollide> -->
   <!-- </gazebo> -->
+  <xacro:if value="$(arg use_gazebo)">
+    <gazebo reference="${p}_palm_link">
+      <selfCollide>false</selfCollide>
+      <implicitSpringDamper>True</implicitSpringDamper>
+    </gazebo>
+  </xacro:if>
+  <xacro:if value="$(arg use_gazebo)">
+    <gazebo reference="${p}_proximal_link">
+      <selfCollide>false</selfCollide>
+      <implicitSpringDamper>True</implicitSpringDamper>
+    </gazebo>
+  </xacro:if>
+  <xacro:if value="$(arg use_gazebo)">
+    <gazebo reference="${p}_proximal_mimic_link">
+      <selfCollide>false</selfCollide>
+      <implicitSpringDamper>True</implicitSpringDamper>
+    </gazebo>
+  </xacro:if>
+  <xacro:if value="$(arg use_gazebo)">
+    <gazebo reference="${p}_distal_link">
+      <selfCollide>false</selfCollide>
+      <implicitSpringDamper>True</implicitSpringDamper>
+    </gazebo>
+  </xacro:if>
+  <xacro:if value="$(arg use_gazebo)">
+    <gazebo reference="${p}_distal_mimic_link">
+      <selfCollide>false</selfCollide>
+      <implicitSpringDamper>True</implicitSpringDamper>
+    </gazebo>
+  </xacro:if>
 </xacro:macro>
 </robot>
