Commit message: seems to work ok in fake

File: reachy_controllers/dynamixel_control/dynamixel_description/ros2_control/dynamixel.ros2_control.xacro (robot description, xacro)
@@ -1,6 +1,8 @@
 <?xml version="1.0" ?>
 <robot xmlns:xacro="http://www.ros.org/wiki/xacro">
-  <xacro:macro name="dynamixel_control" params="name config_file">
-  <xacro:include filename="$(find pollen_generic_description)/ros2_control/joint.ros2_control.xacro"/>
+  <xacro:include filename="$(find dynamixel_description)/ros2_control/dynamixel_actuator_control.ros2_control.xacro"/>
+  <xacro:include filename="$(find dynamixel_description)/ros2_control/dynamixel_axis_control.ros2_control.xacro"/>
+  <xacro:include filename="$(find dynamixel_description)/ros2_control/dynamixel_raw_motor_control.ros2_control.xacro"/>
+  <xacro:macro name="dynamixel_control" params="name joint1 joint2 config_file ">
     <ros2_control name="${name}" type="system">
       <hardware>
@@ -21,6 +23,10 @@
         </xacro:if>
       </hardware>
-      <xacro:position_joint_control name="${name}_left_joint"/>
-      <xacro:position_joint_control name="${name}_right_joint"/>
+      <xacro:dynamixel_actuator_control name="${name}_${joint1}"/>
+      <xacro:dynamixel_actuator_control name="${name}_${joint2}"/>
+      <xacro:dynamixel_axis_control name="${name}_${joint1}"/>
+      <xacro:dynamixel_axis_control name="${name}_${joint2}"/>
+      <xacro:dynamixel_raw_motor_control name="${name}_raw_motor_${joint1}"/>
+      <xacro:dynamixel_raw_motor_control name="${name}_raw_motor_${joint2}"/>
     </ros2_control>
   </xacro:macro>

File: reachy_description/urdf/head.urdf.xacro (robot description, xacro)
@@ -101,5 +101,5 @@
     </joint>
     <!-- test antennas -->
-    <link name="antenna_left" >
+    <link name="antenna_left_link" >
       <inertial>
 	<origin xyz="0.0 0.0 0.0" rpy="0.0 0.0 0.0"/>
@@ -117,12 +117,12 @@
     </link>
     <!-- revolute joint -->
-    <joint name="antenna_left_joint" type="revolute">
+    <joint name="antenna_left" type="revolute">
       <origin xyz="0.0 0.1 0.1" rpy="0 0.0 0"/>
       <parent link="head" />
-      <child link="antenna_left" />
+      <child link="antenna_left_link" />
       <axis xyz="0 1 0"/>
       <limit effort="0.0" velocity="0.0" lower="-0.5" upper="0.5"/>
     </joint>
-    <link name="antenna_right" >
+    <link name="antenna_right_link" >
       <inertial>
 	<origin xyz="0.0 0.0 0.0" rpy="0.0 0.0 0.0"/>
@@ -140,13 +140,13 @@
     </link>
     <!-- revolute joint -->
-    <joint name="antenna_right_joint" type="revolute">
+    <joint name="antenna_right" type="revolute">
       <origin xyz="0.0 -0.1 0.1" rpy="0 0.0 0"/>
       <parent link="head" />
-      <child link="antenna_right" />
+      <child link="antenna_right_link" />
       <axis xyz="0 1 0"/>
       <limit effort="0.0" velocity="0.0" lower="-0.5" upper="0.5"/>
     </joint>
   <xacro:dynamixel_control
-    name="antenna"
+    name="antenna" joint1="left" joint2="right"
     config_file="${antenna_config}"
     />

Commit message: grippers dont move in gazebo

File: reachy_controllers/dynamixel_control/dynamixel_description/ros2_control/dynamixel.ros2_control.xacro (robot description, xacro)
@@ -3,4 +3,5 @@
   <xacro:include filename="$(find dynamixel_description)/ros2_control/dynamixel_actuator_control.ros2_control.xacro"/>
   <xacro:include filename="$(find dynamixel_description)/ros2_control/dynamixel_axis_control.ros2_control.xacro"/>
+  <!-- <xacro:include filename="$(find dynamixel_description)/ros2_control/dynamixel_gripper_axis_control.ros2_control.xacro"/> -->
   <xacro:include filename="$(find dynamixel_description)/ros2_control/dynamixel_raw_motor_control.ros2_control.xacro"/>
   <xacro:macro name="dynamixel_control" params="name joint1 joint2 config_file ">
@@ -30,4 +31,6 @@
       <xacro:dynamixel_axis_control name="${name}_${joint1}" />
       <xacro:dynamixel_axis_control name="${name}_${joint2}" />
+      <!-- <xacro:dynamixel_gripper_axis_control name="${joint1}_finger" fake="$(arg use_fake_hardware)" gazebo="$(arg use_gazebo)"/> -->
+      <!-- <xacro:dynamixel_gripper_axis_control name="${joint2}_finger" fake="$(arg use_fake_hardware)" gazebo="$(arg use_gazebo)"/> -->
       <xacro:dynamixel_raw_motor_control name="${name}_${joint1}_raw_motor"/>
       <xacro:dynamixel_raw_motor_control name="${name}_${joint2}_raw_motor"/>

File: reachy_controllers/dynamixel_control/dynamixel_description/ros2_control/dynamixel_gripper.ros2_control.xacro (robot description, xacro)
@@ -2,8 +2,8 @@
 <robot xmlns:xacro="http://www.ros.org/wiki/xacro">
   <xacro:include filename="$(find dynamixel_description)/ros2_control/dynamixel_actuator_control.ros2_control.xacro"/>
-  <!-- <xacro:include filename="$(find dynamixel_description)/ros2_control/dynamixel_gripper_axis_control.ros2_control.xacro"/> -->
-  <xacro:include filename="$(find dynamixel_description)/ros2_control/dynamixel_axis_control.ros2_control.xacro"/>
+  <xacro:include filename="$(find dynamixel_description)/ros2_control/dynamixel_gripper_axis_control.ros2_control.xacro"/>
+  <!-- <xacro:include filename="$(find dynamixel_description)/ros2_control/dynamixel_axis_control.ros2_control.xacro"/> -->
   <xacro:include filename="$(find dynamixel_description)/ros2_control/dynamixel_raw_motor_control.ros2_control.xacro"/>
-  <xacro:macro name="dynamixel_gripper_control" params="name joint1 joint2 config_file ">
+  <xacro:macro name="dynamixel_gripper_control" params="name joint1 joint2 config_file">
     <ros2_control name="${name}" type="system">
       <hardware>
@@ -29,8 +29,12 @@
       <xacro:dynamixel_actuator_control name="${joint1}"/>
       <xacro:dynamixel_actuator_control name="${joint2}"/>
-      <xacro:dynamixel_axis_control name="${joint1}_finger"/>
-      <xacro:dynamixel_axis_control name="${joint2}_finger"/>
+      <!-- <xacro:dynamixel_axis_control name="${joint1}_finger"/> -->
+      <!-- <xacro:dynamixel_axis_control name="${joint2}_finger"/> -->
       <!-- <xacro:dynamixel_gripper_axis_control name="${joint1}_finger" fake="$(arg use_fake_hardware)" gazebo="$(arg use_gazebo)"/> -->
       <!-- <xacro:dynamixel_gripper_axis_control name="${joint2}_finger" fake="$(arg use_fake_hardware)" gazebo="$(arg use_gazebo)"/> -->
+      <!-- <xacro:dynamixel_gripper_axis_control name="${joint1}_finger" fake="${use_fake_hardware}" gazebo="${use_gazebo}"/> -->
+      <!-- <xacro:dynamixel_gripper_axis_control name="${joint2}_finger" fake="${use_fake_hardware}" gazebo="${use_gazebo}"/> -->
+      <xacro:dynamixel_gripper_axis_control name="${joint1}_finger"/>
+      <xacro:dynamixel_gripper_axis_control name="${joint2}_finger"/>
       <xacro:dynamixel_raw_motor_control name="${joint1}_raw_motor_1"/>
       <xacro:dynamixel_raw_motor_control name="${joint2}_raw_motor_1"/>

File: reachy_controllers/dynamixel_control/dynamixel_description/ros2_control/dynamixel_gripper_axis_control.ros2_control.xacro (robot description, xacro)
@@ -1,5 +1,5 @@
 <?xml version="1.0" ?>
 <robot xmlns:xacro="http://www.ros.org/wiki/xacro">
-  <xacro:macro name="dynamixel_gripper_axis_control" params="name fake gazebo" >
+  <xacro:macro name="dynamixel_gripper_axis_control" params="name" >
     <joint name="${name}">
       <state_interface name="position">
@@ -14,42 +14,42 @@
       <command_interface name="position"/>
     </joint>
-    <xacro:if value="${fake}">
+    <xacro:if value="$(arg use_fake_hardware)">
+      <xacro:if value="$(arg use_gazebo)">
       <!-- Use gazebo as hardware simulation, then handle the mimic joints. -->
-      <xacro:if value="${gazebo}">
 	<joint name="${name}_proximal">
-	  <param name="mimic">${name}_finger</param>
-	  <param name="multiplier">-0.4689</param>
-	  <!-- offset = 0.554 WHY DIDN'T YOU IMPLEMENT THAT?!! -->
-        <!-- <param name="initial_value">0.554</param> -->
-	  <command_interface name="position"/>
-	  <state_interface name="position"/>
-	  <state_interface name="velocity"/>
-	  <state_interface name="effort"/>
+	  <!-- <param name="mimic">${name}_finger</param> -->
+	<!--   <param name="multiplier">-0.4689</param> -->
+	<!--   <!-\- offset = 0.554 WHY DIDN'T YOU IMPLEMENT THAT?!! -\-> -->
+        <!-- <!-\- <param name="initial_value">0.554</param> -\-> -->
+	<!--   <command_interface name="position"/> -->
+	<!--   <state_interface name="position"/> -->
+	<!--   <state_interface name="velocity"/> -->
+	<!--   <state_interface name="effort"/> -->
 	</joint>
 	<joint name="${name}_proximal_mimic" >
-	  <param name="mimic">${name}_finger_proximal</param>
-	  <param name="multiplier">1</param>
-	  <command_interface name="position"/>
-	  <state_interface name="position"/>
-	  <state_interface name="velocity"/>
-	  <state_interface name="effort"/>
+	  <!-- <param name="mimic">${name}_finger_proximal</param> -->
+	  <!-- <param name="multiplier">1</param> -->
+	  <!-- <command_interface name="position"/> -->
+	  <!-- <state_interface name="position"/> -->
+	  <!-- <state_interface name="velocity"/> -->
+	  <!-- <state_interface name="effort"/> -->
 	</joint>
 	<joint name="${name}_distal" >
-	  <param name="mimic">${name}_finger</param>
-	  <param name="multiplier">0.4689</param>
-	  <!-- offset = -0.554 WHY DIDN'T YOU IMPLEMENT THAT?!! -->
-	  <command_interface name="position"/>
-	  <state_interface name="position"/>
-	  <state_interface name="velocity"/>
-	  <state_interface name="effort"/>
+	  <!-- <param name="mimic">${name}_finger</param> -->
+	  <!-- <param name="multiplier">0.4689</param> -->
+	  <!-- <!-\- offset = -0.554 WHY DIDN'T YOU IMPLEMENT THAT?!! -\-> -->
+	  <!-- <command_interface name="position"/> -->
+	  <!-- <state_interface name="position"/> -->
+	  <!-- <state_interface name="velocity"/> -->
+	  <!-- <state_interface name="effort"/> -->
 	</joint>
 	<joint name="${name}_distal_mimic">
-	  <param name="mimic">${name}_finger</param>
-	  <param name="multiplier">0.4689</param>
-	  <!-- offset = -0.554 WHY DIDN'T YOU IMPLEMENT THAT?!! -->
-	  <command_interface name="position"/>
-	  <state_interface name="position"/>
-	  <state_interface name="velocity"/>
-	  <state_interface name="effort"/>
+	  <!-- <param name="mimic">${name}_finger</param> -->
+	  <!-- <param name="multiplier">0.4689</param> -->
+	  <!-- <!-\- offset = -0.554 WHY DIDN'T YOU IMPLEMENT THAT?!! -\-> -->
+	  <!-- <command_interface name="position"/> -->
+	  <!-- <state_interface name="position"/> -->
+	  <!-- <state_interface name="velocity"/> -->
+	  <!-- <state_interface name="effort"/> -->
 	</joint>
       </xacro:if>

File: reachy_controllers/dynamixel_control/dynamixel_description/urdf/dynamixel_gripper.urdf.xacro (robot description, xacro)
@@ -27,10 +27,6 @@
       <xacro:if value="${side == 'right'}">
     <collision>
-      <!-- <origin xyz="0 0 0.04 " rpy="0 0 0"/> -->
       <origin xyz="0 0 0.0 " rpy="0 0 0"/>
       <geometry>
-        <!-- <box size="${gripper_radius} ${gripper_radius*2} ${gripper_length/2}"/> -->
-        <!-- <box size="0.08 0.12 0.07"/> -->
-	  <!-- <mesh filename="package://arm_description/meshes/pincette_right_collider.dae" /> -->
 	  <mesh filename="file://$(find dynamixel_description)/meshes/pincette_right_collider.dae" />
       </geometry>
@@ -47,16 +43,12 @@
 	<mass value="0.30798029"/>
 	<inertia ixx="0.00021928" ixy="-0.00003149" ixz="-0.00001759"
-		 iyx="-0.00003149" iyy="0.00016859" iyz="-0.00001396"
-		 izx="-0.00001759" izy="-0.00001396" izz="0.0002333"/>
+		  iyy="0.00016859" iyz="-0.00001396"
+		  izz="0.0002333"/>
       </inertial>
    </xacro:if>
   <xacro:if value="${side == 'left'}">
     <collision>
-      <!-- <origin xyz="0 0 0.04 " rpy="0 0 0"/> -->
       <origin xyz="0 0 0.0 " rpy="0 0 0"/>
       <geometry>
-        <!-- <box size="${gripper_radius} ${gripper_radius*2} ${gripper_length/2}"/> -->
-        <!-- <box size="0.08 0.12 0.07"/> -->
-	  <!-- <mesh filename="file://$(find arm_description)/meshes/pincette_left_collider.dae" /> -->
 	  <mesh filename="file://$(find dynamixel_description)/meshes/pincette_left_collider.dae" />
       </geometry>
@@ -73,6 +65,6 @@
 	<mass value="0.30798029"/>
 	<inertia ixx="0.00021812" ixy="0.00003057" ixz="-0.00001759"
-		 iyx="0.00003057" iyy="0.00016868" iyz="0.00001416"
-		 izx="-0.00001759" izy="0.00001416" izz="0.00023207"/>
+		  iyy="0.00016868" iyz="0.00001416"
+		  izz="0.00023207"/>
       </inertial>
   </xacro:if>
@@ -87,5 +79,5 @@
         <origin xyz="0.0 0.0 0.0" rpy="0.0 0.0 0.0"/>
         <mass value="0.01"/>
-        <inertia ixx="1.0e-6" ixy="1.0e-8" ixz="1.0e-8" iyy="1.0e-6" iyz="1.0e-8" izz="1.0e-6"/>
+        <inertia ixx="1.0e-5" ixy="1.0e-6" ixz="1.0e-6" iyy="1.0e-5" iyz="1.0e-6" izz="1.0e-5"/>
       </inertial>
   </link>
@@ -103,15 +95,10 @@
 	<mass value="0.03926395"/>
 	 <inertia ixx="0.00001937" ixy="0.0" ixz="0.00000007"
-		  iyx="0.0" iyy="0.00002003" iyz="0.00000036"
-		  izx="0.00000007" izy="0.00000036" izz="0.00000463"/>
-      </inertial>
-    <collision>
-      <!-- <origin xyz="0 0.006 0.03 " rpy="0 0 0"/> -->
-      <!-- <geometry> -->
-      <!--   <box size="0.031 0.026 0.06"/> -->
-      <!-- </geometry> -->
+		   iyy="0.00002003" iyz="0.00000036"
+		   izz="0.00000463"/>
+      </inertial>
+    <collision>
       <origin xyz="0 0.00 0.0 " rpy="0 0 0"/>
       <geometry>
-	  <!-- <mesh filename="file://$(find arm_description)/meshes/pincette_proximal_collider.dae" /> -->
 	  <mesh filename="file://$(find dynamixel_description)/meshes/pincette_proximal_collider.dae" />
       </geometry>
@@ -120,5 +107,4 @@
       <origin xyz="0 0 0 " rpy="0 0 0"/>
       <geometry>
-	  <!-- <mesh filename="file://$(find arm_description)/meshes/pincette_proximal_visual.dae" /> -->
 	  <mesh filename="file://$(find dynamixel_description)/meshes/pincette_proximal_visual.dae" />
       </geometry>
@@ -130,13 +116,10 @@
 	<mass value="0.03926395"/>
 	 <inertia ixx="0.00001937" ixy="0.0" ixz="0.00000007"
-		  iyx="0.0" iyy="0.00002003" iyz="0.00000036"
-		  izx="0.00000007" izy="0.00000036" izz="0.00000463"/>
-      </inertial>
-    <collision>
-      <!-- <origin xyz="0 0.006 0.03 " rpy="0 0 0"/> -->
+		   iyy="0.00002003" iyz="0.00000036"
+		   izz="0.00000463"/>
+      </inertial>
+    <collision>
       <origin xyz="0 0.0 0.0 " rpy="0 0 0"/>
       <geometry>
-        <!-- <box size="0.031 0.026 0.06"/> -->
-	  <!-- <mesh filename="file://$(find arm_description)/meshes/pincette_proximal_collider.dae" /> -->
 	  <mesh filename="file://$(find dynamixel_description)/meshes/pincette_proximal_collider.dae" />
       </geometry>
@@ -145,5 +128,4 @@
       <origin xyz="0 0 0 " rpy="0 0 0"/>
       <geometry>
-	  <!-- <mesh filename="file://$(find arm_description)/meshes/pincette_proximal_visual.dae" /> -->
 	  <mesh filename="file://$(find dynamixel_description)/meshes/pincette_proximal_visual.dae" />
       </geometry>
@@ -155,6 +137,7 @@
     <child link="${p}_proximal_link"/>
     <axis xyz="1 0 0"/>
-    <limit lower="${min_grasping_finger}" upper="${max_grasping_finger}" effort="100.0" velocity="10.0"/>
+    <limit lower="${min_grasping_finger}" upper="${max_grasping_finger}" effort="10.0" velocity="1.0"/>
     <mimic joint="${p}_finger" multiplier="-0.4689" offset="0.554" />
+    <!-- <mimic joint="${p}_finger" multiplier="-0.4689" offset="0.0" /> -->
     <dynamics damping="${damping}" friction="${friction}"/>
   </joint>
@@ -164,5 +147,5 @@
     <child link="${p}_proximal_mimic_link"/>
     <axis xyz="1 0 0"/>
-    <limit lower="${min_grasping_finger}" upper="${max_grasping_finger}" effort="100.0" velocity="10.0"/>
+    <limit lower="${min_grasping_finger}" upper="${max_grasping_finger}" effort="10.0" velocity="1.0"/>
     <dynamics damping="${damping}" friction="${friction}"/>
     <mimic joint="${p}_finger_proximal" multiplier="1" offset="0" />
@@ -173,13 +156,10 @@
 	<mass value="0.02821091"/>
 	 <inertia ixx="0.00000683" ixy="0.0" ixz="0.0"
-		  iyx="0.0" iyy="0.00000696" iyz="0.00000127"
-		  izx="0.0" izy="0.00000127" izz="0.0000028"/>
-      </inertial>
-    <collision>
-      <!-- <origin xyz="0 0.0015 0.023 " rpy="0 0 0"/> -->
+		   iyy="0.00000696" iyz="0.00000127"
+		   izz="0.0000028"/>
+      </inertial>
+    <collision>
       <origin xyz="0 0.0 0.0 " rpy="0 0 0"/>
       <geometry>
-        <!-- <box size="0.031 0.026 0.046"/> -->
-	  <!-- <mesh filename="file://$(find arm_description)/meshes/pincette_distal_collider.dae" /> -->
 	  <mesh filename="file://$(find dynamixel_description)/meshes/pincette_distal_collider.dae" />
       </geometry>
@@ -198,7 +178,7 @@
     <child link="${p}_distal_link"/>
     <axis xyz="1 0 0"/>
-    <limit lower="${min_grasping_finger}" upper="${max_grasping_finger}" effort="100.0" velocity="10.0"/>
-    <!-- <mimic joint="${p}_finger_proximal" multiplier="-1" offset="0" /> -->
+    <limit lower="${min_grasping_finger}" upper="${max_grasping_finger}" effort="10.0" velocity="1.0"/>
     <mimic joint="${p}_finger" multiplier="0.4689" offset="-0.554" />
+    <!-- <mimic joint="${p}_finger" multiplier="0.4689" offset="0" /> -->
     <dynamics damping="${damping}" friction="${friction}"/>
   </joint>
@@ -208,13 +188,10 @@
 	<mass value="0.02821091"/>
 	 <inertia ixx="0.00000683" ixy="0.0" ixz="0.0"
-		  iyx="0.0" iyy="0.00000696" iyz="0.00000127"
-		  izx="0.0" izy="0.00000127" izz="0.0000028"/>
-      </inertial>
-    <collision>
-      <!-- <origin xyz="0 0.0015 0.023 " rpy="0 0 0"/> -->
+		   iyy="0.00000696" iyz="0.00000127"
+		   izz="0.0000028"/>
+      </inertial>
+    <collision>
       <origin xyz="0 0.00 0.0 " rpy="0 0 0"/>
       <geometry>
-        <!-- <box size="0.031 0.026 0.046"/> -->
-	  <!-- <mesh filename="file://$(find arm_description)/meshes/pincette_distal_collider.dae" /> -->
 	  <mesh filename="file://$(find dynamixel_description)/meshes/pincette_distal_collider.dae" />
       </geometry>
@@ -233,15 +210,14 @@
     <child link="${p}_distal_mimic_link"/>
     <axis xyz="1 0 0"/>
-    <limit lower="${min_grasping_finger}" upper="${max_grasping_finger}" effort="100.0" velocity="10.0"/>
-    <!-- <mimic joint="${p}_finger_proximal" multiplier="-1" offset="0" /> -->
+    <limit lower="${min_grasping_finger}" upper="${max_grasping_finger}" effort="10.0" velocity="1.0"/>
     <mimic joint="${p}_finger" multiplier="0.4689" offset="-0.554" />
     <dynamics damping="${damping}" friction="${friction}"/>
   </joint>
-  <!-- <gazebo reference="${p}_finger_distal_link"> -->
-  <!--   <selfCollide>false</selfCollide> -->
-  <!-- </gazebo> -->
-  <!-- <gazebo reference="${p}_finger_distal_link_mimic"> -->
-  <!--   <selfCollide>false</selfCollide> -->
-  <!-- </gazebo> -->
+  <gazebo reference="${p}_finger_distal_link">
+    <selfCollide>false</selfCollide>
+  </gazebo>
+  <gazebo reference="${p}_finger_distal_link_mimic">
+    <selfCollide>false</selfCollide>
+  </gazebo>
 </xacro:macro>
 </robot>

File: reachy_description/urdf/reachy.urdf.xacro (robot description, xacro)
@@ -74,10 +74,10 @@
   <!--   <child link="torso" /> -->
   <!-- </joint> -->
-  <!-- <link name="world" />
-  <joint name="world_joint" type="fixed">
-    <origin xyz="0 0 0.0" rpy="0 0 0" />
-    <parent link="world" />
-    <child link="base_link" />
-  </joint> -->
+  <!-- <link name="world" /> -->
+  <!-- <joint name="world_joint" type="fixed"> -->
+  <!--   <origin xyz="0 0 0.0" rpy="0 0 0" /> -->
+  <!--   <parent link="world" /> -->
+  <!--   <child link="base_link" /> -->
+  <!-- </joint> -->
   <link name="back_bar">
     <visual>
