Commit message: add mujoco plugin

File: reachy_controllers/dynamixel_control/dynamixel_description/ros2_control/dynamixel.ros2_control.xacro (robot description, xacro)
@@ -1,8 +1,12 @@
-<?xml version="1.0" ?>
+<?xml version="1.0"?>
 <robot xmlns:xacro="http://www.ros.org/wiki/xacro">
-  <xacro:include filename="$(find dynamixel_description)/ros2_control/dynamixel_actuator_control.ros2_control.xacro"/>
-  <!-- <xacro:include filename="$(find dynamixel_description)/ros2_control/dynamixel_gripper_axis_control.ros2_control.xacro"/> -->
-  <xacro:include filename="$(find dynamixel_description)/ros2_control/dynamixel_axis_control.ros2_control.xacro"/>
-  <xacro:include filename="$(find dynamixel_description)/ros2_control/dynamixel_raw_motor_control.ros2_control.xacro"/>
+  <xacro:include
+    filename="$(find dynamixel_description)/ros2_control/dynamixel_actuator_control.ros2_control.xacro" />
+  <!-- <xacro:include filename="$(find
+  dynamixel_description)/ros2_control/dynamixel_gripper_axis_control.ros2_control.xacro"/> -->
+  <xacro:include
+    filename="$(find dynamixel_description)/ros2_control/dynamixel_axis_control.ros2_control.xacro" />
+  <xacro:include
+    filename="$(find dynamixel_description)/ros2_control/dynamixel_raw_motor_control.ros2_control.xacro" />
   <xacro:macro name="dynamixel_control" params="name joint1 joint2 config_file ">
     <ros2_control name="${name}" type="system">
@@ -18,19 +22,25 @@
             <plugin>gazebo_ros2_control/GazeboSystem</plugin>
           </xacro:if>
-          <!-- Use fake components. -->
+          <!-- Else, when gazebo is not enabled -->
           <xacro:unless value="$(arg use_gazebo)">
-            <!-- <plugin>fake_components/GenericSystem</plugin> -->
-	    <!-- test -->
-          <plugin>dynamixel_2joints_system_hwi/DynamixelSystem</plugin>
-          <param name="dxl_config_file">${config_file}</param>
+            <!-- If mujoco mode is enabled -->
+            <xacro:if value="$(arg use_mujoco)">
+              <plugin>mujoco_ros2_control/MujocoSystem</plugin>
+            </xacro:if>
+            <!-- If neither gazebo nor mujoco are enabled -->
+            <xacro:unless value="$(arg use_mujoco)">
+              <!-- Pollen controller fake system -->
+              <plugin>dynamixel_2joints_system_hwi/DynamixelSystem</plugin>
+              <param name="dxl_config_file">${config_file}</param>
+            </xacro:unless>
           </xacro:unless>
         </xacro:if>
       </hardware>
-      <xacro:dynamixel_actuator_control name="${name}_${joint1}"/>
-      <xacro:dynamixel_actuator_control name="${name}_${joint2}"/>
+      <xacro:dynamixel_actuator_control name="${name}_${joint1}" />
+      <xacro:dynamixel_actuator_control name="${name}_${joint2}" />
       <xacro:dynamixel_axis_control name="${name}_${joint1}" />
       <xacro:dynamixel_axis_control name="${name}_${joint2}" />
-      <xacro:dynamixel_raw_motor_control name="${name}_${joint1}_raw_motor"/>
-      <xacro:dynamixel_raw_motor_control name="${name}_${joint2}_raw_motor"/>
+      <xacro:dynamixel_raw_motor_control name="${name}_${joint1}_raw_motor" />
+      <xacro:dynamixel_raw_motor_control name="${name}_${joint2}_raw_motor" />
     </ros2_control>
   </xacro:macro>

File: reachy_description/urdf/head.urdf.xacro (robot description, xacro)
@@ -1,35 +1,38 @@
 <?xml version="1.0"?>
 <robot xmlns:xacro="http://www.ros.org/wiki/xacro">
-  <xacro:arg name="depth_camera" default="true"/>
+  <xacro:arg name="depth_camera" default="true" />
   <xacro:property name="camera_link" value="0.05" /> <!-- Size of square 'camera' box -->
-  <xacro:property name="camera_convergence" value="0.0" /> <!-- convergence angle (rad) of the cameras. 0=parallel-->
-  <xacro:property name="neck_length" value="0.05"/>
-  <xacro:property name="neck_radius" value="0.03"/>
-  <xacro:property name="neck_mass" value="0.5"/>
+  <xacro:property name="camera_convergence" value="0.0" /> <!-- convergence angle (rad) of the
+  cameras. 0=parallel-->
+  <xacro:property name="neck_length" value="0.05" />
+  <xacro:property name="neck_radius" value="0.03" />
+  <xacro:property name="neck_mass" value="0.5" />
   <!-- <xacro:property name="neck_offset_x" value="-0.0465"/> -->
-  <xacro:property name="neck_offset_x" value="0.0"/>
-  <xacro:property name="neck_offset_y" value="0"/>
-  <xacro:property name="neck_offset_z" value="0.115"/>
-  <xacro:property name="neck_offset_pitch" value="${radians(10)}"/> <!-- 10 degrees -->
-  <xacro:property name="neck_offset_yaw" value="0.0"/>
-  <xacro:include filename="$(find orbita3d_description)/urdf/orbita3d.urdf.xacro"/>
-  <xacro:include filename="$(find dynamixel_description)/ros2_control/dynamixel.ros2_control.xacro"/>
-    <material name="camblack">
-        <color rgba="0.2 0.2 0.2 1"/>
-    </material>
-    <material name="neckwhite">
-        <color rgba="0.9 0.9 0.9 1"/>
-    </material>
+  <xacro:property name="neck_offset_x" value="0.0" />
+  <xacro:property name="neck_offset_y" value="0" />
+  <xacro:property name="neck_offset_z" value="0.115" />
+  <xacro:property name="neck_offset_pitch" value="${radians(10)}" /> <!-- 10 degrees -->
+  <xacro:property name="neck_offset_yaw" value="0.0" />
+  <xacro:include filename="$(find orbita3d_description)/urdf/orbita3d.urdf.xacro" />
+  <xacro:include filename="$(find dynamixel_description)/ros2_control/dynamixel.ros2_control.xacro" />
+  <material name="camblack">
+    <color rgba="0.2 0.2 0.2 1" />
+  </material>
+  <material name="neckwhite">
+    <color rgba="0.9 0.9 0.9 1" />
+  </material>
   <xacro:macro name="head" params="parent damping friction neck_config antenna_config">
-    <!-- xyz="${neck_offset_x} ${neck_offset_y} ${neck_offset_z}" rpy="${pi} ${neck_offset_pitch} ${neck_offset_yaw}" -->
-  <xacro:orbita3d
-    name="neck" parent="${parent}"
-    length="${neck_length}" radius="${neck_radius}" mass="${neck_mass}"
-    xyz="${neck_offset_x} ${neck_offset_y} ${neck_offset_z}" rpy="0 ${neck_offset_pitch} ${neck_offset_yaw}"
-    damping="${damping}" friction="${friction}"
-    config_file="${neck_config}"
+    <!-- xyz="${neck_offset_x} ${neck_offset_y} ${neck_offset_z}" rpy="${pi} ${neck_offset_pitch}
+    ${neck_offset_yaw}" -->
+    <xacro:orbita3d
+      name="neck" parent="${parent}"
+      length="${neck_length}" radius="${neck_radius}" mass="${neck_mass}"
+      xyz="${neck_offset_x} ${neck_offset_y} ${neck_offset_z}"
+      rpy="0 ${neck_offset_pitch} ${neck_offset_yaw}"
+      damping="${damping}" friction="${friction}"
+      config_file="${neck_config}"
     />
     <joint name="neck_fixed" type="fixed">
-      <origin xyz="0 0 0" rpy="0.0 0.0 0.0"/>
+      <origin xyz="0 0 0" rpy="0.0 0.0 0.0" />
       <parent link="neck_out_link" />
       <child link="head" />
@@ -38,23 +41,23 @@
     <link name="head">
       <inertial>
-        <origin xyz="0.0116978 -0.00022144 0.0611705" rpy="0.0 0.0 0.0"/>
-        <mass value="0.325"/>
-	 <inertia ixx="0.00085265" ixy="-0.00000298" ixz="0.00000932"
-		  iyx="-0.00000298" iyy="0.00063136" iyz="-0.000000039"
-		  izx="0.00000932" izy="-0.000000039" izz="0.0008951"/>
+        <origin xyz="0.0116978 -0.00022144 0.0611705" rpy="0.0 0.0 0.0" />
+        <mass value="0.325" />
+        <inertia ixx="0.00085265" ixy="-0.00000298" ixz="0.00000932"
+          iyx="-0.00000298" iyy="0.00063136" iyz="-0.000000039"
+          izx="0.00000932" izy="-0.000000039" izz="0.0008951" />
       </inertial>
       <visual>
-        <origin xyz="0.00 0.0 0.0" rpy="0.0 0.0 0.0"/>
+        <origin xyz="0.00 0.0 0.0" rpy="0.0 0.0 0.0" />
         <geometry>
-          <mesh filename="file://$(find reachy_description)/meshes/head_visual.dae"/>
+          <mesh filename="file://$(find reachy_description)/meshes/head_visual.dae" />
           <!-- <mesh filename="file://$(find reachy_description)/meshes/head_visual_high.dae"/> -->
         </geometry>
       </visual>
       <collision>
-	<!-- <origin xyz="0.0 0.0 0.05" rpy="0.0 0.0 0.0"/> -->
-	<origin xyz="0.0 0.0 0.0" rpy="0.0 0.0 0.0"/>
+        <!-- <origin xyz="0.0 0.0 0.05" rpy="0.0 0.0 0.0"/> -->
+        <origin xyz="0.0 0.0 0.0" rpy="0.0 0.0 0.0" />
         <geometry>
-	  <!-- <box size="0.12 0.162 0.1"/> -->
-          <mesh filename="file://$(find reachy_description)/meshes/head_collider.dae"/>
+          <!-- <box size="0.12 0.162 0.1"/> -->
+          <mesh filename="file://$(find reachy_description)/meshes/head_collider.dae" />
         </geometry>
       </collision>
@@ -62,11 +65,11 @@
     <link name="head_base">
       <inertial>
-        <origin xyz="0.0 0.0 0.0" rpy="0.0 0.0 0.0"/>
-        <mass value="0.001"/>
-        <inertia ixx="1.0e-6" ixy="1.0e-8" ixz="1.0e-8" iyy="1.0e-6" iyz="1.0e-8" izz="1.0e-6"/>
+        <origin xyz="0.0 0.0 0.0" rpy="0.0 0.0 0.0" />
+        <mass value="0.001" />
+        <inertia ixx="1.0e-6" ixy="1.0e-8" ixz="1.0e-8" iyy="1.0e-6" iyz="1.0e-8" izz="1.0e-6" />
       </inertial>
     </link>
     <joint name="head_base_fixed" type="fixed">
-      <origin xyz="0.0 0 0.0" rpy="0.0 0.0 0"/>
+      <origin xyz="0.0 0 0.0" rpy="0.0 0.0 0" />
       <parent link="head" />
       <child link="head_base" />
@@ -86,14 +89,14 @@
     <!--   <child link="head_tracker" /> -->
     <!-- </joint> -->
-    <link name="head_tip" >
-      <inertial>
-        <origin xyz="0.0 0.0 0.0" rpy="0.0 0.0 0.0"/>
-        <mass value="0.001"/>
-        <inertia ixx="1.0e-6" ixy="1.0e-8" ixz="1.0e-8" iyy="1.0e-6" iyz="1.0e-8" izz="1.0e-6"/>
+    <link name="head_tip">
+      <inertial>
+        <origin xyz="0.0 0.0 0.0" rpy="0.0 0.0 0.0" />
+        <mass value="0.001" />
+        <inertia ixx="1.0e-6" ixy="1.0e-8" ixz="1.0e-8" iyy="1.0e-6" iyz="1.0e-8" izz="1.0e-6" />
       </inertial>
     </link>
     <joint name="head_tip_fixed" type="fixed">
       <!-- between the cameras -->
-      <origin xyz="0.05643 0.0 0.062" rpy="0 0.0 0"/>
+      <origin xyz="0.05643 0.0 0.062" rpy="0 0.0 0" />
       <!-- Rotation center -->
       <!-- <origin xyz="0.0 0 0.0" rpy="0.0 0.0 0"/> -->
@@ -102,18 +105,18 @@
     </joint>
     <!-- test antennas -->
-    <link name="antenna_left_link" >
-      <inertial>
-	<origin xyz="0.0 0.0 0.0" rpy="0.0 0.0 0.0"/>
-	<mass value="0.001"/>
-	<inertia ixx="1.0e-6" ixy="1.0e-8" ixz="1.0e-8" iyy="1.0e-6" iyz="1.0e-8" izz="1.0e-6"/>
+    <link name="antenna_left_link">
+      <inertial>
+        <origin xyz="0.0 0.0 0.0" rpy="0.0 0.0 0.0" />
+        <mass value="0.001" />
+        <inertia ixx="1.0e-6" ixy="1.0e-8" ixz="1.0e-8" iyy="1.0e-6" iyz="1.0e-8" izz="1.0e-6" />
       </inertial>
       <!-- cylinder geometry -->
       <visual>
-	<origin xyz="0 0 0" rpy="0 0 0"/>
-	<geometry>
-	  <!-- <cylinder length="0.1" radius="0.005"/> -->
-        <mesh filename="file://$(find reachy_description)/meshes/head_antenna_visual.dae" />
-	</geometry>
-	<material name="neckwhite"/>
+        <origin xyz="0 0 0" rpy="0 0 0" />
+        <geometry>
+          <!-- <cylinder length="0.1" radius="0.005"/> -->
+          <mesh filename="file://$(find reachy_description)/meshes/head_antenna_visual.dae" />
+        </geometry>
+        <material name="neckwhite" />
       </visual>
     </link>
@@ -123,24 +126,25 @@
       <!-- <origin xyz="-0.023 0.055 0.091" rpy="${radians(32)} ${radians(-55)} ${radians(-90)}"/> -->
       <!-- Horrible... -->
-      <origin xyz="-0.023 0.055 0.091" rpy="${radians(4.225)} ${radians(-60.807)} ${radians(-57.500)}"/>
+      <origin xyz="-0.023 0.055 0.091"
+        rpy="${radians(4.225)} ${radians(-60.807)} ${radians(-57.500)}" />
       <parent link="head" />
       <child link="antenna_left_link" />
-      <axis xyz="0 0 1"/>
-      <limit effort="0.0" velocity="0.0" lower="${-pi/2}" upper="${pi/2}"/>
-    </joint>
-    <link name="antenna_right_link" >
-      <inertial>
-	<origin xyz="0.0 0.0 0.0" rpy="0.0 0.0 0.0"/>
-	<mass value="0.001"/>
-	<inertia ixx="1.0e-6" ixy="1.0e-8" ixz="1.0e-8" iyy="1.0e-6" iyz="1.0e-8" izz="1.0e-6"/>
+      <axis xyz="0 0 1" />
+      <limit effort="0.0" velocity="0.0" lower="${-pi/2}" upper="${pi/2}" />
+    </joint>
+    <link name="antenna_right_link">
+      <inertial>
+        <origin xyz="0.0 0.0 0.0" rpy="0.0 0.0 0.0" />
+        <mass value="0.001" />
+        <inertia ixx="1.0e-6" ixy="1.0e-8" ixz="1.0e-8" iyy="1.0e-6" iyz="1.0e-8" izz="1.0e-6" />
       </inertial>
       <!-- cylinder geometry -->
       <visual>
-	<origin xyz="0 0 0" rpy="0 0 0"/>
-	<geometry>
-	  <!-- <cylinder length="0.1" radius="0.005"/> -->
+        <origin xyz="0 0 0" rpy="0 0 0" />
+        <geometry>
+          <!-- <cylinder length="0.1" radius="0.005"/> -->
           <mesh filename="file://$(find reachy_description)/meshes/head_antenna_visual.dae" />
-	</geometry>
-	<material name="neckwhite"/>
+        </geometry>
+        <material name="neckwhite" />
       </visual>
     </link>
@@ -148,92 +152,119 @@
     <joint name="antenna_right" type="revolute">
       <!-- <origin xyz="0.0 -0.1 0.1" rpy="0 0.0 0"/> -->
-      <origin xyz="-0.023 -0.055 0.091" rpy="${radians(-4.225)} ${radians(-60.807)} ${radians(57.500)}"/>
+      <origin xyz="-0.023 -0.055 0.091"
+        rpy="${radians(-4.225)} ${radians(-60.807)} ${radians(57.500)}" />
       <parent link="head" />
       <child link="antenna_right_link" />
-      <axis xyz="0 0 1"/>
-      <limit effort="0.0" velocity="0.0" lower="${-pi/2}" upper="${pi/2}"/>
-    </joint>
-  <xacro:dynamixel_control
-    name="antenna" joint1="left" joint2="right"
-    config_file="${antenna_config}"
+      <axis xyz="0 0 1" />
+      <limit effort="0.0" velocity="0.0" lower="${-pi/2}" upper="${pi/2}" />
+    </joint>
+    <xacro:dynamixel_control
+      name="antenna" joint1="left" joint2="right"
+      config_file="${antenna_config}"
     />
     <!-- Reachy Cameras -->
-      <joint name="left_cam_fixed" type="fixed">
-	<origin xyz="0.03531 0.0325 0.062" rpy="0.0 0.0  ${-camera_convergence/2.0}"/>
-	<parent link="head" />
-	<child link="left_camera" />
-      </joint>
-      <link name="left_camera" >
-	<inertial>
-	  <mass value="1e-5" />
-	  <origin xyz="0 0 0" rpy="0 0 0"/>
-	  <inertia ixx="1e-6" ixy="0" ixz="0" iyy="1e-6" iyz="0" izz="1e-6" />
-	</inertial>
-      </link>
-      <link name="left_camera_optical">
-      <inertial>
-        <origin xyz="0.0 0.0 0.0" rpy="0.0 0.0 0.0"/>
-        <mass value="0.001"/>
-        <inertia ixx="1.0e-6" ixy="1.0e-8" ixz="1.0e-8" iyy="1.0e-6" iyz="1.0e-8" izz="1.0e-6"/>
-      </inertial>
-      </link>
-      <joint name="left_camera_optical_joint" type="fixed">
-	<!-- these values have to be these values otherwise the gazebo camera
+    <joint name="left_cam_fixed" type="fixed">
+      <origin xyz="0.03531 0.0325 0.062" rpy="0.0 0.0  ${-camera_convergence/2.0}" />
+      <parent link="head" />
+      <child link="left_camera" />
+    </joint>
+    <link name="left_camera">
+      <inertial>
+        <mass value="1e-5" />
+        <origin xyz="0 0 0" rpy="0 0 0" />
+        <inertia ixx="1e-6" ixy="0" ixz="0" iyy="1e-6" iyz="0" izz="1e-6" />
+      </inertial>
+    </link>
+    <link name="left_camera_optical">
+      <inertial>
+        <origin xyz="0.0 0.0 0.0" rpy="0.0 0.0 0.0" />
+        <mass value="0.001" />
+        <inertia ixx="1.0e-6" ixy="1.0e-8" ixz="1.0e-8" iyy="1.0e-6" iyz="1.0e-8" izz="1.0e-6" />
+      </inertial>
+    </link>
+    <joint name="left_camera_optical_joint" type="fixed">
+      <!-- these values have to be these values otherwise the gazebo camera
              image won't be aligned properly with the frame it is supposedly
              originating from -->
-	<origin xyz="0 0 0" rpy="${-pi/2.0} 0 ${-pi/2.0}"/>
-	<parent link="left_camera"/>
-	<child link="left_camera_optical"/>
-      </joint>
-      <joint name="right_cam_fixed" type="fixed">
-	<origin xyz="0.03531 -0.0325 0.062" rpy="0.0 0.0 ${camera_convergence/2.0}"/>
-	<parent link="head" />
-	<child link="right_camera" />
-      </joint>
-      <link name="right_camera" >
-	<inertial>
-	  <mass value="1e-5" />
-	  <origin xyz="0 0 0" rpy="0 0 0"/>
-	  <inertia ixx="1e-6" ixy="0" ixz="0" iyy="1e-6" iyz="0" izz="1e-6" />
-	</inertial>
-      </link>
-      <link name="right_camera_optical">
-      </link>
-      <joint name="right_camera_optical_joint" type="fixed">
-	<!-- these values have to be these values otherwise the gazebo camera
+      <origin xyz="0 0 0" rpy="${-pi/2.0} 0 ${-pi/2.0}" />
+      <parent link="left_camera" />
+      <child link="left_camera_optical" />
+    </joint>
+    <link name="left_camera_optical_frame">
+      <inertial>
+        <origin xyz="0.0 0.0 0.0" rpy="0.0 0.0 0.0" />
+        <mass value="0.001" />
+        <inertia ixx="1.0e-6" ixy="1.0e-8" ixz="1.0e-8" iyy="1.0e-6" iyz="1.0e-8" izz="1.0e-6" />
+      </inertial>
+    </link>
+    <joint name="left_camera_optical_frame_joint" type="fixed">
+      <!-- these values have to be these values otherwise the gazebo camera
              image won't be aligned properly with the frame it is supposedly
              originating from -->
-	<origin xyz="0 0 0" rpy="${-pi/2.0} 0 ${-pi/2.0}"/>
-	<!-- <origin xyz="0.03531 -0.0325 0.056" rpy="${-pi/2.0} 0 ${-pi/2.0}"/> -->
-	<parent link="right_camera"/>
-	<child link="right_camera_optical"/>
-      </joint>
-      <joint name="tof_cam_fixed" type="fixed">
-	<origin xyz="0.05643 0 0.061954" rpy="0.0 0.0 0"/>
-	<parent link="head" />
-	<child link="tof_camera" />
-      </joint>
-      <link name="tof_camera" >
-	<inertial>
-	  <mass value="1e-5" />
-	  <origin xyz="0 0 0" rpy="0 0 0"/>
-	  <inertia ixx="1e-6" ixy="0" ixz="0" iyy="1e-6" iyz="0" izz="1e-6" />
-	</inertial>
-      </link>
-      <link name="tof_camera_optical">
-      </link>
-      <joint name="tof_camera_optical_joint" type="fixed">
-	<!-- these values have to be these values otherwise the gazebo camera
+      <origin xyz="0 0 0" rpy="${-pi/2.0} 0 ${-pi/2.0}" />
+      <parent link="left_camera" />
+      <child link="left_camera_optical_frame" />
+    </joint>
+    <joint name="right_cam_fixed" type="fixed">
+      <origin xyz="0.03531 -0.0325 0.062" rpy="0.0 0.0 ${camera_convergence/2.0}" />
+      <parent link="head" />
+      <child link="right_camera" />
+    </joint>
+    <link name="right_camera">
+      <inertial>
+        <mass value="1e-5" />
+        <origin xyz="0 0 0" rpy="0 0 0" />
+        <inertia ixx="1e-6" ixy="0" ixz="0" iyy="1e-6" iyz="0" izz="1e-6" />
+      </inertial>
+    </link>
+    <link name="right_camera_optical">
+    </link>
+    <joint name="right_camera_optical_joint" type="fixed">
+      <!-- these values have to be these values otherwise the gazebo camera
              image won't be aligned properly with the frame it is supposedly
              originating from -->
-	<origin xyz="0 0 0" rpy="${-pi/2.0} 0 ${-pi/2.0}"/>
-	<!-- <origin xyz="0.03531 -0.0325 0.056" rpy="${-pi/2.0} 0 ${-pi/2.0}"/> -->
-	<parent link="tof_camera"/>
-	<child link="tof_camera_optical"/>
-      </joint>
+      <origin xyz="0 0 0" rpy="${-pi/2.0} 0 ${-pi/2.0}" />
+      <!-- <origin xyz="0.03531 -0.0325 0.056" rpy="${-pi/2.0} 0 ${-pi/2.0}"/> -->
+      <parent link="right_camera" />
+      <child link="right_camera_optical" />
+    </joint>
+    <link name="right_camera_optical_frame">
+    </link>
+    <joint name="right_camera_optical_frame_joint" type="fixed">
+      <!-- these values have to be these values otherwise the gazebo camera
+             image won't be aligned properly with the frame it is supposedly
+             originating from -->
+      <origin xyz="0 0 0" rpy="${-pi/2.0} 0 ${-pi/2.0}" />
+      <!-- <origin xyz="0.03531 -0.0325 0.056" rpy="${-pi/2.0} 0 ${-pi/2.0}"/> -->
+      <parent link="right_camera" />
+      <child link="right_camera_optical_frame" />
+    </joint>
+    <joint name="tof_cam_fixed" type="fixed">
+      <origin xyz="0.05643 0 0.061954" rpy="0.0 0.0 0" />
+      <parent link="head" />
+      <child link="tof_camera" />
+    </joint>
+    <link name="tof_camera">
+      <inertial>
+        <mass value="1e-5" />
+        <origin xyz="0 0 0" rpy="0 0 0" />
+        <inertia ixx="1e-6" ixy="0" ixz="0" iyy="1e-6" iyz="0" izz="1e-6" />
+      </inertial>
+    </link>
+    <link name="tof_camera_optical">
+    </link>
+    <joint name="tof_camera_optical_joint" type="fixed">
+      <!-- these values have to be these values otherwise the gazebo camera
+             image won't be aligned properly with the frame it is supposedly
+             originating from -->
+      <origin xyz="0 0 0" rpy="${-pi/2.0} 0 ${-pi/2.0}" />
+      <!-- <origin xyz="0.03531 -0.0325 0.056" rpy="${-pi/2.0} 0 ${-pi/2.0}"/> -->
+      <parent link="tof_camera" />
+      <child link="tof_camera_optical" />
+    </joint>
     <xacro:if value="$(arg use_gazebo)">
       <gazebo reference="left_camera">
-	<!-- <link name="left_camera"> -->
-	<sensor type="camera" name="left_camera">
+        <!-- <link name="left_camera"> -->
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