Commit message: wip

File: reachy_controllers/dynamixel_control/dynamixel_description/urdf/dynamixel_gripper.urdf.xacro (robot description, xacro)
@@ -27,11 +27,8 @@
       <xacro:if value="${side == 'right'}">
     <collision>
-      <!-- <origin xyz="0 0 0.04 " rpy="0 0 0"/> -->
       <origin xyz="0 0 0.0 " rpy="0 0 0"/>
       <geometry>
-        <!-- <box size="${gripper_radius} ${gripper_radius*2} ${gripper_length/2}"/> -->
-        <!-- <box size="0.08 0.12 0.07"/> -->
-	  <!-- <mesh filename="package://arm_description/meshes/pincette_right_collider.dae" /> -->
-	  <mesh filename="file://$(find dynamixel_description)/meshes/pincette_right_collider.dae" />
+	  <!-- <mesh filename="file://$(find dynamixel_description)/meshes/pincette_right_collider.dae" /> -->
+	  <mesh filename="file://$(find dynamixel_description)/meshes/pincette_base_collider.dae" />
       </geometry>
     </collision>
@@ -39,6 +36,6 @@
       	<origin xyz="0 0 0" rpy="0 0 0"/>
       	<geometry>
-	  <!-- <mesh filename="file://$(find arm_description)/meshes/pincette_right_visual.dae" /> -->
-	  <mesh filename="file://$(find dynamixel_description)/meshes/pincette_right_visual.dae" />
+	  <!-- <mesh filename="file://$(find dynamixel_description)/meshes/pincette_right_visual.dae" /> -->
+	  <mesh filename="file://$(find dynamixel_description)/meshes/pincette_base_visual.dae" />
       	</geometry>
       </visual>
@@ -53,11 +50,8 @@
   <xacro:if value="${side == 'left'}">
     <collision>
-      <!-- <origin xyz="0 0 0.04 " rpy="0 0 0"/> -->
       <origin xyz="0 0 0.0 " rpy="0 0 0"/>
       <geometry>
-        <!-- <box size="${gripper_radius} ${gripper_radius*2} ${gripper_length/2}"/> -->
-        <!-- <box size="0.08 0.12 0.07"/> -->
-	  <!-- <mesh filename="file://$(find arm_description)/meshes/pincette_left_collider.dae" /> -->
-	  <mesh filename="file://$(find dynamixel_description)/meshes/pincette_left_collider.dae" />
+	  <!-- <mesh filename="file://$(find dynamixel_description)/meshes/pincette_left_collider.dae" /> -->
+	  <mesh filename="file://$(find dynamixel_description)/meshes/pincette_base_collider.dae" />
       </geometry>
     </collision>
@@ -65,6 +59,6 @@
       	<origin xyz="0 0 0" rpy="0 0 0"/>
       	<geometry>
-	  <!-- <mesh filename="file://$(find arm_description)/meshes/pincette_left_visual.dae" /> -->
-	  <mesh filename="file://$(find dynamixel_description)/meshes/pincette_left_visual.dae" />
+	  <!-- <mesh filename="file://$(find dynamixel_description)/meshes/pincette_left_visual.dae" /> -->
+	  <mesh filename="file://$(find dynamixel_description)/meshes/pincette_base_visual.dae" />
       	</geometry>
       </visual>
@@ -107,8 +101,4 @@
       </inertial>
     <collision>
-      <!-- <origin xyz="0 0.006 0.03 " rpy="0 0 0"/> -->
-      <!-- <geometry> -->
-      <!--   <box size="0.031 0.026 0.06"/> -->
-      <!-- </geometry> -->
       <origin xyz="0 0.00 0.0 " rpy="0 0 0"/>
       <geometry>
@@ -134,5 +124,4 @@
       </inertial>
     <collision>
-      <!-- <origin xyz="0 0.006 0.03 " rpy="0 0 0"/> -->
       <origin xyz="0 0.0 0.0 " rpy="0 0 0"/>
       <geometry>
@@ -177,9 +166,6 @@
       </inertial>
     <collision>
-      <!-- <origin xyz="0 0.0015 0.023 " rpy="0 0 0"/> -->
       <origin xyz="0 0.0 0.0 " rpy="0 0 0"/>
       <geometry>
-        <!-- <box size="0.031 0.026 0.046"/> -->
-	  <!-- <mesh filename="file://$(find arm_description)/meshes/pincette_distal_collider.dae" /> -->
 	  <mesh filename="file://$(find dynamixel_description)/meshes/pincette_distal_collider.dae" />
       </geometry>
@@ -188,5 +174,4 @@
       <origin xyz="0 0 0 " rpy="0 0 0"/>
       <geometry>
-	  <!-- <mesh filename="file://$(find arm_description)/meshes/pincette_distal.dae" /> -->
 	  <mesh filename="file://$(find dynamixel_description)/meshes/pincette_distal.dae" />
       </geometry>
@@ -212,9 +197,6 @@
       </inertial>
     <collision>
-      <!-- <origin xyz="0 0.0015 0.023 " rpy="0 0 0"/> -->
       <origin xyz="0 0.00 0.0 " rpy="0 0 0"/>
       <geometry>
-        <!-- <box size="0.031 0.026 0.046"/> -->
-	  <!-- <mesh filename="file://$(find arm_description)/meshes/pincette_distal_collider.dae" /> -->
 	  <mesh filename="file://$(find dynamixel_description)/meshes/pincette_distal_collider.dae" />
       </geometry>
@@ -223,5 +205,4 @@
       <origin xyz="0 0 0 " rpy="0 0 0"/>
       <geometry>
-	  <!-- <mesh filename="file://$(find arm_description)/meshes/pincette_distal.dae" /> -->
 	  <mesh filename="file://$(find dynamixel_description)/meshes/pincette_distal.dae" />
       </geometry>

File: reachy_description/urdf/head.urdf.xacro (robot description, xacro)
@@ -10,5 +10,5 @@
   <xacro:property name="neck_offset_x" value="0.0"/>
   <xacro:property name="neck_offset_y" value="0"/>
-  <xacro:property name="neck_offset_z" value="0.125"/>
+  <xacro:property name="neck_offset_z" value="0.115"/>
   <xacro:property name="neck_offset_pitch" value="${radians(10)}"/> <!-- 10 degrees -->
   <xacro:property name="neck_offset_yaw" value="0.0"/>
@@ -48,4 +48,5 @@
         <geometry>
           <mesh filename="file://$(find reachy_description)/meshes/head_visual.dae"/>
+          <!-- <mesh filename="file://$(find reachy_description)/meshes/head_visual_high.dae"/> -->
         </geometry>
       </visual>
@@ -94,5 +95,5 @@
     <joint name="head_tip_fixed" type="fixed">
       <!-- between the cameras -->
-      <origin xyz="0.057 0.0 0.056" rpy="0 0.0 0"/>
+      <origin xyz="0.05643 0.0 0.062" rpy="0 0.0 0"/>
       <!-- Rotation center -->
       <!-- <origin xyz="0.0 0 0.0" rpy="0.0 0.0 0"/> -->
@@ -111,5 +112,6 @@
 	<origin xyz="0 0 0" rpy="0 0 0"/>
 	<geometry>
-	  <cylinder length="0.1" radius="0.005"/>
+	  <!-- <cylinder length="0.1" radius="0.005"/> -->
+        <mesh filename="file://$(find reachy_description)/meshes/head_antenna_visual.dae" />
 	</geometry>
 	<material name="neckwhite"/>
@@ -118,9 +120,12 @@
     <!-- revolute joint -->
     <joint name="antenna_left" type="revolute">
-      <origin xyz="0.0 0.1 0.1" rpy="0 0.0 0"/>
+      <!-- <origin xyz="-0.023 0.055 0.091" rpy="${radians(145-90)} 0.0 ${radians(32)}"/> -->
+      <!-- <origin xyz="-0.023 0.055 0.091" rpy="${radians(32)} ${radians(-55)} ${radians(-90)}"/> -->
+      <!-- Horrible... -->
+      <origin xyz="-0.023 0.055 0.091" rpy="${radians(4.225)} ${radians(-60.807)} ${radians(-57.500)}"/>
       <parent link="head" />
       <child link="antenna_left_link" />
-      <axis xyz="0 1 0"/>
-      <limit effort="0.0" velocity="0.0" lower="-0.5" upper="0.5"/>
+      <axis xyz="0 0 1"/>
+      <limit effort="0.0" velocity="0.0" lower="${-pi/2}" upper="${pi/2}"/>
     </joint>
     <link name="antenna_right_link" >
@@ -134,5 +139,6 @@
 	<origin xyz="0 0 0" rpy="0 0 0"/>
 	<geometry>
-	  <cylinder length="0.1" radius="0.005"/>
+	  <!-- <cylinder length="0.1" radius="0.005"/> -->
+          <mesh filename="file://$(find reachy_description)/meshes/head_antenna_visual.dae" />
 	</geometry>
 	<material name="neckwhite"/>
@@ -141,9 +147,10 @@
     <!-- revolute joint -->
     <joint name="antenna_right" type="revolute">
-      <origin xyz="0.0 -0.1 0.1" rpy="0 0.0 0"/>
+      <!-- <origin xyz="0.0 -0.1 0.1" rpy="0 0.0 0"/> -->
+      <origin xyz="-0.023 -0.055 0.091" rpy="${radians(-4.225)} ${radians(-60.807)} ${radians(57.500)}"/>
       <parent link="head" />
       <child link="antenna_right_link" />
-      <axis xyz="0 1 0"/>
-      <limit effort="0.0" velocity="0.0" lower="-0.5" upper="0.5"/>
+      <axis xyz="0 0 1"/>
+      <limit effort="0.0" velocity="0.0" lower="${-pi/2}" upper="${pi/2}"/>
     </joint>
   <xacro:dynamixel_control
@@ -153,5 +160,5 @@
     <!-- Reachy Cameras -->
       <joint name="left_cam_fixed" type="fixed">
-	<origin xyz="0.03531 0.0325 0.056" rpy="0.0 0.0  ${-camera_convergence/2.0}"/>
+	<origin xyz="0.03531 0.0325 0.062" rpy="0.0 0.0  ${-camera_convergence/2.0}"/>
 	<parent link="head" />
 	<child link="left_camera" />
@@ -180,5 +187,5 @@
       </joint>
       <joint name="right_cam_fixed" type="fixed">
-	<origin xyz="0.03531 -0.0325 0.056" rpy="0.0 0.0 ${camera_convergence/2.0}"/>
+	<origin xyz="0.03531 -0.0325 0.062" rpy="0.0 0.0 ${camera_convergence/2.0}"/>
 	<parent link="head" />
 	<child link="right_camera" />
@@ -201,4 +208,27 @@
 	<parent link="right_camera"/>
 	<child link="right_camera_optical"/>
+      </joint>
+      <joint name="tof_cam_fixed" type="fixed">
+	<origin xyz="0.05643 0 0.061954" rpy="0.0 0.0 0"/>
+	<parent link="head" />
+	<child link="tof_camera" />
+      </joint>
+      <link name="tof_camera" >
+	<inertial>
+	  <mass value="1e-5" />
+	  <origin xyz="0 0 0" rpy="0 0 0"/>
+	  <inertia ixx="1e-6" ixy="0" ixz="0" iyy="1e-6" iyz="0" izz="1e-6" />
+	</inertial>
+      </link>
+      <link name="tof_camera_optical">
+      </link>
+      <joint name="tof_camera_optical_joint" type="fixed">
+	<!-- these values have to be these values otherwise the gazebo camera
+             image won't be aligned properly with the frame it is supposedly
+             originating from -->
+	<origin xyz="0 0 0" rpy="${-pi/2.0} 0 ${-pi/2.0}"/>
+	<!-- <origin xyz="0.03531 -0.0325 0.056" rpy="${-pi/2.0} 0 ${-pi/2.0}"/> -->
+	<parent link="tof_camera"/>
+	<child link="tof_camera_optical"/>
       </joint>
     <xacro:if value="$(arg use_gazebo)">
