Commit message: wip

File: reachy_description/urdf/reachy.urdf.xacro (robot description, xacro)
@@ -45,4 +45,36 @@
   <xacro:arg name="grippers_config" default="$(find dynamixel_description)/config/two_fake.yaml"/>
   <xacro:arg name="robot_model" default="none" />
+  <!-- all the robot configurations -->
+  <xacro:property name="mobile_base" value="false" />
+  <xacro:property name="left_arm" value="false" />
+  <xacro:property name="right_arm" value="false" />
+  <xacro:property name="left_gripper" value="false" />
+  <xacro:property name="right_gripper" value="false" />
+  <xacro:property name="robot_config" value="$(arg robot_config)" />
+  <xacro:if value="${robot_config == 'full_kit'}">
+      <xacro:property name="mobile_base" value="true" />
+      <xacro:property name="left_arm" value="true" />
+      <xacro:property name="left_gripper" value="true" />
+      <xacro:property name="right_arm" value="true" />
+      <xacro:property name="right_gripper" value="true" />
+  </xacro:if>
+  <xacro:if value="${robot_config == 'left_arm'}">
+      <xacro:property name="mobile_base" value="true" />
+      <xacro:property name="left_arm" value="true" />
+      <xacro:property name="left_gripper" value="true" />
+  </xacro:if>
+  <xacro:if value="${robot_config == 'right_arm'}">
+      <xacro:property name="mobile_base" value="true" />
+      <xacro:property name="right_arm" value="true" />
+      <xacro:property name="right_gripper" value="true" />
+  </xacro:if>
+  <xacro:if value="${robot_config == 'left_arm_no_gripper'}">
+      <xacro:property name="mobile_base" value="true" />
+      <xacro:property name="left_arm" value="true" />
+  </xacro:if>
+  <xacro:if value="${robot_config == 'right_arm_no_gripper'}">
+      <xacro:property name="mobile_base" value="true" />
+      <xacro:property name="right_arm" value="true" />
+  </xacro:if>
   <!-- config  -->
   <!-- MODEL PARAMETERS -->
@@ -51,6 +83,5 @@
   <xacro:property name="damping" value="0.1" />
   <xacro:property name="friction" value="0.1" />
-  <!-- Height of the Torso Origin Min=0.9 Max=1.3 (TODO: make it a parameter at launch)  -->
-  <xacro:property name="base_height" value="1.2" />
+  <!-- Base height (torso) = 1000mm when back bar joint=525mm -->
   <!-- Parameters for the 3 bar base height -->
   <xacro:property name="back_bar_min_length" value="0.520" />
@@ -59,13 +90,7 @@
   <xacro:property name="bar_angle" value="${radians(10.937)}" />
   <xacro:property name="bar_angle_offset" value="${pi/2-atan2(back_bar_min_length-0.03-0.018,bar_small_triangle_base-0.09)}" />
-  <xacro:property name="bar_triangle_base" value="0.226186" />
-  <!-- <xacro:property name="bar_small_triangle_base" value="0.13857" /> -->
   <xacro:property name="bar_small_triangle_base" value="0.186" />
   <xacro:property name="back_bar_z" value="0.241" />
   <xacro:property name="back_bar_x" value="-0.09" />
-  <!-- <xacro:property name="left_bar_x" value="0.080966" /> -->
-  <!-- <xacro:property name="left_bar_y" value="0.117182" /> -->
-  <!-- <xacro:property name="right_bar_x" value="0.080966" /> -->
-  <!-- <xacro:property name="right_bar_y" value="-0.117182" /> -->
   <xacro:property name="left_bar_x" value="0.084" />
   <xacro:property name="left_bar_y" value="0.066" />
@@ -75,73 +100,4 @@
   <!-- <xacro:property name="back_bar_length" value="${base_height-0.2-back_bar_z}" /> -->
   <xacro:property name="back_bar_length" value="0.485" />
-  <xacro:property name="front_bar_length"
-    value="${sqrt(back_bar_length*back_bar_length+bar_small_triangle_base*bar_small_triangle_base)}" />
-  <!-- <link name="back_bar"> -->
-  <!--   <visual> -->
-  <!--     <origin xyz="0 0 ${back_bar_length/2}" rpy="0 0 0" /> -->
-  <!--     <geometry> -->
-  <!--       <box size="0.04 0.04 ${back_bar_length}" /> -->
-  <!--     </geometry> -->
-  <!--     <xacro:reachy_grey /> -->
-  <!--   </visual> -->
-  <!--   <collision> -->
-  <!--     <origin xyz="0 0 ${back_bar_length/2}" rpy="0 0 0" /> -->
-  <!--     <geometry> -->
-  <!--       <box size="0.04 0.04 ${back_bar_length}" /> -->
-  <!--     </geometry> -->
-  <!--   </collision> -->
-  <!-- </link> -->
-  <!-- <link name="left_bar"> -->
-  <!--   <visual> -->
-  <!--     <origin xyz="0.0 0 ${front_bar_length/2}" rpy="0 0 0" /> -->
-  <!--     <geometry> -->
-  <!--       <box size="0.04 0.04 ${front_bar_length}" /> -->
-  <!--     </geometry> -->
-  <!--     <xacro:reachy_grey /> -->
-  <!--   </visual> -->
-  <!--   <collision> -->
-  <!--     <origin xyz="0.0 0 ${front_bar_length/2}" rpy="0 0 0" /> -->
-  <!--     <geometry> -->
-  <!--       <box size="0.04 0.04 ${front_bar_length}" /> -->
-  <!--     </geometry> -->
-  <!--   </collision> -->
-  <!-- </link> -->
-  <!-- <link name="right_bar"> -->
-  <!--   <visual> -->
-  <!--     <origin xyz="0.0 0 ${front_bar_length/2}" rpy="0 0 0" /> -->
-  <!--     <geometry> -->
-  <!--       <box size="0.04 0.04 ${front_bar_length}" /> -->
-  <!--     </geometry> -->
-  <!--     <xacro:reachy_grey /> -->
-  <!--   </visual> -->
-  <!--   <collision> -->
-  <!--     <origin xyz="0.0 0 ${front_bar_length/2}" rpy="0 0 0" /> -->
-  <!--     <geometry> -->
-  <!--       <box size="0.04 0.04 ${front_bar_length}" /> -->
-  <!--     </geometry> -->
-  <!--   </collision> -->
-  <!-- </link> -->
-  <!-- <joint name="back_bar_joint" type="fixed"> -->
-  <!--   <!-\- <origin xyz="-0.122 0 0.057" rpy="0 0 0"/> -\-> -->
-  <!--   <origin xyz="${back_bar_x} 0 ${back_bar_z}" rpy="0 0 0" /> -->
-  <!--   <parent link="base_link" /> -->
-  <!--   <child link="back_bar" /> -->
-  <!-- </joint> -->
-  <!-- <joint name="left_bar_joint" type="fixed"> -->
-  <!--   <!-\- <origin xyz="0.080966 0.11718 0.057" rpy="0 -->
-  <!--   ${-pi/2+atan2(back_bar_length,bar_small_triangle_base)} ${bar_angle}"/> -\-> -->
-  <!--   <origin xyz="${left_bar_x} ${left_bar_y} ${back_bar_z}" -->
-  <!--     rpy="0 ${-pi/2+atan2(back_bar_length,bar_small_triangle_base)} ${bar_angle}" /> -->
-  <!--   <parent link="base_link" /> -->
-  <!--   <child link="left_bar" /> -->
-  <!-- </joint> -->
-  <!-- <joint name="right_bar_joint" type="fixed"> -->
-  <!--   <!-\- <origin xyz="0.080966 -0.11718 0.057" rpy="0 -->
-  <!--   ${-pi/2+atan2(back_bar_length,bar_small_triangle_base)} ${-bar_angle}"/> -\-> -->
-  <!--   <origin xyz="${right_bar_x} ${right_bar_y} ${back_bar_z}" -->
-  <!--     rpy="0 ${-pi/2+atan2(back_bar_length,bar_small_triangle_base)} ${-bar_angle}" /> -->
-  <!--   <parent link="base_link" /> -->
-  <!--   <child link="right_bar" /> -->
-  <!-- </joint> -->
   <link name="back_bar_base">
    <visual>
@@ -155,5 +111,5 @@
       <origin xyz="0 0 ${back_bar_length/2}" rpy="0 0 0" />
       <geometry>
-        <box size="0.04 0.04 ${back_bar_length}" />
+        <box size="0.05 0.05 ${back_bar_length}" />
       </geometry>
     </collision>
@@ -170,5 +126,5 @@
       <origin xyz="0 0 ${back_bar_length/2}" rpy="0 0 0" />
       <geometry>
-        <box size="0.03 0.03 ${back_bar_length}" />
+        <box size="0.05 0.05 ${back_bar_length}" />
       </geometry>
     </collision>
@@ -181,4 +137,22 @@
     <axis xyz="0 0 1"/>
   </joint>
+    <ros2_control name="tripod" type="system">
+      <hardware>
+          <!-- Use gazebo as hardware simulation. -->
+          <xacro:if value="$(arg use_gazebo)">
+            <plugin>gazebo_ros2_control/GazeboSystem</plugin>
+          </xacro:if>
+          <!-- Use fake components. -->
+          <xacro:unless value="$(arg use_gazebo)">
+            <plugin>fake_components/GenericSystem</plugin>
+          </xacro:unless>
+      </hardware>
+    <joint name="back_bar_prism_joint">
+      <state_interface name="position">
+        <param name="initial_value">0.0</param>
+      </state_interface>
+      <command_interface name="position"/>
+    </joint>
+    </ros2_control>
   <joint name="back_bar_joint" type="fixed">
     <origin xyz="${back_bar_x} 0 ${back_bar_z}" rpy="0 0 0" />
@@ -197,5 +171,5 @@
       <origin xyz="0 0 ${back_bar_length/2}" rpy="0 0 0" />
       <geometry>
-        <box size="0.04 0.04 ${back_bar_length}" />
+        <box size="0.05 0.05 ${back_bar_length}" />
       </geometry>
     </collision>
@@ -232,4 +206,5 @@
     <limit effort="1000.0" lower="-10.0" upper="10.0" velocity="0.5"/>
     <axis xyz="0 1 0"/>
+    <!-- 3rd order poly fit (pretty good): -0.82037152*x**3 + 2.02405982*x**2 -1.84920731*x + 0.73024573 -->
     <!-- fit of the arctan -->
     <mimic joint="back_bar_prism_joint" multiplier="0.2864183599287582" offset="-0.1967146343049915" />
@@ -248,5 +223,5 @@
       <origin xyz="0 0 ${back_bar_length/2}" rpy="0 0 0" />
       <geometry>
-        <box size="0.03 0.03 ${back_bar_length}" />
+        <box size="0.05 0.05 ${back_bar_length}" />
       </geometry>
     </collision>
@@ -272,5 +247,5 @@
       <origin xyz="0 0 ${back_bar_length/2}" rpy="0 0 0" />
       <geometry>
-        <box size="0.04 0.04 ${back_bar_length}" />
+        <box size="0.05 0.05 ${back_bar_length}" />
       </geometry>
     </collision>
@@ -323,5 +298,5 @@
       <origin xyz="0 0 ${back_bar_length/2}" rpy="0 0 0" />
       <geometry>
-        <box size="0.03 0.03 ${back_bar_length}" />
+        <box size="0.05 0.05 ${back_bar_length}" />
       </geometry>
     </collision>
@@ -340,7 +315,6 @@
       <origin xyz="0 0 0 " rpy="0 0 0" />
       <geometry>
-        <!-- <mesh filename="package://reachy_description/meshes/torso_visual_high.dae" /> -->
-        <mesh filename="file://$(find reachy_description)/meshes/torso_visual_high.dae" />
-        <!-- <mesh filename="file://$(find reachy_description)/meshes/torso_visual_high2.dae" /> -->
+        <!-- <mesh filename="file://$(find reachy_description)/meshes/torso_visual_high.dae" /> -->
+        <mesh filename="file://$(find reachy_description)/meshes/torso_visual.dae" />
       </geometry>
     </visual>
@@ -356,26 +330,26 @@
       <origin xyz="0 0 0 " rpy="0 0 0" />
       <geometry>
-        <!-- <mesh filename="package://reachy_description/meshes/torso_collider_no_cone.dae" /> -->
-        <mesh filename="file://$(find reachy_description)/meshes/torso_collider_no_cone.dae" />
+        <!-- <mesh filename="file://$(find reachy_description)/meshes/torso_collider_no_cone.dae" /> -->
+        <mesh filename="file://$(find reachy_description)/meshes/torso_collider.dae" />
       </geometry>
     </collision>
   </link>
   <joint name="torso_base" type="fixed">
-    <origin xyz="0.08 0 ${0.235+back_bar_length-0.035}" rpy="0 0 0" />
+    <origin xyz="0.08 0 ${0.235+back_bar_length}" rpy="0 0 0" />
     <parent link="back_bar_inner" />
     <child link="torso" />
   </joint>
-  <link name="logo">
-    <inertial>
-      <origin xyz="0.0 0.0 0.0" rpy="0.0 0.0 0.0" />
-      <mass value="0.001" />
-      <inertia ixx="1.0e-6" ixy="1.0e-8" ixz="1.0e-8" iyy="1.0e-6" iyz="1.0e-8" izz="1.0e-6" />
-    </inertial>
-  </link>
-  <joint name="logo_joint" type="fixed">
-    <origin xyz="0.047 0 0.0" rpy="0 0 0" />
-    <parent link="torso" />
-    <child link="logo" />
-  </joint>
+  <!-- <link name="logo"> -->
+  <!--   <inertial> -->
+  <!--     <origin xyz="0.0 0.0 0.0" rpy="0.0 0.0 0.0" /> -->
+  <!--     <mass value="0.001" /> -->
+  <!--     <inertia ixx="1.0e-6" ixy="1.0e-8" ixz="1.0e-8" iyy="1.0e-6" iyz="1.0e-8" izz="1.0e-6" /> -->
+  <!--   </inertial> -->
+  <!-- </link> -->
+  <!-- <joint name="logo_joint" type="fixed"> -->
+  <!--   <origin xyz="0.047 0 0.0" rpy="0 0 0" /> -->
+  <!--   <parent link="torso" /> -->
+  <!--   <child link="logo" /> -->
+  <!-- </joint> -->
   <!-- <gazebo reference="torso"> -->
   <!--   <!-\- <material>Gazebo/Black</material> -\-> -->
@@ -389,4 +363,5 @@
   />
   <!-- RIGHT ARM -->
+  <xacro:if value="${right_arm}">
   <xacro:arm
     prefix="r" parent="torso" side="right"
@@ -397,4 +372,6 @@
     robot_model="$(arg robot_model)"
   />
+</xacro:if>
+  <xacro:if value="${right_gripper}">
     <xacro:dynamixel_gripper
       prefix="r_hand" parent="r_wrist_out_link" side="right"
@@ -432,5 +409,7 @@
       <child link="r_arm_tip_bottom" />
     </joint>
+</xacro:if>
   <!-- LEFT ARM -->
+  <xacro:if value="${left_arm}">
   <xacro:arm
     prefix="l" parent="torso" side="left"
@@ -441,4 +420,6 @@
     robot_model="$(arg robot_model)"
   />
+</xacro:if>
+  <xacro:if value="${left_gripper}">
     <xacro:dynamixel_gripper
       prefix="l_hand" parent="l_wrist_out_link" side="right"
@@ -476,8 +457,11 @@
       <child link="l_arm_tip_bottom" />
     </joint>
+</xacro:if>
+<xacro:if value="${left_gripper or right_gripper}">
   <xacro:dynamixel_gripper_control
     name="gripper" joint1="l_hand" joint2="r_hand"
     config_file="$(arg grippers_config)"
     />
+</xacro:if>
   <link name="depth_cam_l_optical">
     <inertial>
@@ -495,12 +479,36 @@
   </link>
   <joint name="depth_cam_l_optical_joint" type="fixed">
-    <origin xyz="0.002597 0.009989 0.038089" rpy="${radians(-48.0-90.0)} 0.0 ${-pi/2}" />
-    <parent link="logo" />
+    <origin xyz="0.058 0.025 -0.03" rpy="${radians(-47.5-90.0)} 0.0 ${-pi/2}" />
+    <parent link="torso" />
     <child link="depth_cam_l_optical" />
   </joint>
   <joint name="depth_cam_l_frame_joint" type="fixed">
-    <origin xyz="0.002597 0.009989 0.038089" rpy="0.0 ${radians(48.0)} 0.0" />
-    <parent link="logo" />
+    <origin xyz="0.058 0.025 -0.03" rpy="0.0 ${radians(47.5)} 0.0" />
+    <parent link="torso" />
     <child link="depth_cam_l_frame" />
+  </joint>
+  <link name="depth_cam_rgb_optical">
+    <inertial>
+      <origin xyz="0.0 0.0 0.0" rpy="0.0 0.0 0.0" />
+      <mass value="0.001" />
+      <inertia ixx="1.0e-6" ixy="1.0e-8" ixz="1.0e-8" iyy="1.0e-6" iyz="1.0e-8" izz="1.0e-6" />
+    </inertial>
+  </link>
+  <link name="depth_cam_rgb_frame">
+    <inertial>
+      <origin xyz="0.0 0.0 0.0" rpy="0.0 0.0 0.0" />
+      <mass value="0.001" />
+      <inertia ixx="1.0e-6" ixy="1.0e-8" ixz="1.0e-8" iyy="1.0e-6" iyz="1.0e-8" izz="1.0e-6" />
+    </inertial>
+  </link>
+  <joint name="depth_cam_rgb_optical_joint" type="fixed">
+    <origin xyz="0.058 0.0155 -0.03" rpy="${radians(-47.5-90.0)} 0.0 ${-pi/2}" />
+    <parent link="torso" />
+    <child link="depth_cam_rgb_optical" />
+  </joint>
+  <joint name="depth_cam_rgb_frame_joint" type="fixed">
+    <origin xyz="0.058 0.0155 -0.03" rpy="0.0 ${radians(47.5)} 0.0" />
+    <parent link="torso" />
+    <child link="depth_cam_rgb_frame" />
   </joint>
   <link name="depth_cam_r_optical">
@@ -519,11 +527,11 @@
   </link>
   <joint name="depth_cam_r_optical_joint" type="fixed">
-    <origin xyz="0.002597 -0.009989 0.038089" rpy="${radians(-48.0-90.0)} 0.0 ${-pi/2}" />
-    <parent link="logo" />
+    <origin xyz="0.058 -0.025 -0.03" rpy="${radians(-47.5-90.0)} 0.0 ${-pi/2}" />
+    <parent link="torso" />
     <child link="depth_cam_r_optical" />
   </joint>
   <joint name="depth_cam_r_frame_joint" type="fixed">
-    <origin xyz="0.002597 -0.009989 0.038089" rpy="0.0 ${radians(48.0)} 0.0 " />
-    <parent link="logo" />
+    <origin xyz="0.058 -0.025 -0.03" rpy="0.0 ${radians(47.5)} 0.0 " />
+    <parent link="torso" />
     <child link="depth_cam_r_frame" />
   </joint>
@@ -662,6 +670,4 @@
         </noise>
       </camera>
-      <!-- https://github.com/mlherd/ros2_turtlebot3_waffle_intel_realsense -->
-      <!-- <plugin name="intel_realsense_d430_depth_driver" filename="libgazebo_ros_camera.so"> -->
       <plugin name="depth_driver" filename="libgazebo_ros_camera.so">
         <ros>

Commit message: Add colored meshes.

File: reachy_controllers/dynamixel_control/dynamixel_description/urdf/dynamixel_gripper.urdf.xacro (robot description, xacro)
@@ -37,6 +37,5 @@
       	<origin xyz="0 0 0" rpy="0 0 0"/>
       	<geometry>
-	  <!-- <mesh filename="file://$(find dynamixel_description)/meshes/pincette_right_visual.dae" /> -->
-	  <mesh filename="file://$(find dynamixel_description)/meshes/pincette_base_visual.dae" />
+	  <mesh filename="file://$(find dynamixel_description)/meshes/pincette_right_visual.dae" />
       	</geometry>
       </visual>
@@ -60,6 +59,5 @@
       	<origin xyz="0 0 0" rpy="0 0 0"/>
       	<geometry>
-	  <!-- <mesh filename="file://$(find dynamixel_description)/meshes/pincette_left_visual.dae" /> -->
-	  <mesh filename="file://$(find dynamixel_description)/meshes/pincette_base_visual.dae" />
+	  <mesh filename="file://$(find dynamixel_description)/meshes/pincette_left_visual.dae" />
       	</geometry>
       </visual>
